File: eagle/row.sch (EAGLE design)
At the start: 14 parts

Commit message: port over routed row from dropbox
Parts:
- removed OUT: (no value), nonolith:HEADER-1X4
- removed S01, S02, S03, S04: MPL115A, nonolith:MPL115A
- removed U$5: ATTINY45, SparkFun:ATTINY45
- added S10, S20, S30, S40: MPL115A, nonolith:MPL115A
- C0, C2, C3, C4: device nonolith:CAP_CERAMIC0402 -> nonolith:CAP_CERAMIC0603
Connections:
- net B0 renamed ADDR00
- net RESET renamed RESET0
- net RST0 renamed RST00
- removed net B1: UC0.PB1
- removed net B2: UC0.PB2
- removed net B3: UC0.PA7/ADC7
- removed net CAP01: C1.P$1, S01.CAP
- removed net CAP02: C2.P$1, S02.CAP
- removed net CAP03: C3.P$1, S03.CAP
- removed net CAP04: C4.P$1, S04.CAP
- removed net RST1: S01.RST, UC0.PA1/ADC1
- removed net RST2: S02.RST, UC0.PA2/ADC2
- removed net RST3: S03.RST, UC0.PA3/ADC3
- removed net RST4: PROG.1, S04.RST, UC0.PA5/MISO
- new net CAP10: C1.P$1, S10.CAP
- new net CAP20: C2.P$1, S20.CAP
- new net CAP30: C3.P$1, S30.CAP
- new net CAP40: C4.P$1, S40.CAP
- new net RST10: S10.RST, UC0.PA1/ADC1
- new net RST20: S20.RST, UC0.PA2/ADC2
- new net RST30: S30.RST, UC0.PA3/ADC3
- new net RST40: PROG.1, S40.RST, UC0.PA5/MISO
- net 3.3V: now also S10.SHDN, S10.VDD, S20.SHDN, S20.VDD, S30.SHDN, S30.VDD, S40.SHDN, S40.VDD; no longer OUT.2, S01.SHDN, S01.VDD, S02.SHDN, S02.VDD, S03.SHDN, S03.VDD, S04.SHDN, S04.VDD
- net GND: now also S10.GND, S20.GND, S30.GND, S40.GND, UC0.PA7/ADC7, UC0.PB1, UC0.PB2; no longer OUT.4, S01.GND, S02.GND, S03.GND, S04.GND
- net SCL: now also S10.SCL, S20.SCL, S30.SCL, S40.SCL; no longer OUT.3, S01.SCL, S02.SCL, S03.SCL, S04.SCL
- net SDA: now also S10.SDA, S20.SDA, S30.SDA, S40.SDA; no longer OUT.1, S01.SDA, S02.SDA, S03.SDA, S04.SDA
Other:
- moved on the sheet: C0, C1, C2, C3, C4, PROG, S00, UC0
