File: eagle/row.brd (EAGLE design)
At the start: 39.8 x 6 mm, 12 parts

Commit message: .8mm hole added
Parts:
- moved UC0 0.51 mm to (13.3, 2.99)
- moved C2 0.13 mm to (17.0, 2.62)
- moved C3 0.13 mm to (18.7, 2.46)
Routing:
- net RST20: track 5.77 -> 8.19 mm
- net RST10: track 3.98 -> 5.91 mm
- net SDA: track 43.2 -> 44.8 mm, vias 3 -> 5
- net GND: track 48.0 -> 49.7 mm
- net SCL: track 50.5 -> 52.0 mm
- net 3.3V: track 63.4 -> 62.2 mm
- net RST30: track 9.76 -> 8.90 mm
- net RST00: track 16.6 -> 17.4 mm
- net RESET0: track 20.8 -> 20.3 mm

Commit message: board work.
Routing:
- net 3.3V: track 62.2 -> 63.2 mm
- net CAP40: track 1.81 -> 2.53 mm
- net GND: track 49.7 -> 49.0 mm
- net SDA: track 44.8 -> 45.5 mm
- net RST40: track 27.9 -> 28.4 mm
