File: eagle/tessellate.brd (EAGLE design)
At the start: 39.8 x 6 mm, 12 parts

Commit message: killed Dimension layer on the tessellateable board
Other:
- board outline removed
Changed lines of the file:
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@@
 <board>
 <plain>
-<wire x1="-0.5" y1="0" x2="39.271" y2="0" width="0" layer="20"/>
-<wire x1="39.271" y1="0" x2="39.271" y2="6" width="0" layer="20"/>
-<wire x1="39.271" y1="6" x2="-0.5" y2="6" width="0" layer="20"/>
-<wire x1="-0.5" y1="6" x2="-0.5" y2="0" width="0" layer="20"/>
 <hole x="10.668" y="4.699" drill="0.8"/>
 <wire x1="22.479" y1="5.588" x2="22.479" y2="0.381" width="0.254" layer="21" style="shortdash"/>

Commit message: reworked silkscreen and snap on tesselate.brd
Parts:
- renumbered PROG to PROG0
Routing:
- net 3.3V: track 65.0 -> 65.9 mm
- net SCL: track 54.4 -> 53.7 mm
- removed copper zone on layer 1, net GND
- removed copper zone on layer 16, net GND
