File: eagle/tessellate.brd (EAGLE design)
At the start: 12 parts

Commit message: start of repeatable / chainable rows w/ 7mm spacing and no vias under qfn tiny
Parts:
- added C5: (no value), nonolith:0402
- C0, C1, C2, C3, C4: device nonolith:0603 -> nonolith:0402
- moved C3 0.40 mm to (18.8, 2.84)
- moved C1 0.25 mm to (7.18, 3.10)
Connections:
- net 3.3V: now also C5.1
- net GND: now also C5.2
Routing:
- net GND: track 62.9 -> 59.6 mm
- net 3.3V: track 65.9 -> 67.2 mm
- net CAP30: track 2.12 -> 1.33 mm
- net CAP20: track 2.59 -> 3.30 mm
- net CAP10: track 1.52 -> 0.99 mm
- net CAP40: track 1.73 -> 2.23 mm

Commit message: major rework of tesselate file - needs a tiny bit of tweaking for full tesselation
Parts:
- removed PROG0: (no value), nonolith:2X03
- renumbered S00 to 0, S10 to 1, S20 to 2, S30 to 3, S40 to 4
Connections:
- net 3.3V: no longer PROG0.2
- net GND: no longer PROG0.6
- net RESET0: no longer PROG0.5
- net RST40: no longer PROG0.1
- net SCL: no longer PROG0.3
- net SDA: no longer PROG0.4
Routing:
- net RESET0: track 20.6 -> 0.00 mm
- net RST40: track 27.7 -> 12.8 mm, vias 2 -> 1
- net SCL: track 53.7 -> 43.8 mm, vias 8 -> 7
- net SDA: track 53.1 -> 43.3 mm, vias 7 -> 5
- net 3.3V: track 67.2 -> 59.7 mm, vias 6 -> 8
- net GND: track 59.6 -> 53.2 mm, vias 10 -> 6
- net CAP40: track 2.23 -> 3.21 mm
- net CAP30: track 1.33 -> 0.57 mm
- net RST00: track 18.0 -> 17.2 mm

Commit message: add 7mm center-to-center ground pour on bottom
Routing:
- net GND: track 53.2 -> 43.6 mm
- added copper zone on layer 16, net GND
Changed lines of the file:
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@@
 <wire x1="27.2" y1="2.375" x2="26.73" y2="2.413" width="0.254" layer="1"/>
 <wire x1="26.73" y1="2.413" x2="26.73" y2="2.48" width="0.254" layer="1"/>
-<wire x1="26.73" y1="2.48" x2="27.686" y2="2.413" width="0.254" layer="1"/>
-<via x="27.686" y="2.413" extent="1-16" drill="0.305" shape="octagon"/>
+<wire x1="26.73" y1="2.48" x2="27.432" y2="2.413" width="0.254" layer="1"/>
+<via x="27.432" y="2.413" extent="1-16" drill="0.305" shape="octagon"/>
 <wire x1="26" y1="2.35" x2="27.622" y2="2.35" width="0.254" layer="16"/>
-<wire x1="27.622" y1="2.35" x2="27.686" y2="2.413" width="0.254" layer="16"/>
+<wire x1="27.622" y1="2.35" x2="27.432" y2="2.413" width="0.254" layer="16"/>
 </signal>
 <signal name="GND">
@@
 <wire x1="7.5565" y1="2.3775" x2="7.4295" y2="2.3495" width="0.254" layer="16"/>
 <wire x1="6.8" y1="2.375" x2="6.477" y2="2.444" width="0.254" layer="1"/>
-<via x="27.686" y="3.683" extent="1-16" drill="0.305" shape="octagon"/>
+<via x="27.432" y="3.683" extent="1-16" drill="0.305" shape="octagon"/>
 <wire x1="18.161" y1="2.375" x2="18.161" y2="2.413" width="0.254" layer="1"/>
 <wire x1="23.622" y1="3.683" x2="25.833" y2="3.683" width="0.254" layer="16"/>
 <wire x1="25.833" y1="3.683" x2="26" y2="3.65" width="0.254" layer="16"/>
-<wire x1="27.686" y1="3.683" x2="26.162" y2="3.683" width="0.254" layer="16"/>
+<wire x1="27.432" y1="3.683" x2="26.162" y2="3.683" width="0.254" layer="16"/>
 <wire x1="26.162" y1="3.683" x2="26.035" y2="3.81" width="0.254" layer="16"/>
 <wire x1="26.035" y1="3.81" x2="26.035" y2="3.815" width="0.254" layer="16"/>
@@
 <wire x1="12.787" y1="4.358" x2="12.787" y2="4.886" width="0.254" layer="16"/>
 <wire x1="12.787" y1="5.675" x2="13.208" y2="6.096" width="0.254" layer="16"/>
-<wire x1="15.621" y1="6.477" x2="21.209" y2="6.477" width="0.254" layer="16"/>
-<wire x1="21.209" y1="6.477" x2="21.463" y2="6.731" width="0.254" layer="16"/>
-<wire x1="21.463" y1="6.731" x2="21.463" y2="8.382" width="0.254" layer="16"/>
 <via x="5.461" y="2.54" extent="1-16" drill="0.4" shape="octagon" alwaysstop="yes"/>
 <wire x1="5.461" y1="2.54" x2="5.334" y2="2.413" width="0.254" layer="16"/>
@@
 <wire x1="13.479" y1="2.794" x2="13.287" y2="2.986" width="0.254" layer="16"/>
 <wire x1="15.367" y1="3.556" x2="17.018" y2="3.556" width="0.254" layer="1"/>
-<wire x1="15.621" y1="6.477" x2="14.287" y2="5.143" width="0.254" layer="16"/>
 <wire x1="14.287" y1="5.143" x2="14.287" y2="4.886" width="0.254" layer="16"/>
-<wire x1="27.686" y1="3.683" x2="27.617" y2="3.625" width="0.254" layer="1"/>
+<wire x1="27.432" y1="3.683" x2="27.617" y2="3.625" width="0.254" layer="1"/>
 <wire x1="27.617" y1="3.625" x2="27.2" y2="3.625" width="0.254" layer="1"/>
 <wire x1="19.13" y1="1.905" x2="21.844" y2="1.905" width="0.254" layer="16"/>
@@
 <wire x1="17.018" y1="3.28" x2="17.007" y2="3.269" width="0.254" layer="16"/>
 <wire x1="11.387" y1="2.986" x2="13.287" y2="2.986" width="0.254" layer="16"/>
+<polygon width="0.254" layer="16">
+<vertex x="0" y="6.5"/>
+<vertex x="0" y="-0.5"/>
+<vertex x="28.067" y="-0.5"/>
+<vertex x="28.067" y="6.5"/>
+</polygon>
 </signal>
 <signal name="3.3V">

Commit message: should tesselate now. I am excite.
Routing:
- net SDA: track 43.3 -> 43.8 mm
- net SCL: track 43.8 -> 44.3 mm
- net 3.3V: track 59.7 -> 60.2 mm
Changed lines of the file:
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@@
 <wire x1="6.477" y1="4.953" x2="6.477" y2="5.588" width="0.254" layer="1"/>
 <via x="6.477" y="5.588" extent="1-16" drill="0.305" shape="octagon"/>
-<wire x1="6.477" y1="5.588" x2="6.477" y2="6.731" width="0.254" layer="16"/>
-<wire x1="6.477" y1="6.731" x2="6.096" y2="7.143" width="0.254" layer="16"/>
+<wire x1="6.477" y1="5.588" x2="6.477" y2="7.231" width="0.254" layer="16"/>
+<wire x1="6.477" y1="7.231" x2="6.096" y2="7.643" width="0.254" layer="16"/>
 <wire x1="6.8" y1="4.875" x2="6.555" y2="4.875" width="0.254" layer="1"/>
 <wire x1="6.555" y1="4.875" x2="6.477" y2="4.953" width="0.254" layer="1"/>
@@
 <wire x1="11.8745" y1="1.7145" x2="10.1346" y2="1.7145" width="0.254" layer="1"/>
 <wire x1="22.098" y1="3.048" x2="22.098" y2="1.016" width="0.254" layer="1"/>
-<wire x1="22.098" y1="7.747" x2="22.098" y2="6.477" width="0.254" layer="1"/>
+<wire x1="22.098" y1="8.247" x2="22.098" y2="6.477" width="0.254" layer="1"/>
 <wire x1="22.098" y1="6.477" x2="21.59" y2="5.969" width="0.254" layer="1"/>
 <wire x1="21.59" y1="5.969" x2="18.034" y2="5.969" width="0.254" layer="1"/>
@@
 <via x="7.874" y="0.635" extent="1-16" drill="0.305" shape="octagon"/>
 <wire x1="7.874" y1="0.635" x2="7.874" y2="0.381" width="0.254" layer="16"/>
-<wire x1="8.255" y1="4.826" x2="8.255" y2="6.096" width="0.254" layer="16"/>
-<wire x1="8.255" y1="6.096" x2="7.874" y2="6.477" width="0.254" layer="16"/>
+<wire x1="8.255" y1="4.826" x2="8.255" y2="6.596" width="0.254" layer="16"/>
+<wire x1="8.255" y1="6.596" x2="7.874" y2="6.977" width="0.254" layer="16"/>
 <wire x1="8.255" y1="4.826" x2="9.151" y2="4.826" width="0.254" layer="1"/>
 <wire x1="9.151" y1="4.826" x2="9.2" y2="4.875" width="0.254" layer="1"/>

Commit message: one index sensors
Parts:
- removed 0: MPL115A, nonolith:LGA-8
- added 5: MPL115A, nonolith:LGA-8
- moved 1 6.00 mm to (2.00, 3.00), turned to 180 degrees
- moved 2 6.00 mm to (8.00, 3.00), turned to 0 degrees
- moved 3 6.00 mm to (14.0, 3.00), turned to 180 degrees
- moved 4 6.00 mm to (20.0, 3.00), turned to 0 degrees
Connections:
- net 3.3V: now also 5.1, 5.4; no longer 0.1, 0.4
- net CAP00: now also 1.2; no longer 0.2
- net CAP10: now also 2.2; no longer 1.2
- net CAP20: now also 3.2; no longer 2.2
- net CAP30: now also 4.2; no longer 3.2
- net CAP40: now also 5.2; no longer 4.2
- net GND: now also 5.3; no longer 0.3
- net RST00: now also 1.5; no longer 0.5
- net RST10: now also 2.5; no longer 1.5
- net RST20: now also 3.5; no longer 2.5
- net RST30: now also 4.5; no longer 3.5
- net RST40: now also 5.5; no longer 4.5
- net SCL: now also 5.8; no longer 0.8
- net SDA: now also 5.7; no longer 0.7
Routing:
- net GND: vias 6 -> 9
- added copper zone on layer 1, net GND
Changed lines of the file:
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@@
 <elements>
 <element name="UC0" library="nonolith" package="QFN20" value="ATTINY24QFN" x="13.287" y="2.986" rot="MR90"/>
-<element name="0" library="nonolith" package="LGA-8" value="MPL115A" x="2" y="3" smashed="yes" rot="R180">
+<element name="1" library="nonolith" package="LGA-8" value="MPL115A" x="2" y="3" smashed="yes" rot="R180">
 <attribute name="NAME" x="0.984" y="-0.5" size="0.75" layer="25" font="vector"/>
 </element>
-<element name="1" library="nonolith" package="LGA-8" value="MPL115A" x="8" y="3" smashed="yes">
+<element name="2" library="nonolith" package="LGA-8" value="MPL115A" x="8" y="3" smashed="yes">
 <attribute name="NAME" x="7.238" y="-0.5" size="0.75" layer="25" font="vector"/>
 </element>
-<element name="2" library="nonolith" package="LGA-8" value="MPL115A" x="14" y="3" smashed="yes" rot="R180">
+<element name="3" library="nonolith" package="LGA-8" value="MPL115A" x="14" y="3" smashed="yes" rot="R180">
 <attribute name="NAME" x="12.984" y="-0.373" size="0.75" layer="25" font="vector"/>
 </element>
@@
 <element name="C1" library="nonolith" package="0402" value="" x="7.18" y="3.096" smashed="yes" rot="MR270"/>
 <element name="C2" library="nonolith" package="0402" value="" x="17.007" y="2.619" smashed="yes" rot="MR90"/>
-<element name="3" library="nonolith" package="LGA-8" value="MPL115A" x="20" y="3" smashed="yes">
+<element name="4" library="nonolith" package="LGA-8" value="MPL115A" x="20" y="3" smashed="yes">
 <attribute name="NAME" x="19.238" y="-0.5" size="0.75" layer="25" font="vector"/>
 </element>
-<element name="4" library="nonolith" package="LGA-8" value="MPL115A" x="26" y="3" smashed="yes" rot="R180">
+<element name="5" library="nonolith" package="LGA-8" value="MPL115A" x="26" y="3" smashed="yes" rot="R180">
 <attribute name="NAME" x="25.111" y="-0.5" size="0.75" layer="25" font="vector"/>
 </element>
@@
 <signal name="CAP20">
 <contactref element="C2" pad="1"/>
-<contactref element="2" pad="2"/>
+<contactref element="3" pad="2"/>
 <wire x1="16.755" y1="2.023" x2="17.018" y2="1.778" width="0.254" layer="16"/>
 <via x="17.018" y="1.778" extent="1-16" drill="0.305" shape="octagon"/>
@@
 </signal>
 <signal name="CAP30">
-<contactref element="3" pad="2"/>
+<contactref element="4" pad="2"/>
 <contactref element="C3" pad="1"/>
 <via x="18.796" y="3.429" extent="1-16" drill="0.305" shape="octagon"/>
@@
 <signal name="CAP40">
 <contactref element="C4" pad="1"/>
-<contactref element="4" pad="2"/>
+<contactref element="5" pad="2"/>
 <wire x1="27.2" y1="2.375" x2="26.73" y2="2.413" width="0.254" layer="1"/>
 <wire x1="26.73" y1="2.413" x2="26.73" y2="2.48" width="0.254" layer="1"/>
@@
 <contactref element="UC0" pad="8"/>
 <contactref element="UC0" pad="0"/>
+<contactref element="2" pad="3"/>
+<contactref element="C1" pad="2"/>
+<contactref element="3" pad="3"/>
+<contactref element="C2" pad="2"/>
+<contactref element="4" pad="3"/>
+<contactref element="C3" pad="2"/>
+<contactref element="5" pad="3"/>
+<contactref element="C4" pad="2"/>
 <contactref element="1" pad="3"/>
-<contactref element="C1" pad="2"/>
-<contactref element="2" pad="3"/>
-<contactref element="C2" pad="2"/>
-<contactref element="3" pad="3"/>
-<contactref element="C3" pad="2"/>
-<contactref element="4" pad="3"/>
-<contactref element="C4" pad="2"/>
-<contactref element="0" pad="3"/>
 <contactref element="C0" pad="2"/>
 <contactref element="UC0" pad="15"/>
@@
 <vertex x="28.067" y="6.5"/>
 </polygon>
+<polygon width="0.254" layer="1">
+<vertex x="0.008" y="6.5"/>
+<vertex x="0" y="-0.5"/>
+<vertex x="28" y="-0.5"/>
+<vertex x="28" y="6.5"/>
+</polygon>
+<via x="2.54" y="-0.127" extent="1-16" drill="0.305" shape="octagon"/>
+<via x="23.241" y="0" extent="1-16" drill="0.305" shape="octagon"/>
+<via x="22.987" y="1.905" extent="1-16" drill="0.305" shape="octagon"/>
 </signal>
 <signal name="3.3V">
+<contactref element="2" pad="1"/>
 <contactref element="1" pad="1"/>
-<contactref element="0" pad="1"/>
-<contactref element="2" pad="1"/>
 <contactref element="3" pad="1"/>
 <contactref element="4" pad="1"/>
+<contactref element="5" pad="1"/>
 <contactref element="UC0" pad="9"/>
-<contactref element="1" pad="4"/>
 <contactref element="2" pad="4"/>
 <contactref element="3" pad="4"/>
 <contactref element="4" pad="4"/>
-<contactref element="0" pad="4"/>
+<contactref element="5" pad="4"/>
+<contactref element="1" pad="4"/>
 <wire x1="15.2" y1="4.875" x2="15.572" y2="4.875" width="0.254" layer="1"/>
 <wire x1="18.415" y1="4.826" x2="18.8" y2="4.875" width="0.254" layer="1"/>
@@
 <signal name="CAP00">
 <contactref element="C0" pad="1"/>
-<contactref element="0" pad="2"/>
+<contactref element="1" pad="2"/>
 <wire x1="2" y1="2.35" x2="2.032" y2="2.118" width="0.254" layer="16"/>
 <wire x1="2.032" y1="2.118" x2="2.032" y2="1.905" width="0.254" layer="16"/>
@@
 </signal>
 <signal name="SDA">
-<contactref element="0" pad="7"/>
+<contactref element="1" pad="7"/>
+<contactref element="5" pad="7"/>
 <contactref element="4" pad="7"/>
 <contactref element="3" pad="7"/>
 <contactref element="2" pad="7"/>
-<contactref element="1" pad="7"/>
 <contactref element="UC0" pad="16"/>
 <wire x1="0.8" y1="2.375" x2="1.143" y2="2.413" width="0.254" layer="1"/>
@@
 <signal name="SCL">
 <contactref element="UC0" pad="1"/>
-<contactref element="0" pad="8"/>
+<contactref element="1" pad="8"/>
+<contactref element="5" pad="8"/>
 <contactref element="4" pad="8"/>
 <contactref element="3" pad="8"/>
 <contactref element="2" pad="8"/>
-<contactref element="1" pad="8"/>
 <wire x1="0.8" y1="1.125" x2="0.8" y2="0.724" width="0.254" layer="1"/>
 <wire x1="0.8" y1="0.724" x2="1.016" y2="0.508" width="0.254" layer="1"/>
@@
 <signal name="RST00">
 <contactref element="UC0" pad="5"/>
-<contactref element="0" pad="5"/>
+<contactref element="1" pad="5"/>
 <wire x1="0.8" y1="4.875" x2="1.094" y2="4.875" width="0.254" layer="1"/>
 <wire x1="1.094" y1="4.875" x2="1.143" y2="4.826" width="0.254" layer="1"/>
@@
 <signal name="RST10">
 <contactref element="UC0" pad="4"/>
-<contactref element="1" pad="5"/>
+<contactref element="2" pad="5"/>
 <wire x1="12.787" y1="1.086" x2="12.787" y2="0.595" width="0.254" layer="16"/>
 <wire x1="12.787" y1="0.595" x2="12.573" y2="0.381" width="0.254" layer="16"/>
@@
 <signal name="RST20">
 <contactref element="UC0" pad="3"/>
-<contactref element="2" pad="5"/>
+<contactref element="3" pad="5"/>
 <wire x1="13.287" y1="1.086" x2="13.287" y2="1.572" width="0.254" layer="16"/>
 <wire x1="13.287" y1="1.572" x2="13.081" y2="1.778" width="0.254" layer="16"/>
@@
 <signal name="RST30">
 <contactref element="UC0" pad="2"/>
-<contactref element="3" pad="5"/>
+<contactref element="4" pad="5"/>
 <wire x1="21.2" y1="1.125" x2="20.837" y2="1.143" width="0.254" layer="1"/>
 <wire x1="13.787" y1="1.086" x2="13.787" y2="0.564" width="0.254" layer="16"/>
@@
 <signal name="CAP10">
 <contactref element="C1" pad="1"/>
-<contactref element="1" pad="2"/>
+<contactref element="2" pad="2"/>
 <wire x1="6.8" y1="3.625" x2="6.731" y2="3.556" width="0.254" layer="1"/>
 <wire x1="6.8" y1="3.625" x2="7.297" y2="3.625" width="0.254" layer="1"/>
@@
 <signal name="RST40">
 <contactref element="UC0" pad="20"/>
-<contactref element="4" pad="5"/>
+<contactref element="5" pad="5"/>
 <wire x1="15.187" y1="1.986" x2="15.829" y2="1.986" width="0.254" layer="16"/>
 <wire x1="15.829" y1="1.986" x2="16.002" y2="2.159" width="0.254" layer="16"/>
