File: eagle/tessellate.brd (EAGLE design)
At the start: 12 parts

Commit message: add via for continuous ground pour
Routing:
- net GND: track 43.6 -> 42.2 mm, vias 9 -> 10
Changed lines of the file:
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@@
 <wire x1="8.509" y1="2.286" x2="7.493" y2="2.286" width="0.254" layer="16"/>
 <wire x1="12.787" y1="4.358" x2="12.787" y2="4.886" width="0.254" layer="16"/>
-<wire x1="12.787" y1="5.675" x2="13.208" y2="6.096" width="0.254" layer="16"/>
 <via x="5.461" y="2.54" extent="1-16" drill="0.4" shape="octagon" alwaysstop="yes"/>
 <wire x1="5.461" y1="2.54" x2="5.334" y2="2.413" width="0.254" layer="16"/>
@@
 <wire x1="2" y1="3.778" x2="2" y2="3.65" width="0.254" layer="16"/>
 <wire x1="17.018" y1="3.556" x2="18.161" y2="2.413" width="0.254" layer="1"/>
-<wire x1="12.787" y1="4.886" x2="12.787" y2="5.675" width="0.254" layer="16"/>
 <wire x1="2" y1="3.778" x2="3.143" y2="3.778" width="0.254" layer="16"/>
 <wire x1="3.143" y1="3.778" x2="3.175" y2="3.81" width="0.254" layer="16"/>
@@
 <via x="23.241" y="0" extent="1-16" drill="0.305" shape="octagon"/>
 <via x="22.987" y="1.905" extent="1-16" drill="0.305" shape="octagon"/>
+<via x="26.797" y="6.096" extent="1-16" drill="0.305" shape="octagon"/>
 </signal>
 <signal name="3.3V">

Commit message: 6mm row-row spacing, numbers at top of sensor, should be good to go for tesselation
Routing:
- net GND: track 42.2 -> 41.1 mm
- net 3.3V: track 60.2 -> 60.3 mm, vias 8 -> 7

Commit message: align traces for tessellation. hopefully the last modification needed to this board...
Routing:
- net SDA: track 43.6 -> 42.5 mm
- net 3.3V: track 60.3 -> 59.8 mm
Changed lines of the file:
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@@
 <wire x1="6.8" y1="4.875" x2="7.161" y2="4.875" width="0.254" layer="1"/>
 <wire x1="5.461" y1="4.953" x2="6.477" y2="4.953" width="0.254" layer="1"/>
-<wire x1="6.096" y1="5.588" x2="6.096" y2="7.643" width="0.254" layer="16"/>
+<wire x1="6.096" y1="5.588" x2="6.096" y2="7.143" width="0.254" layer="16"/>
 <wire x1="6.8" y1="4.875" x2="6.555" y2="4.875" width="0.254" layer="1"/>
 <wire x1="6.555" y1="4.875" x2="6.477" y2="4.953" width="0.254" layer="1"/>
@@
 <wire x1="11.8745" y1="1.7145" x2="10.14" y2="1.72" width="0.254" layer="1"/>
 <wire x1="22.098" y1="3.048" x2="22.098" y2="1.016" width="0.254" layer="1"/>
-<wire x1="22.098" y1="8.247" x2="22.098" y2="6.477" width="0.254" layer="1"/>
-<wire x1="22.098" y1="6.477" x2="21.59" y2="5.969" width="0.254" layer="1"/>
-<wire x1="21.59" y1="5.969" x2="18.288" y2="5.969" width="0.254" layer="1"/>
+<wire x1="22.098" y1="7.016" x2="22.098" y2="6.223" width="0.254" layer="1"/>
+<wire x1="21.844" y1="5.969" x2="18.288" y2="5.969" width="0.254" layer="1"/>
 <wire x1="17.145" y1="4.699" x2="20.701" y2="4.699" width="0.254" layer="16"/>
 <wire x1="22.098" y1="1.016" x2="23.622" y2="1.016" width="0.254" layer="1"/>
@@
 <wire x1="17.145" y1="4.826" x2="16.891" y2="4.826" width="0.254" layer="1"/>
 <wire x1="16.891" y1="4.826" x2="16.256" y2="4.191" width="0.254" layer="1"/>
+<wire x1="21.844" y1="5.969" x2="22.098" y2="6.223" width="0.254" layer="1"/>
 </signal>
 <signal name="SCL">
@@
 <wire x1="7.874" y1="0.635" x2="7.874" y2="0.381" width="0.254" layer="16"/>
 <wire x1="8.255" y1="4.826" x2="7.874" y2="5.207" width="0.254" layer="16"/>
-<wire x1="7.874" y1="5.207" x2="7.874" y2="6.596" width="0.254" layer="16"/>
-<wire x1="7.874" y1="6.596" x2="7.874" y2="6.977" width="0.254" layer="16"/>
+<wire x1="7.874" y1="5.207" x2="7.874" y2="6.635" width="0.254" layer="16"/>
 <wire x1="8.255" y1="4.826" x2="9.151" y2="4.826" width="0.254" layer="1"/>
 <wire x1="9.151" y1="4.826" x2="9.2" y2="4.875" width="0.254" layer="1"/>

Commit message: explicit ground connections, remove bothersome ground via
Routing:
- net GND: track 41.1 -> 43.9 mm, vias 10 -> 9
- removed copper zone on layer 1, net GND
- removed copper zone on layer 16, net GND
Changed lines of the file:
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@@
 <wire x1="17.018" y1="3.28" x2="17.007" y2="3.269" width="0.254" layer="16"/>
 <wire x1="11.387" y1="2.986" x2="13.287" y2="2.986" width="0.254" layer="16"/>
-<polygon width="0.254" layer="16">
-<vertex x="0" y="6"/>
-<vertex x="0" y="0"/>
-<vertex x="28.067" y="0"/>
-<vertex x="28.067" y="6"/>
-</polygon>
-<polygon width="0.254" layer="1">
-<vertex x="0.008" y="6"/>
-<vertex x="0" y="0"/>
-<vertex x="28" y="0"/>
-<vertex x="28" y="6"/>
-</polygon>
 <via x="23.114" y="0.381" extent="1-16" drill="0.305" shape="octagon"/>
 <via x="22.987" y="1.905" extent="1-16" drill="0.305" shape="octagon"/>
 <via x="26.416" y="5.6" extent="1-16" drill="0.305" shape="octagon"/>
-<via x="14.986" y="5.727" extent="1-16" drill="0.305" shape="octagon"/>
+<wire x1="21.844" y1="1.905" x2="22.987" y2="1.905" width="0.254" layer="16"/>
+<wire x1="22.987" y1="1.905" x2="23.114" y2="1.905" width="0.4064" layer="16"/>
+<wire x1="23.114" y1="1.905" x2="23.114" y2="0.381" width="0.254" layer="16"/>
+<wire x1="26.035" y1="3.81" x2="26.416" y2="5.6" width="0" layer="19" extent="16-16"/>
 </signal>
 <signal name="3.3V">
@@
 </signal>
 </signals>
-<errors>
-</errors>
 </board>
 </drawing>

Commit message: rename some signals and stuff
Parts:
- removed C0: (no value), nonolith:0402
- added C6: (no value), nonolith:0402
- moved C5 16.1 mm to (26.0, 3.00), turned to 90 degrees
- moved C2 9.84 mm to (7.18, 3.10), turned to 270 degrees
- moved C4 7.16 mm to (18.8, 2.84), turned to 270 degrees
- moved C1 5.18 mm to (2.00, 3.00), turned to 90 degrees
- moved C3 1.85 mm to (17.0, 2.62), turned to 90 degrees
- renumbered UC0 to UC1
Connections:
- net RESET0 renamed RESET1
- net RST00 renamed RST1
- net RST10 renamed RST2
- net RST20 renamed RST3
- net RST30 renamed RST4
- net RST40 renamed RST5
- net 3.3V: now also C6.1; no longer C5.1
- net CAP00: now also C1.1; no longer C0.1
- net CAP10: now also C2.1; no longer C1.1
- net CAP20: now also C3.1; no longer C2.1
- net CAP30: now also C4.1; no longer C3.1
- net CAP40: now also C5.1; no longer C4.1
- net GND: now also C6.2; no longer C0.2
Changed lines of the file:
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@@
 </autorouter>
 <elements>
-<element name="UC0" library="nonolith" package="QFN20" value="ATTINY24QFN" x="13.287" y="2.986" rot="MR90"/>
+<element name="UC1" library="nonolith" package="QFN20" value="ATTINY24QFN" x="13.287" y="2.986" rot="MR90"/>
 <element name="1" library="nonolith" package="LGA-8" value="MPL115A" x="2" y="3" smashed="yes" rot="R180">
 <attribute name="NAME" x="1.873" y="5.596" size="0.5" layer="25" font="vector" ratio="12"/>
@@
 <attribute name="NAME" x="13.94" y="5.636" size="0.5" layer="25" font="vector" ratio="12"/>
 </element>
-<element name="C0" library="nonolith" package="0402" value="" x="2" y="3" smashed="yes" rot="MR90"/>
-<element name="C1" library="nonolith" package="0402" value="" x="7.18" y="3.096" smashed="yes" rot="MR270"/>
-<element name="C2" library="nonolith" package="0402" value="" x="17.007" y="2.619" smashed="yes" rot="MR90"/>
+<element name="C1" library="nonolith" package="0402" value="" x="2" y="3" smashed="yes" rot="MR90"/>
+<element name="C2" library="nonolith" package="0402" value="" x="7.18" y="3.096" smashed="yes" rot="MR270"/>
+<element name="C3" library="nonolith" package="0402" value="" x="17.007" y="2.619" smashed="yes" rot="MR90"/>
 <element name="4" library="nonolith" package="LGA-8" value="MPL115A" x="20" y="3" smashed="yes">
 <attribute name="NAME" x="20" y="5.667" size="0.5" layer="25" font="vector" ratio="12"/>
@@
 <attribute name="NAME" x="25.943" y="5.636" size="0.5" layer="25" font="vector" ratio="12"/>
 </element>
-<element name="C3" library="nonolith" package="0402" value="" x="18.843" y="2.842" smashed="yes" rot="MR270"/>
-<element name="C4" library="nonolith" package="0402" value="" x="26" y="3" smashed="yes" rot="MR90"/>
-<element name="C5" library="nonolith" package="0402" value="" x="10.033" y="4.826" rot="MR0"/>
+<element name="C4" library="nonolith" package="0402" value="" x="18.843" y="2.842" smashed="yes" rot="MR270"/>
+<element name="C5" library="nonolith" package="0402" value="" x="26" y="3" smashed="yes" rot="MR90"/>
+<element name="C6" library="nonolith" package="0402" value="" x="10.033" y="4.826" rot="MR0"/>
 </elements>
 <signals>
 <signal name="CAP20">
-<contactref element="C2" pad="1"/>
+<contactref element="C3" pad="1"/>
 <contactref element="3" pad="2"/>
 <wire x1="16.755" y1="2.023" x2="17.018" y2="1.778" width="0.254" layer="16"/>
@@
 <signal name="CAP30">
 <contactref element="4" pad="2"/>
-<contactref element="C3" pad="1"/>
+<contactref element="C4" pad="1"/>
 <via x="18.796" y="3.429" extent="1-16" drill="0.305" shape="octagon"/>
 <wire x1="18.796" y1="3.629" x2="18.8" y2="3.625" width="0.254" layer="1"/>
@@
 </signal>
 <signal name="CAP40">
-<contactref element="C4" pad="1"/>
+<contactref element="C5" pad="1"/>
 <contactref element="5" pad="2"/>
 <wire x1="27.2" y1="2.375" x2="26.73" y2="2.413" width="0.254" layer="1"/>
@@
 </signal>
 <signal name="GND">
-<contactref element="UC0" pad="8"/>
-<contactref element="UC0" pad="0"/>
+<contactref element="UC1" pad="8"/>
+<contactref element="UC1" pad="0"/>
 <contactref element="2" pad="3"/>
+<contactref element="C2" pad="2"/>
+<contactref element="3" pad="3"/>
+<contactref element="C3" pad="2"/>
+<contactref element="4" pad="3"/>
+<contactref element="C4" pad="2"/>
+<contactref element="5" pad="3"/>
+<contactref element="C5" pad="2"/>
+<contactref element="1" pad="3"/>
 <contactref element="C1" pad="2"/>
-<contactref element="3" pad="3"/>
-<contactref element="C2" pad="2"/>
-<contactref element="4" pad="3"/>
-<contactref element="C3" pad="2"/>
-<contactref element="5" pad="3"/>
-<contactref element="C4" pad="2"/>
-<contactref element="1" pad="3"/>
-<contactref element="C0" pad="2"/>
-<contactref element="UC0" pad="15"/>
-<contactref element="UC0" pad="12"/>
-<contactref element="UC0" pad="14"/>
+<contactref element="UC1" pad="15"/>
+<contactref element="UC1" pad="12"/>
+<contactref element="UC1" pad="14"/>
 <wire x1="14.287" y1="4.886" x2="13.787" y2="4.886" width="0.254" layer="16"/>
 <wire x1="15.2" y1="3.625" x2="15.258" y2="3.683" width="0.254" layer="1"/>
@@
 <wire x1="7.366" y1="2.413" x2="5.461" y2="2.413" width="0.254" layer="16"/>
 <wire x1="5.461" y1="2.413" x2="5.461" y2="2.54" width="0.254" layer="16"/>
-<contactref element="C5" pad="2"/>
+<contactref element="C6" pad="2"/>
 <wire x1="9.383" y1="4.826" x2="9.144" y2="4.826" width="0.2032" layer="16"/>
 <wire x1="9.144" y1="4.826" x2="9.144" y2="4.064" width="0.2032" layer="16"/>
@@
 <contactref element="4" pad="1"/>
 <contactref element="5" pad="1"/>
-<contactref element="UC0" pad="9"/>
+<contactref element="UC1" pad="9"/>
 <contactref element="2" pad="4"/>
 <contactref element="3" pad="4"/>
@@
 <wire x1="5.08" y1="4.953" x2="5.461" y2="4.953" width="0.254" layer="16"/>
 <wire x1="27.698" y1="1.125" x2="27.2" y2="1.125" width="0.254" layer="1"/>
-<contactref element="C5" pad="1"/>
+<contactref element="C6" pad="1"/>
 <wire x1="10.683" y1="4.826" x2="11.557" y2="4.826" width="0.2032" layer="16"/>
 <wire x1="11.557" y1="4.826" x2="11.557" y2="5.588" width="0.2032" layer="16"/>
@@
 </signal>
 <signal name="CAP00">
-<contactref element="C0" pad="1"/>
+<contactref element="C1" pad="1"/>
 <contactref element="1" pad="2"/>
 <wire x1="2" y1="2.35" x2="2.032" y2="2.118" width="0.254" layer="16"/>
@@
 <contactref element="3" pad="7"/>
 <contactref element="2" pad="7"/>
-<contactref element="UC0" pad="16"/>
+<contactref element="UC1" pad="16"/>
 <wire x1="0.8" y1="2.375" x2="1.143" y2="2.413" width="0.254" layer="1"/>
 <wire x1="1.143" y1="2.413" x2="1.651" y2="2.413" width="0.254" layer="1"/>
@@
 </signal>
 <signal name="SCL">
-<contactref element="UC0" pad="1"/>
+<contactref element="UC1" pad="1"/>
 <contactref element="1" pad="8"/>
 <contactref element="5" pad="8"/>
@@
 <wire x1="24.384" y1="2.032" x2="24.384" y2="1.143" width="0.254" layer="16"/>
 </signal>
-<signal name="RST00">
-<contactref element="UC0" pad="5"/>
+<signal name="RST1">
+<contactref element="UC1" pad="5"/>
 <contactref element="1" pad="5"/>
 <wire x1="0.8" y1="4.875" x2="1.094" y2="4.875" width="0.254" layer="1"/>
@@
 <wire x1="3.81" y1="1.778" x2="6.35" y2="1.778" width="0.254" layer="16"/>
 </signal>
-<signal name="RST10">
-<contactref element="UC0" pad="4"/>
+<signal name="RST2">
+<contactref element="UC1" pad="4"/>
 <contactref element="2" pad="5"/>
 <wire x1="12.787" y1="1.086" x2="12.787" y2="0.595" width="0.254" layer="16"/>
@@
 <wire x1="9.218" y1="1.143" x2="9.2" y2="1.125" width="0.254" layer="1"/>
 </signal>
-<signal name="RST20">
-<contactref element="UC0" pad="3"/>
+<signal name="RST3">
+<contactref element="UC1" pad="3"/>
 <contactref element="3" pad="5"/>
 <wire x1="13.287" y1="1.086" x2="13.287" y2="1.572" width="0.254" layer="16"/>
@@
 <wire x1="10.75" y1="2.413" x2="10.75" y2="1.397" width="0.254" layer="16"/>
 </signal>
-<signal name="RST30">
-<contactref element="UC0" pad="2"/>
+<signal name="RST4">
+<contactref element="UC1" pad="2"/>
 <contactref element="4" pad="5"/>
 <wire x1="21.2" y1="1.125" x2="20.837" y2="1.143" width="0.254" layer="1"/>
@@
 </signal>
 <signal name="CAP10">
-<contactref element="C1" pad="1"/>
+<contactref element="C2" pad="1"/>
 <contactref element="2" pad="2"/>
 <wire x1="6.8" y1="3.625" x2="6.731" y2="3.556" width="0.254" layer="1"/>
@@
 <wire x1="7.18" y1="3.742" x2="7.239" y2="3.556" width="0.254" layer="16"/>
 </signal>
-<signal name="RESET0">
-<contactref element="UC0" pad="13"/>
-</signal>
-<signal name="RST40">
-<contactref element="UC0" pad="20"/>
+<signal name="RESET1">
+<contactref element="UC1" pad="13"/>
+</signal>
+<signal name="RST5">
+<contactref element="UC1" pad="20"/>
 <contactref element="5" pad="5"/>
 <wire x1="15.187" y1="1.986" x2="15.829" y2="1.986" width="0.254" layer="16"/>
@@
 </signal>
 <signal name="ADDR00">
-<contactref element="UC0" pad="11"/>
+<contactref element="UC1" pad="11"/>
 </signal>
 </signals>

Commit message: fix numbering scheme for tesselation
Parts:
- renumbered 1 to 01, 2 to 02, 3 to 03, 4 to 04, 5 to 05, C1 to C01, C2 to C02, C3 to C03, C4 to C04, C5 to C05, UC1 to UC01
Connections:
- net CAP00 renamed CAP01
- net CAP10 renamed CAP02
- net CAP20 renamed CAP03
- net CAP30 renamed CAP04
- net CAP40 renamed CAP05
- net RESET1 renamed RESET01
- net RST1 renamed RST01
- net RST2 renamed RST02
- net RST3 renamed RST03
- net RST4 renamed RST04
- net RST5 renamed RST05
