File: eagle/fullArray.brd (EAGLE design)
At the start: 69 parts

Commit message: full 8 rows with standardized naming
Parts:
- removed PROG0: (no value), nonolith:2X03
- added (5,1), (5,2), (5,3), (5,4), (5,5), (6,1), (6,2), (6,3), (6,4), (6,5), (7,1), (7,2), (7,3), (7,4), (7,5), (8,1), (8,2), (8,3), (8,4), (8,5): MPL115A, nonolith:LGA-8
- added AT5, AT6, AT7, AT8: ATTINY24QFN, nonolith:QFN20
- added C23, C24, C25, C26, C27, C28, C29, C30, C31, C32, C33, C34, C35, C36, C37, C38, C39, C40, C41, C42: (no value), nonolith:0603
- added PROG4, PROG5, PROG6, PROG7, PROG8: (no value), nonolith:2X03
- moved PROG1 6.00 mm to (15.5, 18.5)
- moved PROG2 6.00 mm to (15.5, 24.5)
- moved PROG3 6.00 mm to (15.5, 30.5)
- renumbered S00 to (1,1), S01 to (2,1), S02 to (2,2), S03 to (2,3), S04 to (2,4), S05 to (2,5), S06 to (3,1), S07 to (3,2), S08 to (3,3), S09 to (3,4), S10 to (1,2), S11 to (3,5), S12 to (4,1), S13 to (4,2), S14 to (4,3), S15 to (4,4), S16 to (4,5), S20 to (1,3), S30 to (1,4), S40 to (1,5), UC0 to AT1, UC1 to AT2, UC2 to AT3, UC3 to AT4
Connections:
- net RST03 renamed RST14
- removed net RST00: (1,1).5, AT1.5
- removed net RST01: (2,1).5, AT2.5
- removed net RST02: (3,1).5, AT3.5
- removed net RST10: (1,2).5, AT1.4
- removed net RST20: (1,3).5, AT1.3
- removed net RST30: (1,4).5, AT1.2
- removed net RST40: (1,5).5, AT1.20, PROG0.1
- new net ADDR04: AT5.11
- new net ADDR05: AT6.11
- new net ADDR06: AT7.11
- new net ADDR07: AT8.11
- new net CAP17: (5,3).2, C25.1
- new net CAP18: (5,4).2, C26.1
- new net CAP19: (5,5).2, C27.1
- new net CAP21: (5,1).2, C23.1
- new net CAP22: (5,2).2, C24.1
- new net CAP23: (6,3).2, C30.1
- new net CAP24: (6,4).2, C31.1
- new net CAP25: (6,5).2, C32.1
- new net CAP26: (6,1).2, C28.1
- new net CAP27: (6,2).2, C29.1
- new net CAP28: (7,3).2, C35.1
- new net CAP29: (7,4).2, C36.1
- new net CAP31: (7,5).2, C37.1
- new net CAP32: (7,1).2, C33.1
- new net CAP33: (7,2).2, C34.1
- new net CAP34: (8,3).2, C40.1
- new net CAP35: (8,4).2, C41.1
- new net CAP36: (8,5).2, C42.1
- new net CAP37: (8,1).2, C38.1
- new net CAP38: (8,2).2, C39.1
- new net RESET4: AT4.13, PROG4.5
- new net RESET5: AT5.13, PROG5.5
- new net RESET6: AT6.13, PROG6.5
- new net RESET7: AT7.13, PROG7.5
- new net RESET8: AT8.13, PROG8.5
- new net RST15: (5,1).5, AT5.5
- new net RST16: (6,1).5, AT6.5
- new net RST17: (7,1).5, AT7.5
- new net RST18: (8,1).5, AT8.5
- new net RST24: (4,2).5, AT4.4
- new net RST25: (5,2).5, AT5.4
- new net RST26: (6,2).5, AT6.4
- new net RST27: (7,2).5, AT7.4
- new net RST28: (8,2).5, AT8.4
- new net RST34: (4,3).5, AT4.3
- new net RST35: (5,3).5, AT5.3
- new net RST36: (6,3).5, AT6.3
- new net RST37: (7,3).5, AT7.3
- new net RST38: (8,3).5, AT8.3
- new net RST44: (4,4).5, AT4.2
- new net RST45: (5,4).5, AT5.2
- new net RST46: (6,4).5, AT6.2
- new net RST47: (7,4).5, AT7.2
- new net RST48: (8,4).5, AT8.2
- new net RST51: (1,5).5, AT1.20, PROG1.1
- new net RST52: (2,5).5, AT2.20, PROG2.1
- new net RST53: (3,5).5, AT3.20, PROG3.1
- new net RST54: (4,5).5, AT4.20, PROG4.1
- new net RST55: (5,5).5, AT5.20, PROG5.1
- new net RST56: (6,5).5, AT6.20, PROG6.1
- new net RST57: (7,5).5, AT7.20, PROG7.1
- new net RST58: (8,5).5, AT8.20, PROG8.1
- net 3.3V: now also (5,1).1, (5,1).4, (5,2).1, (5,2).4, (5,3).1, (5,3).4, (5,4).1, (5,4).4, (5,5).1, (5,5).4, (6,1).1, (6,1).4, (6,2).1, (6,2).4, (6,3).1, (6,3).4, (6,4).1, (6,4).4, (6,5).1, (6,5).4, (7,1).1, (7,1).4, (7,2).1, (7,2).4, (7,3).1, (7,3).4, (7,4).1, (7,4).4, (7,5).1, (7,5).4, (8,1).1, (8,1).4, (8,2).1, (8,2).4, (8,3).1, (8,3).4, (8,4).1, (8,4).4, (8,5).1, (8,5).4, AT5.9, AT6.9, AT7.9, AT8.9, PROG4.2, PROG5.2, PROG6.2, PROG7.2, PROG8.2; no longer PROG0.2
- net GND: now also (5,1).3, (5,2).3, (5,3).3, (5,4).3, (5,5).3, (6,1).3, (6,2).3, (6,3).3, (6,4).3, (6,5).3, (7,1).3, (7,2).3, (7,3).3, (7,4).3, (7,5).3, (8,1).3, (8,2).3, (8,3).3, (8,4).3, (8,5).3, AT5.0, AT5.12, AT5.14, AT5.15, AT5.8, AT6.0, AT6.12, AT6.14, AT6.15, AT6.8, AT7.0, AT7.12, AT7.14, AT7.15, AT7.8, AT8.0, AT8.12, AT8.14, AT8.15, AT8.8, C23.2, C24.2, C25.2, C26.2, C27.2, C28.2, C29.2, C30.2, C31.2, C32.2, C33.2, C34.2, C35.2, C36.2, C37.2, C38.2, C39.2, C40.2, C41.2, C42.2, PROG4.6, PROG5.6, PROG6.6, PROG7.6, PROG8.6; no longer PROG0.6
- net RESET0: no longer PROG0.5
- net RESET1: no longer AT2.13
- net RESET2: now also AT2.13; no longer AT3.13
- net RESET3: now also AT3.13; no longer AT4.13
- net RST11: now also (1,1).5, AT1.5; no longer (2,2).5, AT2.4
- net RST12: now also (2,1).5, AT2.5; no longer (3,2).5, AT3.4
- net RST13: now also (3,1).5, AT3.5; no longer (4,2).5, AT4.4
- net RST21: now also (1,2).5, AT1.4; no longer (2,3).5, AT2.3
- net RST22: now also (2,2).5, AT2.4; no longer (3,3).5, AT3.3
- net RST23: now also (3,2).5, AT3.4; no longer (4,3).5, AT4.3
- net RST31: now also (1,3).5, AT1.3; no longer (2,4).5, AT2.2
- net RST32: now also (2,3).5, AT2.3; no longer (3,4).5, AT3.2
- net RST33: now also (3,3).5, AT3.3; no longer (4,4).5, AT4.2
- net RST41: now also (1,4).5, AT1.2; no longer (2,5).5, AT2.20, PROG1.1
- net RST42: now also (2,4).5, AT2.2; no longer (3,5).5, AT3.20, PROG2.1
- net RST43: now also (3,4).5, AT3.2; no longer (4,5).5, AT4.20, PROG3.1
- net SCL: now also (5,1).8, (5,2).8, (5,3).8, (5,4).8, (5,5).8, (6,1).8, (6,2).8, (6,3).8, (6,4).8, (6,5).8, (7,1).8, (7,2).8, (7,3).8, (7,4).8, (7,5).8, (8,1).8, (8,2).8, (8,3).8, (8,4).8, (8,5).8, AT5.1, AT6.1, AT7.1, AT8.1, PROG4.3, PROG5.3, PROG6.3, PROG7.3, PROG8.3; no longer PROG0.3
- net SDA: now also (5,1).7, (5,2).7, (5,3).7, (5,4).7, (5,5).7, (6,1).7, (6,2).7, (6,3).7, (6,4).7, (6,5).7, (7,1).7, (7,2).7, (7,3).7, (7,4).7, (7,5).7, (8,1).7, (8,2).7, (8,3).7, (8,4).7, (8,5).7, AT5.16, AT6.16, AT7.16, AT8.16, PROG4.4, PROG5.4, PROG6.4, PROG7.4, PROG8.4; no longer PROG0.4
Routing:
- net 3.3V: track 340.6 -> 603.2 mm, vias 27 -> 50
- net GND: track 262.7 -> 503.1 mm, vias 40 -> 80
- net SCL: track 228.8 -> 441.8 mm, vias 33 -> 65
- net SDA: track 229.7 -> 432.2 mm, vias 28 -> 56
- net RST58: track 0.00 -> 27.8 mm, vias 0 -> 2
- net RST57: track 0.00 -> 27.8 mm, vias 0 -> 2
- net RST40: track 27.8 -> 0.00 mm, vias 2 -> 0
- net RST56: track 0.00 -> 27.8 mm, vias 0 -> 2
- net RST53: track 0.00 -> 27.8 mm, vias 0 -> 2
- net RST52: track 0.00 -> 27.8 mm, vias 0 -> 2
- net RST51: track 0.00 -> 27.8 mm, vias 0 -> 2
- net RST55: track 0.00 -> 27.1 mm, vias 0 -> 2
- net RST54: track 0.00 -> 27.1 mm, vias 0 -> 2
- net RESET1: track 20.6 -> 0.00 mm
- net RESET8: track 0.00 -> 20.6 mm
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- added copper zone on layer 16, net GND
Other:
- board outline added: 40 x 64 mm

Commit message: now with proper address pin configurations
Connections:
- net ADDR00 renamed ADDR1
- removed net ADDR01: AT2.11
- removed net ADDR02: AT3.11
- removed net ADDR03: AT4.11
- removed net ADDR04: AT5.11
- removed net ADDR05: AT6.11
- removed net ADDR06: AT7.11
- removed net ADDR07: AT8.11
- new net ADDR2: AT2.12
- new net ADDR3: AT3.11, AT3.12
- new net ADDR4: AT4.14
- new net ADDR5: AT5.11, AT5.14
- new net ADDR6: AT6.12, AT6.14
- new net ADDR7: AT7.11, AT7.12, AT7.14
- new net ADDR8: AT8.15
- net GND: now also AT2.11, AT4.11, AT6.11, AT8.11; no longer AT2.12, AT3.12, AT4.14, AT5.14, AT6.12, AT6.14, AT7.12, AT7.14, AT8.15
Routing:
- net GND: track 503.1 -> 500.0 mm
Changed lines of the file:
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@@
 <contactref element="C5" pad="2"/>
 <contactref element="AT2" pad="15"/>
-<contactref element="AT2" pad="12"/>
 <contactref element="AT2" pad="14"/>
 <wire x1="-5.213" y1="26.386" x2="-5.713" y2="26.386" width="0.254" layer="16"/>
@@
 <contactref element="C13" pad="2"/>
 <contactref element="AT3" pad="15"/>
-<contactref element="AT3" pad="12"/>
 <contactref element="AT3" pad="14"/>
 <wire x1="-5.213" y1="32.386" x2="-5.713" y2="32.386" width="0.254" layer="16"/>
@@
 <contactref element="AT4" pad="15"/>
 <contactref element="AT4" pad="12"/>
-<contactref element="AT4" pad="14"/>
-<wire x1="-5.213" y1="38.386" x2="-5.713" y2="38.386" width="0.254" layer="16"/>
 <wire x1="-4.3" y1="37.125" x2="-4.242" y2="37.183" width="0.254" layer="1"/>
 <wire x1="-4.202" y1="37.125" x2="-4.133" y2="37.056" width="0.254" layer="1"/>
@@
 <contactref element="AT5" pad="15"/>
 <contactref element="AT5" pad="12"/>
-<contactref element="AT5" pad="14"/>
-<wire x1="-5.213" y1="44.386" x2="-5.713" y2="44.386" width="0.254" layer="16"/>
 <wire x1="-4.3" y1="43.125" x2="-4.242" y2="43.183" width="0.254" layer="1"/>
 <wire x1="-4.202" y1="43.125" x2="-4.133" y2="43.056" width="0.254" layer="1"/>
@@
 <contactref element="C28" pad="2"/>
 <contactref element="AT6" pad="15"/>
-<contactref element="AT6" pad="12"/>
-<contactref element="AT6" pad="14"/>
-<wire x1="-5.213" y1="50.386" x2="-5.713" y2="50.386" width="0.254" layer="16"/>
 <wire x1="-4.3" y1="49.125" x2="-4.242" y2="49.183" width="0.254" layer="1"/>
 <wire x1="-4.202" y1="49.125" x2="-4.133" y2="49.056" width="0.254" layer="1"/>
@@
 <contactref element="C33" pad="2"/>
 <contactref element="AT7" pad="15"/>
-<contactref element="AT7" pad="12"/>
-<contactref element="AT7" pad="14"/>
-<wire x1="-5.213" y1="56.386" x2="-5.713" y2="56.386" width="0.254" layer="16"/>
 <wire x1="-4.3" y1="55.125" x2="-4.242" y2="55.183" width="0.254" layer="1"/>
 <wire x1="-4.202" y1="55.125" x2="-4.133" y2="55.056" width="0.254" layer="1"/>
@@
 <contactref element="(8,1)" pad="3"/>
 <contactref element="C38" pad="2"/>
-<contactref element="AT8" pad="15"/>
 <contactref element="AT8" pad="12"/>
-<contactref element="AT8" pad="14"/>
-<wire x1="-5.213" y1="62.386" x2="-5.713" y2="62.386" width="0.254" layer="16"/>
 <wire x1="-4.3" y1="61.125" x2="-4.242" y2="61.183" width="0.254" layer="1"/>
 <wire x1="-4.202" y1="61.125" x2="-4.133" y2="61.056" width="0.254" layer="1"/>
@@
 <wire x1="-5.276" y1="61.691" x2="-5.403" y2="61.564" width="0.254" layer="16"/>
 <wire x1="-5.403" y1="61.564" x2="-5.213" y2="61.754" width="0.254" layer="16"/>
-<wire x1="-5.213" y1="61.754" x2="-5.213" y2="62.386" width="0.254" layer="16"/>
 <wire x1="-17.5" y1="61.35" x2="-17.341" y2="61.509" width="0.254" layer="16"/>
 <wire x1="-17.341" y1="61.509" x2="-17.341" y2="61.564" width="0.254" layer="16"/>
@@
 </polygon>
 <via x="10" y="12.5" extent="1-16" drill="0.475" shape="octagon"/>
+<contactref element="AT8" pad="11"/>
+<contactref element="AT8" pad="14"/>
+<contactref element="AT6" pad="11"/>
+<contactref element="AT4" pad="11"/>
+<contactref element="AT2" pad="11"/>
+<wire x1="-5.713" y1="62.386" x2="-4.26" y2="63.342" width="0" layer="19" extent="16-16"/>
+<wire x1="-5.213" y1="61.754" x2="-5.713" y2="62.386" width="0" layer="19" extent="16-16"/>
+<wire x1="1.963" y1="59.882" x2="1.963" y2="60.04" width="0" layer="19" extent="16-16"/>
+<wire x1="1.963" y1="53.882" x2="1.963" y2="54.04" width="0" layer="19" extent="16-16"/>
+<wire x1="1.963" y1="47.882" x2="1.963" y2="48.04" width="0" layer="19" extent="16-16"/>
+<wire x1="1.963" y1="41.882" x2="1.963" y2="42.04" width="0" layer="19" extent="16-16"/>
+<wire x1="1.963" y1="35.882" x2="1.963" y2="36.04" width="0" layer="19" extent="16-16"/>
+<wire x1="1.963" y1="29.882" x2="1.963" y2="30.04" width="0" layer="19" extent="16-16"/>
+<wire x1="1.963" y1="23.882" x2="1.963" y2="24.04" width="0" layer="19" extent="16-16"/>
+<wire x1="-6.713" y1="62.386" x2="-6.713" y2="61.858" width="0" layer="19" extent="16-16"/>
+<wire x1="-7.213" y1="62.386" x2="-6.713" y2="62.386" width="0" layer="19" extent="16-16"/>
+<wire x1="-6.713" y1="44.386" x2="-6.713" y2="43.858" width="0" layer="19" extent="16-16"/>
+<wire x1="-6.713" y1="38.386" x2="-6.713" y2="37.858" width="0" layer="19" extent="16-16"/>
+<wire x1="-7.213" y1="38.386" x2="-6.713" y2="38.386" width="0" layer="19" extent="16-16"/>
+<wire x1="-6.713" y1="20.386" x2="-6.713" y2="19.858" width="0" layer="19" extent="16-16"/>
+<wire x1="-7.213" y1="50.386" x2="-6.713" y2="49.858" width="0" layer="19" extent="16-16"/>
+<wire x1="-7.213" y1="26.386" x2="-6.713" y2="25.858" width="0" layer="19" extent="16-16"/>
+<wire x1="1" y1="13.5" x2="-0.784" y2="17.111" width="0" layer="19" extent="16-16"/>
+<wire x1="-0.5" y1="12.5" x2="1" y2="13.5" width="0" layer="19" extent="1-1"/>
+<wire x1="-1" y1="7.5" x2="-1" y2="11.4" width="0" layer="19" extent="1-1"/>
+<wire x1="6" y1="7.75" x2="3.4" y2="7.5" width="0" layer="19" extent="1-1"/>
+<wire x1="10" y1="12.5" x2="12.552" y2="17.23" width="0" layer="19" extent="1-1"/>
+<wire x1="-8.55" y1="10.05" x2="-3.4" y2="7.5" width="0" layer="19" extent="1-1"/>
+<wire x1="-14.15" y1="10.25" x2="-8.55" y2="10.05" width="0" layer="19" extent="1-1"/>
+<wire x1="-14.15" y1="8.25" x2="-14.15" y2="10.25" width="0" layer="19" extent="1-1"/>
+<wire x1="-14.15" y1="6.25" x2="-14.15" y2="8.25" width="0" layer="19" extent="1-1"/>
+<wire x1="-9.2" y1="4.175" x2="-14.15" y2="6.25" width="0" layer="19" extent="1-1"/>
+<wire x1="6.84" y1="1.5" x2="6" y2="7.75" width="0" layer="19" extent="1-1"/>
+<wire x1="12.96" y1="6.73" x2="10" y2="12.5" width="0" layer="19" extent="1-1"/>
 </signal>
 <signal name="3.3V">
@@
 <wire x1="-3.625" y1="21.088" x2="11.615" y2="21.088" width="0.254" layer="16"/>
 </signal>
-<signal name="ADDR00">
+<signal name="ADDR1">
 <contactref element="AT1" pad="11"/>
 </signal>
@@
 <wire x1="-3.625" y1="27.088" x2="11.615" y2="27.088" width="0.254" layer="16"/>
 </signal>
-<signal name="ADDR01">
-<contactref element="AT2" pad="11"/>
-</signal>
 <signal name="CAP06">
 <contactref element="C15" pad="1"/>
@@
 <wire x1="-3.625" y1="33.088" x2="11.615" y2="33.088" width="0.254" layer="16"/>
 </signal>
-<signal name="ADDR02">
+<signal name="ADDR3">
 <contactref element="AT3" pad="11"/>
+<contactref element="AT3" pad="12"/>
+<wire x1="-6.713" y1="32.386" x2="-7.213" y2="32.386" width="0" layer="19" extent="16-16"/>
 </signal>
 <signal name="CAP12">
@@
 <wire x1="-12.057" y1="37.437" x2="-12.32" y2="37.7" width="0.254" layer="16"/>
 </signal>
-<signal name="ADDR03">
-<contactref element="AT4" pad="11"/>
-</signal>
 <signal name="CAP17">
 <contactref element="C25" pad="1"/>
@@
 <wire x1="-3.625" y1="45.088" x2="11.615" y2="45.088" width="0.254" layer="16"/>
 </signal>
-<signal name="ADDR04">
+<signal name="ADDR5">
 <contactref element="AT5" pad="11"/>
+<contactref element="AT5" pad="14"/>
+<wire x1="-5.713" y1="44.386" x2="-7.213" y2="44.386" width="0" layer="19" extent="16-16"/>
 </signal>
 <signal name="CAP23">
@@
 <wire x1="-3.625" y1="51.088" x2="11.615" y2="51.088" width="0.254" layer="16"/>
 </signal>
-<signal name="ADDR05">
-<contactref element="AT6" pad="11"/>
-</signal>
 <signal name="CAP28">
 <contactref element="C35" pad="1"/>
@@
 <wire x1="9.995" y1="56.357" x2="10" y2="56.357" width="0.254" layer="16"/>
 </signal>
-<signal name="ADDR06">
+<signal name="ADDR7">
 <contactref element="AT7" pad="11"/>
+<contactref element="AT7" pad="12"/>
+<contactref element="AT7" pad="14"/>
+<wire x1="-6.713" y1="56.386" x2="-7.213" y2="56.386" width="0" layer="19" extent="16-16"/>
+<wire x1="-5.713" y1="56.386" x2="-6.713" y2="56.386" width="0" layer="19" extent="16-16"/>
 </signal>
 <signal name="CAP34">
@@
 <wire x1="9.995" y1="62.357" x2="10" y2="62.357" width="0.254" layer="16"/>
 </signal>
-<signal name="ADDR07">
-<contactref element="AT8" pad="11"/>
-</signal>
 <signal name="RST56">
 <contactref element="PROG6" pad="1"/>
@@
 <contactref element="PROG1" pad="5"/>
 </signal>
+<signal name="ADDR8">
+<contactref element="AT8" pad="15"/>
+</signal>
+<signal name="ADDR6">
+<contactref element="AT6" pad="12"/>
+<contactref element="AT6" pad="14"/>
+<wire x1="-5.713" y1="50.386" x2="-6.713" y2="50.386" width="0" layer="19" extent="16-16"/>
+</signal>
+<signal name="ADDR4">
+<contactref element="AT4" pad="14"/>
+</signal>
+<signal name="ADDR2">
+<contactref element="AT2" pad="12"/>
+</signal>
 </signals>
-<errors>
-</errors>
 </board>
 </drawing>

Commit message: fixed few ERC glitches and ADDR routing
Parts:
- R1: value (none) -> 120o
- R2, R3: value (none) -> 4.7K
- R4: value (none) -> 4.7k
Connections:
- removed net RESET0: AT1.13
- net RESET1: now also AT1.13
Routing:
- net RESET1: track 0.00 -> 20.5 mm
- net RESET0: track 20.5 -> 0.00 mm
- net GND: track 500.0 -> 491.0 mm
