File: eagle/fullArray.brd (EAGLE design)
At the start: 43 x 72 mm, 119 parts

Commit message: center, center, and recenter...
Parts:
- moved 01 1.12 mm to (2.50, 26.0)
- moved 02 1.12 mm to (8.50, 26.0)
- moved 03 1.12 mm to (14.5, 26.0)
- moved 04 1.12 mm to (20.5, 26.0)
- moved 05 1.12 mm to (26.5, 26.0)
- moved 06 1.12 mm to (2.50, 32.0)
- moved 07 1.12 mm to (8.50, 32.0)
- moved 08 1.12 mm to (14.5, 32.0)
- moved 09 1.12 mm to (20.5, 32.0)
- moved 10 1.12 mm to (26.5, 32.0)
- moved 11 1.12 mm to (2.50, 38.0)
- moved 12 1.12 mm to (8.50, 38.0)
- moved 13 1.12 mm to (14.5, 38.0)
- moved 14 1.12 mm to (20.5, 38.0)
- moved 15 1.12 mm to (26.5, 38.0)
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
Commit message: shorten board by 2mm, move mounting holes in
Parts:
- removed U$1, U$2: (no value), nonolith:STAND-OFF
- moved U$4 7.07 mm to (26.5, 17.0)
- moved U$3 6.58 mm to (2.50, 17.0)
- moved C53 2.69 mm to (7.00, 15.5)
- moved 01 2.06 mm to (2.00, 24.0)
- moved 02 2.06 mm to (8.00, 24.0)
- moved 03 2.06 mm to (14.0, 24.0)
- moved 04 2.06 mm to (20.0, 24.0)
- moved 05 2.06 mm to (26.0, 24.0)
- moved 06 2.06 mm to (2.00, 30.0)
- moved 07 2.06 mm to (8.00, 30.0)
- moved 08 2.06 mm to (14.0, 30.0)
- moved 09 2.06 mm to (20.0, 30.0)
- moved 10 2.06 mm to (26.0, 30.0)
- moved 11 2.06 mm to (2.00, 36.0)
- moved 12 2.06 mm to (8.00, 36.0)
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Routing:
- net 3.3V: track 571.6 -> 559.6 mm
- net SDA: track 366.2 -> 363.2 mm, vias 42 -> 43
- net SCL: track 369.8 -> 368.3 mm
- net GND: track 359.3 -> 358.2 mm, vias 78 -> 77
- net 5V: track 27.3 -> 26.6 mm
- net PE0: track 11.8 -> 12.3 mm
Other:
- board size 43 x 72 mm -> 29 x 70.1 mm

Commit message: drop 4-40 header holes for 2.4mm holes, clean a few dimensions
Parts:
- removed U$3, U$4: (no value), nonolith:STAND-OFF
Changed lines of the file:
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@@
 <layer number="43" name="vRestrict" color="2" fill="10" visible="no" active="yes"/>
 <layer number="44" name="Drills" color="7" fill="1" visible="no" active="yes"/>
-<layer number="45" name="Holes" color="7" fill="1" visible="no" active="yes"/>
+<layer number="45" name="Holes" color="7" fill="1" visible="yes" active="yes"/>
 <layer number="46" name="Milling" color="3" fill="1" visible="no" active="yes"/>
 <layer number="47" name="Measures" color="7" fill="1" visible="no" active="yes"/>
@@
 <text x="12.5" y="19.5" size="0.6096" layer="21" font="vector" ratio="12">Cut Here!</text>
 <text x="21" y="19.5" size="0.6096" layer="21" font="vector" ratio="12">Cut Here!</text>
+<hole x="2.5" y="17" drill="2.4"/>
+<hole x="26.5" y="17" drill="2.4"/>
 </plain>
 <attributes>
@@
 <attribute name="VALUE" x="9.23" y="14.825" size="1.27" layer="27"/>
 </element>
-<element name="U$3" library="nonolith" package="STAND-OFF" value="" x="2.5" y="17" smashed="yes"/>
-<element name="U$4" library="nonolith" package="STAND-OFF" value="" x="26.5" y="17"/>
 <element name="JP1" library="nonolith" package="1X01_2MM" value="" x="16.5" y="18" smashed="yes">
 <attribute name="VALUE" x="15.23" y="14.825" size="1.27" layer="27"/>

Commit message: once again, tweak the outline.
Parts:
- moved 01 0.50 mm to (2.50, 24.0)
- moved 02 0.50 mm to (8.50, 24.0)
- moved 03 0.50 mm to (14.5, 24.0)
- moved 04 0.50 mm to (20.5, 24.0)
- moved 05 0.50 mm to (26.5, 24.0)
- moved 06 0.50 mm to (2.50, 30.0)
- moved 07 0.50 mm to (8.50, 30.0)
- moved 08 0.50 mm to (14.5, 30.0)
- moved 09 0.50 mm to (20.5, 30.0)
- moved 10 0.50 mm to (26.5, 30.0)
- moved 11 0.50 mm to (2.50, 36.0)
- moved 12 0.50 mm to (8.50, 36.0)
- moved 13 0.50 mm to (14.5, 36.0)
- moved 14 0.50 mm to (20.5, 36.0)
- moved 15 0.50 mm to (26.5, 36.0)
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Other:
- board size 29 x 70.1 mm -> 29 x 70 mm

Commit message: added branding, version number, and reorganized 4 lines out of USB array to match layout on board
Parts:
- moved JP2 4.00 mm to (11.0, 18.0)
- moved SCL 4.00 mm to (17.0, 18.0)
- moved JP1 2.00 mm to (15.0, 18.0)
- moved SDA 2.00 mm to (13.0, 18.0)
- moved R2 1.00 mm to (19.5, 16.0)
Routing:
- net SCL: track 368.3 -> 363.6 mm
- net SDA: track 363.2 -> 358.6 mm
- net 3.3V: track 559.6 -> 560.6 mm
- net GND: vias 77 -> 78
Other:
- board text added: "TakkArray v1.0"
- board text added: "http://biorobotics.harvard.edu"
- board text added: "www.nonolithlabs.com"
- board text added: "www.takktile.com"
Changed lines of the file:
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@@
 <?xml version="1.0" encoding="utf-8"?>
 <!DOCTYPE eagle SYSTEM "eagle.dtd">
-<eagle version="6.3">
+<eagle version="6.2">
 <drawing>
 <settings>
@@
 <text x="4.818" y="65.032" size="0.7" layer="27" font="vector" ratio="12">G</text>
 <text x="4.818" y="63.127" size="0.7" layer="27" font="vector" ratio="12">C</text>
-<text x="10.5" y="16" size="0.75" layer="21" font="vector" ratio="12">D</text>
-<text x="16.5" y="16" size="0.75" layer="21" font="vector" ratio="12">G</text>
-<text x="12.5" y="16" size="0.75" layer="21" font="vector" ratio="12">C</text>
+<text x="12.5" y="16.5" size="0.75" layer="21" font="vector" ratio="12">D</text>
+<text x="14.5" y="16.5" size="0.75" layer="21" font="vector" ratio="12">G</text>
+<text x="16.5" y="16.5" size="0.75" layer="21" font="vector" ratio="12">C</text>
 <wire x1="0.5" y1="20.5" x2="29.5" y2="20.5" width="0.3048" layer="21"/>
 <wire x1="0.5" y1="19" x2="29.5" y2="19" width="0.3048" layer="21"/>
 <text x="4" y="19.5" size="0.6096" layer="21" font="vector" ratio="12">Cut Here!</text>
-<text x="14.5" y="16" size="0.75" layer="21" font="vector" ratio="12">V</text>
+<text x="10.5" y="16.5" size="0.75" layer="21" font="vector" ratio="12">V</text>
 <text x="13" y="19.5" size="0.6096" layer="21" font="vector" ratio="12">Cut Here!</text>
 <text x="21.5" y="19.5" size="0.6096" layer="21" font="vector" ratio="12">Cut Here!</text>
-<hole x="3" y="17" drill="2.4"/>
-<hole x="27" y="17" drill="2.4"/>
+<hole x="2.5" y="17" drill="2.4"/>
+<hole x="26.5" y="17" drill="2.4"/>
+<circle x="26.5" y="17" radius="2" width="0.1" layer="21"/>
+<circle x="2.5" y="17" radius="2" width="0.1" layer="21"/>
+<text x="23" y="15" size="1.5" layer="26" rot="MR0">www.takktile.com</text>
+<text x="22" y="12" size="1" layer="22" rot="MR0">www.nonolithlabs.com</text>
+<text x="24" y="13.5" size="1" layer="26" rot="MR0">http://biorobotics.harvard.edu</text>
+<text x="20" y="4.5" size="1" layer="22" rot="MR0">TakkArray v1.0</text>
 </plain>
 <attributes>
@@
 </class>
 </classes>
-<designrules name="ITead_rule">
+<designrules>
 <description language="de">&lt;b&gt;EAGLE Design Rules&lt;/b&gt;
 &lt;p&gt;
@@
 <attribute name="VALUE" x="22.393" y="8.73" size="0.4064" layer="27" rot="R90"/>
 </element>
-<element name="R2" library="nonolith" package="0603" value="4.7K" x="18.5" y="16"/>
+<element name="R2" library="nonolith" package="0603" value="4.7K" x="19.5" y="16"/>
 <element name="R3" library="nonolith" package="0603" value="4.7K" x="18.5" y="14"/>
 <element name="DAISY" library="nonolith" package="1X06_ROUND_2MM" value="" x="23" y="1.5" smashed="yes" rot="R180">
@@
 </element>
 <element name="R4" library="nonolith" package="0603" value="4.7k" x="22" y="4.5" smashed="yes" rot="R90"/>
-<element name="SCL" library="nonolith" package="1X01_2MM" value="" x="13" y="18" smashed="yes">
-<attribute name="VALUE" x="11.73" y="14.825" size="1.27" layer="27"/>
-</element>
-<element name="SDA" library="nonolith" package="1X01_2MM" value="" x="11" y="18" smashed="yes">
-<attribute name="VALUE" x="9.73" y="14.825" size="1.27" layer="27"/>
-</element>
-<element name="JP1" library="nonolith" package="1X01_2MM" value="" x="17" y="18" smashed="yes">
+<element name="SCL" library="nonolith" package="1X01_2MM" value="" x="17" y="18" smashed="yes">
 <attribute name="VALUE" x="15.73" y="14.825" size="1.27" layer="27"/>
 </element>
-<element name="JP2" library="nonolith" package="1X01_2MM" value="" x="15" y="18" smashed="yes">
+<element name="SDA" library="nonolith" package="1X01_2MM" value="" x="13" y="18" smashed="yes">
+<attribute name="VALUE" x="11.73" y="14.825" size="1.27" layer="27"/>
+</element>
+<element name="JP1" library="nonolith" package="1X01_2MM" value="" x="15" y="18" smashed="yes">
 <attribute name="VALUE" x="13.73" y="14.825" size="1.27" layer="27"/>
 </element>
+<element name="JP2" library="nonolith" package="1X01_2MM" value="" x="11" y="18" smashed="yes">
+<attribute name="VALUE" x="9.73" y="14.825" size="1.27" layer="27"/>
+</element>
 <element name="U$5" library="nonolith" package="LOGO_NONOLITH" value="" x="17.9" y="6.1" rot="MR0"/>
 <element name="C52" library="microbuilder" package="EIA7343-31/D-R" value="470uF" x="26.5" y="5.5" smashed="yes" rot="R90"/>
@@
 <wire x1="15" y1="7.5" x2="12.6" y2="7.5" width="0.254" layer="1"/>
 <contactref element="JP1" pad="1"/>
-<via x="28.5" y="11" extent="1-16" drill="0.305" shape="octagon"/>
+<via x="28" y="13.5" extent="1-16" drill="0.305" shape="octagon"/>
 <contactref element="C52" pad="-"/>
 <wire x1="15" y1="11.4" x2="15" y2="12" width="0.254" layer="1"/>
@@
 <via x="28" y="5" extent="1-16" drill="0.305" shape="octagon"/>
 <via x="25.5" y="6.5" extent="1-16" drill="0.305" shape="octagon"/>
+<via x="15" y="16" extent="1-16" drill="0.305" shape="octagon"/>
 </signal>
 <signal name="3.3V">
@@
 <via x="15" y="13" extent="1-16" drill="0.305" shape="octagon"/>
 <wire x1="15" y1="13" x2="15" y2="8" width="0.254" layer="16"/>
-<wire x1="15" y1="15" x2="15" y2="18" width="0.4064" layer="1"/>
+<wire x1="11" y1="15" x2="11" y2="18" width="0.4064" layer="1"/>
 <wire x1="19.35" y1="12.85" x2="19.35" y2="14" width="0.254" layer="1"/>
 <wire x1="19.35" y1="14" x2="19.35" y2="14.75" width="0.4064" layer="1"/>
 <wire x1="19.35" y1="14.75" x2="19.35" y2="15" width="0.4064" layer="1"/>
-<wire x1="19.35" y1="15" x2="19.35" y2="16" width="0.4064" layer="1"/>
+<wire x1="19.35" y1="15" x2="20.35" y2="16" width="0.4064" layer="1"/>
 <wire x1="22.65" y1="14.75" x2="19.35" y2="14.75" width="0.4064" layer="1"/>
 <wire x1="19.4" y1="8" x2="20.5" y2="8" width="0.254" layer="1"/>
@@
 <wire x1="22.65" y1="13.25" x2="22.65" y2="12.25" width="0.4064" layer="1"/>
 <wire x1="22.65" y1="12.25" x2="23.15" y2="11.75" width="0.4064" layer="1"/>
-<wire x1="15" y1="15" x2="19.35" y2="15" width="0.4064" layer="1"/>
-<wire x1="15" y1="18" x2="15" y2="19.5" width="0.254" layer="16"/>
-<wire x1="15" y1="19.5" x2="9.239" y2="19.5" width="0.254" layer="16"/>
-<wire x1="9.239" y1="19.5" x2="6.596" y2="22.143" width="0.254" layer="16"/>
+<wire x1="11" y1="15" x2="19.35" y2="15" width="0.4064" layer="1"/>
+<wire x1="11" y1="18" x2="11" y2="20.5" width="0.254" layer="16"/>
+<wire x1="11" y1="20.5" x2="8.239" y2="20.5" width="0.254" layer="16"/>
+<wire x1="8.239" y1="20.5" x2="6.596" y2="22.143" width="0.254" layer="16"/>
 </signal>
 <signal name="SDA">
@@
 <contactref element="R3" pad="1"/>
 <wire x1="14" y1="11.4" x2="14" y2="12" width="0.254" layer="1"/>
-<wire x1="14" y1="12" x2="13.5" y2="12.5" width="0.254" layer="1"/>
-<wire x1="13.5" y1="12.5" x2="11" y2="12.5" width="0.254" layer="1"/>
+<wire x1="14" y1="12" x2="13" y2="14" width="0.254" layer="1"/>
 <contactref element="SDA" pad="1"/>
-<wire x1="17.65" y1="14" x2="15" y2="14" width="0.254" layer="1"/>
-<wire x1="15" y1="14" x2="13.5" y2="12.5" width="0.254" layer="1"/>
-<via x="11" y="12.5" extent="1-16" drill="0.305" shape="octagon"/>
-<wire x1="11" y1="12.5" x2="11" y2="18" width="0.254" layer="16"/>
-<wire x1="11" y1="18" x2="11" y2="20.5" width="0.254" layer="1"/>
-<via x="11" y="20.5" extent="1-16" drill="0.305" shape="octagon"/>
-<wire x1="11" y1="20.5" x2="18" y2="20.5" width="0.254" layer="16"/>
+<wire x1="17.65" y1="14" x2="13" y2="14" width="0.254" layer="1"/>
+<via x="13" y="14" extent="1-16" drill="0.305" shape="octagon"/>
+<wire x1="13" y1="14" x2="13" y2="18" width="0.254" layer="16"/>
+<wire x1="13" y1="18" x2="13" y2="20.5" width="0.254" layer="1"/>
+<via x="13" y="20.5" extent="1-16" drill="0.305" shape="octagon"/>
+<wire x1="13" y1="20.5" x2="18" y2="20.5" width="0.254" layer="16"/>
 <via x="18" y="20.5" extent="1-16" drill="0.305" shape="octagon"/>
 <wire x1="18" y1="20.5" x2="22.598" y2="20.5" width="0.254" layer="1"/>
@@
 <wire x1="13.5" y1="11.4" x2="13.5" y2="11.5" width="0.254" layer="1"/>
 <contactref element="SCL" pad="1"/>
-<wire x1="13" y1="18" x2="13" y2="16" width="0.254" layer="16"/>
-<wire x1="13" y1="16" x2="13" y2="13" width="0.254" layer="16"/>
-<wire x1="13.5" y1="11.5" x2="11.5" y2="11.5" width="0.254" layer="1"/>
-<via x="11.5" y="11.5" extent="1-16" drill="0.305" shape="octagon"/>
-<wire x1="11.5" y1="11.5" x2="13" y2="13" width="0.254" layer="16"/>
-<wire x1="17.65" y1="16" x2="16" y2="16" width="0.254" layer="1"/>
-<via x="16" y="16" extent="1-16" drill="0.305" shape="octagon"/>
-<wire x1="16" y1="16" x2="13" y2="16" width="0.254" layer="16"/>
-<wire x1="13" y1="18" x2="13" y2="22.125" width="0.254" layer="1"/>
-<wire x1="13" y1="22.125" x2="13.3" y2="22.125" width="0.254" layer="1"/>
+<wire x1="17" y1="18" x2="17" y2="16" width="0.254" layer="16"/>
+<wire x1="17" y1="16" x2="16.5" y2="15.5" width="0.254" layer="16"/>
+<wire x1="13.5" y1="11.5" x2="13" y2="12.5" width="0.254" layer="1"/>
+<via x="13" y="12.5" extent="1-16" drill="0.305" shape="octagon"/>
+<wire x1="13" y1="12.5" x2="16.5" y2="15.5" width="0.254" layer="16"/>
+<wire x1="18.65" y1="16" x2="17" y2="16" width="0.254" layer="1"/>
+<via x="17" y="16" extent="1-16" drill="0.305" shape="octagon"/>
+<wire x1="17" y1="18" x2="17" y2="21.125" width="0.254" layer="1"/>
+<wire x1="17" y1="21.125" x2="16.756" y2="21.125" width="0.3" layer="1"/>
+<wire x1="16.756" y1="21.125" x2="16.756" y2="21.127" width="0.3" layer="1"/>
 </signal>
 <signal name="CAP03">

Commit message: s/proportional font/vector font/, move a few traces to 45deg
Parts:
- moved R1 0.50 mm to (23.0, 8.05)
Changed lines of the file:
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@@
 <?xml version="1.0" encoding="utf-8"?>
 <!DOCTYPE eagle SYSTEM "eagle.dtd">
-<eagle version="6.2">
+<eagle version="6.3">
 <drawing>
 <settings>
@@
 <circle x="26.5" y="17" radius="2" width="0.1" layer="21"/>
 <circle x="2.5" y="17" radius="2" width="0.1" layer="21"/>
-<text x="23" y="15" size="1.5" layer="26" rot="MR0">www.takktile.com</text>
-<text x="22" y="12" size="1" layer="22" rot="MR0">www.nonolithlabs.com</text>
-<text x="24" y="13.5" size="1" layer="26" rot="MR0">http://biorobotics.harvard.edu</text>
+<text x="23" y="15" size="1.5" layer="26" font="vector" ratio="12" rot="MR0">www.takktile.com</text>
+<text x="22" y="12" size="1" layer="22" font="vector" ratio="12" rot="MR0">www.nonolithlabs.com</text>
+<text x="24" y="13.5" size="1" layer="26" font="vector" ratio="12" rot="MR0">http://biorobotics.harvard.edu</text>
 <text x="20" y="4.5" size="1" layer="22" rot="MR0">TakkArray v1.0</text>
 </plain>
@@
 </class>
 </classes>
-<designrules>
+<designrules name="default">
 <description language="de">&lt;b&gt;EAGLE Design Rules&lt;/b&gt;
 &lt;p&gt;
@@
 <attribute name="NAME" x="25.778" y="12.504" size="0.762" layer="25" font="vector" ratio="10"/>
 </element>
-<element name="R1" library="nonolith" package="0603" value="120o" x="23" y="8.55" smashed="yes" rot="R90"/>
+<element name="R1" library="nonolith" package="0603" value="120o" x="23" y="8.05" smashed="yes" rot="R90"/>
 <element name="LED1" library="microbuilder" package="CHIPLED_0603" value="" x="21.25" y="10" smashed="yes">
 <attribute name="VALUE" x="22.393" y="8.73" size="0.4064" layer="27" rot="R90"/>
@@
 <contactref element="XM1" pad="10"/>
 <contactref element="R3" pad="1"/>
-<wire x1="14" y1="11.4" x2="14" y2="12" width="0.254" layer="1"/>
-<wire x1="14" y1="12" x2="13" y2="14" width="0.254" layer="1"/>
 <contactref element="SDA" pad="1"/>
 <wire x1="17.65" y1="14" x2="13" y2="14" width="0.254" layer="1"/>
@@
 <wire x1="18" y1="20.5" x2="22.598" y2="20.5" width="0.254" layer="1"/>
 <wire x1="22.598" y1="20.5" x2="22.598" y2="22.016" width="0.254" layer="1"/>
+<wire x1="14" y1="11.4" x2="14" y2="13" width="0.254" layer="1"/>
+<wire x1="14" y1="13" x2="13" y2="14" width="0.254" layer="1"/>
 </signal>
 <signal name="SCL">
@@
 <contactref element="XM1" pad="11"/>
 <contactref element="R2" pad="1"/>
-<wire x1="13.5" y1="11.4" x2="13.5" y2="11.5" width="0.254" layer="1"/>
 <contactref element="SCL" pad="1"/>
 <wire x1="17" y1="18" x2="17" y2="16" width="0.254" layer="16"/>
-<wire x1="17" y1="16" x2="16.5" y2="15.5" width="0.254" layer="16"/>
-<wire x1="13.5" y1="11.5" x2="13" y2="12.5" width="0.254" layer="1"/>
-<via x="13" y="12.5" extent="1-16" drill="0.305" shape="octagon"/>
-<wire x1="13" y1="12.5" x2="16.5" y2="15.5" width="0.254" layer="16"/>
 <wire x1="18.65" y1="16" x2="17" y2="16" width="0.254" layer="1"/>
 <via x="17" y="16" extent="1-16" drill="0.305" shape="octagon"/>
@@
 <wire x1="17" y1="21.125" x2="16.756" y2="21.125" width="0.3" layer="1"/>
 <wire x1="16.756" y1="21.125" x2="16.756" y2="21.127" width="0.3" layer="1"/>
+<wire x1="13.5" y1="11.4" x2="13.5" y2="12" width="0.254" layer="1"/>
+<wire x1="13.5" y1="12" x2="13" y2="12.5" width="0.254" layer="1"/>
+<via x="13" y="12.5" extent="1-16" drill="0.305" shape="octagon"/>
+<wire x1="13" y1="12.5" x2="13.5" y2="12.5" width="0.254" layer="16"/>
+<wire x1="13.5" y1="12.5" x2="17" y2="16" width="0.254" layer="16"/>
 </signal>
 <signal name="CAP03">
@@
 <contactref element="R1" pad="1"/>
 <wire x1="19.4" y1="7" x2="22.5" y2="7" width="0.254" layer="1"/>
-<wire x1="23" y1="7.7" x2="23" y2="7.5" width="0.254" layer="1"/>
+<wire x1="23" y1="7.2" x2="23" y2="7.5" width="0.254" layer="1"/>
 <wire x1="23" y1="7.5" x2="22.5" y2="7" width="0.254" layer="1"/>
 </signal>
@@
 <contactref element="R1" pad="2"/>
 <contactref element="LED1" pad="A"/>
-<wire x1="23" y1="9.4" x2="21.4" y2="9.4" width="0.254" layer="1"/>
 <wire x1="21.4" y1="9.4" x2="21.25" y2="9.25" width="0.254" layer="1"/>
+<wire x1="23" y1="8.9" x2="21.6" y2="8.9" width="0.254" layer="1"/>
+<wire x1="21.6" y1="8.9" x2="21.25" y2="9.25" width="0.254" layer="1"/>
 </signal>
 <signal name="BOOTLOAD">

Commit message: s/0603 resistor/solder jumper/, clean power traces, add 0.5mm vias for PDI-DATA and PDI-CLK
Parts:
- removed R4: 4.7k, nonolith:0603
- added SJ1: (no value), jumper:SJ
- moved R3 1.00 mm to (19.5, 14.0)
- moved C11 0.50 mm to (23.5, 11.8), turned to 0 degrees
- turned C10 to 0 degrees
- turned C12 to 0 degrees
Connections:
- net 3.3V: now also SJ1.2; no longer R4.2
- net PE0: now also SJ1.1; no longer R4.1
Routing:
- net 3.3V: track 560.6 -> 575.9 mm, vias 60 -> 61
- net PDI-DATA: track 0.00 -> 1.60 mm, vias 0 -> 1
- net PDI-CLK: track 0.00 -> 1.10 mm, vias 0 -> 1
- net SDA: track 358.7 -> 359.7 mm
- net PE0: track 12.3 -> 13.0 mm
- net GND: vias 78 -> 84
