File: eagle/fullArray.sch (EAGLE design)
At the start: 96 parts

Commit message: Connected vertically stacked boards
Full 8-vertical layout now has power and SPI lines connected betwble een
boards.
Added the tessellatable layout go make arbitrarily high stacks.
Parts:
- removed S41, S42, S43, S44, S45, S46: MPL115A, nonolith:MPL115A
- added S08, S09, S18, S19, S28, S29: MPL115A, nonolith:MPL115A
- renumbered S47 to S38
Connections:
- net ADDR01 renamed ADDR00-2
- net ADDR02 renamed ADDR00-3
- net ADDR03 renamed ADDR00-4
- net ADDR04 renamed ADDR00-5
- net ADDR05 renamed ADDR00-6
- net ADDR06 renamed ADDR00-7
- net ADDR07 renamed ADDR00-8
- net CAP01 renamed CAP04-2
- net CAP13 renamed CAP05-4
- net CAP25 renamed CAP01-6
- net CAP37 renamed CAP02-8
- net CAP47 renamed CAP03-8
- net RESET1 renamed RESET0-2
- net RESET2 renamed RESET0-3
- net RESET3 renamed RESET0-4
- net RESET4 renamed RESET0-5
- net RESET5 renamed RESET0-6
- net RESET6 renamed RESET0-7
- net RESET7 renamed RESET0-8
- net RST01 renamed RST00-2
- net RST13 renamed RST10-4
- net RST25 renamed RST20-6
- net RST37 renamed RST30-8
- net RST47 renamed RST40-8
- removed net CAP02: C10.P$1, S02.CAP
- removed net CAP03: C15.P$1, S03.CAP
- removed net CAP04: C20.P$1, S04.CAP
- removed net CAP05: C25.P$1, S05.CAP
- removed net CAP06: C30.P$1, S06.CAP
- removed net CAP07: C35.P$1, S07.CAP
- removed net CAP11: C6.P$1, S11.CAP
- removed net CAP12: C11.P$1, S12.CAP
- removed net CAP14: C21.P$1, S14.CAP
- removed net CAP15: C26.P$1, S15.CAP
- removed net CAP16: C31.P$1, S16.CAP
- removed net CAP17: C36.P$1, S17.CAP
- removed net CAP21: C7.P$1, S21.CAP
- removed net CAP22: C12.P$1, S22.CAP
- removed net CAP23: C17.P$1, S23.CAP
- removed net CAP24: C22.P$1, S24.CAP
- removed net CAP26: C32.P$1, S26.CAP
- removed net CAP27: C37.P$1, S27.CAP
- removed net CAP31: C8.P$1, S31.CAP
- removed net CAP32: C13.P$1, S32.CAP
- removed net CAP33: C18.P$1, S33.CAP
- removed net CAP34: C23.P$1, S34.CAP
- removed net CAP35: C28.P$1, S35.CAP
- removed net CAP36: C33.P$1, S36.CAP
- removed net CAP41: C9.P$1, S41.CAP
- removed net CAP42: C14.P$1, S42.CAP
- removed net CAP43: C19.P$1, S43.CAP
- removed net CAP44: C24.P$1, S44.CAP
- removed net CAP45: C29.P$1, S45.CAP
- removed net CAP46: C34.P$1, S46.CAP
- removed net RST02: S02.RST, UC2.PA0/ADC0
- removed net RST03: S03.RST, UC3.PA0/ADC0
- removed net RST04: S04.RST, UC4.PA0/ADC0
- removed net RST05: S05.RST, UC5.PA0/ADC0
- removed net RST06: S06.RST, UC6.PA0/ADC0
- removed net RST07: S07.RST, UC7.PA0/ADC0
- removed net RST11: S11.RST, UC1.PA1/ADC1
- removed net RST12: S12.RST, UC2.PA1/ADC1
- removed net RST14: S14.RST, UC4.PA1/ADC1
- removed net RST15: S15.RST, UC5.PA1/ADC1
- removed net RST16: S16.RST, UC6.PA1/ADC1
- removed net RST17: S17.RST, UC7.PA1/ADC1
- removed net RST21: S21.RST, UC1.PA2/ADC2
- removed net RST22: S22.RST, UC2.PA2/ADC2
- removed net RST23: S23.RST, UC3.PA2/ADC2
- removed net RST24: S24.RST, UC4.PA2/ADC2
- removed net RST26: S26.RST, UC6.PA2/ADC2
- removed net RST27: S27.RST, UC7.PA2/ADC2
- removed net RST31: S31.RST, UC1.PA3/ADC3
- removed net RST32: S32.RST, UC2.PA3/ADC3
- removed net RST33: S33.RST, UC3.PA3/ADC3
- removed net RST34: S34.RST, UC4.PA3/ADC3
- removed net RST35: S35.RST, UC5.PA3/ADC3
- removed net RST36: S36.RST, UC6.PA3/ADC3
- removed net RST41: PROG1.1, S41.RST, UC1.PA5/MISO
- removed net RST42: PROG2.1, S42.RST, UC2.PA5/MISO
- removed net RST43: PROG3.1, S43.RST, UC3.PA5/MISO
- removed net RST44: PROG4.1, S44.RST, UC4.PA5/MISO
- removed net RST45: PROG5.1, S45.RST, UC5.PA5/MISO
- removed net RST46: PROG6.1, S46.RST, UC6.PA5/MISO
- new net CAP01-2: C7.P$1, S03.CAP
- new net CAP01-3: C12.P$1, S08.CAP
- new net CAP01-4: C17.P$1, S14.CAP
- new net CAP01-5: C22.P$1, S19.CAP
- new net CAP01-7: C32.P$1, S31.CAP
- new net CAP01-8: C37.P$1, S36.CAP
- new net CAP02-2: C8.P$1, S04.CAP
- new net CAP02-3: C13.P$1, S09.CAP
- new net CAP02-4: C18.P$1, S15.CAP
- new net CAP02-5: C23.P$1, S21.CAP
- new net CAP02-6: C28.P$1, S26.CAP
- new net CAP02-7: C33.P$1, S32.CAP
- new net CAP03-2: C9.P$1, S05.CAP
- new net CAP03-3: C14.P$1, S11.CAP
- new net CAP03-4: C19.P$1, S16.CAP
- new net CAP03-5: C24.P$1, S22.CAP
- new net CAP03-6: C29.P$1, S27.CAP
- new net CAP03-7: C34.P$1, S33.CAP
- new net CAP04-3: C10.P$1, S06.CAP
- new net CAP04-4: C15.P$1, S12.CAP
- new net CAP04-5: C20.P$1, S17.CAP
- new net CAP04-6: C25.P$1, S23.CAP
- new net CAP04-7: C30.P$1, S28.CAP
- new net CAP04-8: C35.P$1, S34.CAP
- new net CAP05-2: C6.P$1, S02.CAP
- new net CAP05-3: C11.P$1, S07.CAP
- new net CAP05-5: C21.P$1, S18.CAP
- new net CAP05-6: C26.P$1, S24.CAP
- new net CAP05-7: C31.P$1, S29.CAP
- new net CAP05-8: C36.P$1, S35.CAP
- new net RST00-3: S06.RST, UC2.PA0/ADC0
- new net RST00-4: S12.RST, UC3.PA0/ADC0
- new net RST00-5: S17.RST, UC4.PA0/ADC0
- new net RST00-6: S23.RST, UC5.PA0/ADC0
- new net RST00-7: S28.RST, UC6.PA0/ADC0
- new net RST00-8: S34.RST, UC7.PA0/ADC0
- new net RST10-2: S02.RST, UC1.PA1/ADC1
- new net RST10-3: S07.RST, UC2.PA1/ADC1
- new net RST10-5: S18.RST, UC4.PA1/ADC1
- new net RST10-6: S24.RST, UC5.PA1/ADC1
- new net RST10-7: S29.RST, UC6.PA1/ADC1
- new net RST10-8: S35.RST, UC7.PA1/ADC1
- new net RST20-2: S03.RST, UC1.PA2/ADC2
- new net RST20-3: S08.RST, UC2.PA2/ADC2
- new net RST20-4: S14.RST, UC3.PA2/ADC2
- new net RST20-5: S19.RST, UC4.PA2/ADC2
- new net RST20-7: S31.RST, UC6.PA2/ADC2
- new net RST20-8: S36.RST, UC7.PA2/ADC2
- new net RST30-2: S04.RST, UC1.PA3/ADC3
- new net RST30-3: S09.RST, UC2.PA3/ADC3
- new net RST30-4: S15.RST, UC3.PA3/ADC3
- new net RST30-5: S21.RST, UC4.PA3/ADC3
- new net RST30-6: S26.RST, UC5.PA3/ADC3
- new net RST30-7: S32.RST, UC6.PA3/ADC3
- new net RST40-2: PROG1.1, S05.RST, UC1.PA5/MISO
- new net RST40-3: PROG2.1, S11.RST, UC2.PA5/MISO
- new net RST40-4: PROG3.1, S16.RST, UC3.PA5/MISO
- new net RST40-5: PROG4.1, S22.RST, UC4.PA5/MISO
- new net RST40-6: PROG5.1, S27.RST, UC5.PA5/MISO
- new net RST40-7: PROG6.1, S33.RST, UC6.PA5/MISO
- net 3.3V: now also S08.SHDN, S08.VDD, S09.SHDN, S09.VDD, S18.SHDN, S18.VDD, S19.SHDN, S19.VDD, S28.SHDN, S28.VDD, S29.SHDN, S29.VDD; no longer S41.SHDN, S41.VDD, S42.SHDN, S42.VDD, S43.SHDN, S43.VDD, S44.SHDN, S44.VDD, S45.SHDN, S45.VDD, S46.SHDN, S46.VDD
- net GND: now also S08.GND, S09.GND, S18.GND, S19.GND, S28.GND, S29.GND; no longer S41.GND, S42.GND, S43.GND, S44.GND, S45.GND, S46.GND
- net SCL: now also S08.SCL, S09.SCL, S18.SCL, S19.SCL, S28.SCL, S29.SCL; no longer S41.SCL, S42.SCL, S43.SCL, S44.SCL, S45.SCL, S46.SCL
- net SDA: now also S08.SDA, S09.SDA, S18.SDA, S19.SDA, S28.SDA, S29.SDA; no longer S41.SDA, S42.SDA, S43.SDA, S44.SDA, S45.SDA, S46.SDA

Commit message: added four row board w/ USB interface.
Parts:
- removed C23, C24, C25, C26, C27, C28, C29, C30, C31, C32, C33, C34, C35, C36, C37, C38, C39: (no value), nonolith:CAP_CERAMIC0603
- removed PROG4, PROG5, PROG6, PROG7: (no value), nonolith:HEADER-2X3
- removed S17, S18, S19, S21, S22, S23, S24, S25, S26, S27, S28, S29, S31, S32, S33, S34, S35, S36, S37, S38: MPL115A, nonolith:MPL115A
- removed UC4, UC5, UC6, UC7: ATTINY24QFN, nonolith:ATTINY24QFN
- added 3.3V: VREG, nonolith:VREG
- added CN1: (no value), nonolith:USBMICROB
- added DAISY: (no value), nonolith:HEADER-1X62MM
- added IC1: (no value), nonolith:ATXMEGAXXA4U-MH
- added JP1, JP2, SCL, SDA: (no value), nonolith:HEADER-1X12MM
- added LED1: (no value), microbuilder:LED0603
- added PROG0: (no value), nonolith:HEADER-2X3
- added R1, R2, R3, R4: (no value), nonolith:RESISTOR0603
- C10: value (none) -> 1uF
- C11: value (none) -> .1uF
- C12: value (none) -> .01uF
Connections:
- net ADDR00-2 renamed ADDR01
- net ADDR00-3 renamed ADDR02
- net ADDR00-4 renamed ADDR03
- net CAP01-2 renamed CAP01
- net CAP02-2 renamed CAP02
- net CAP03-2 renamed CAP03
- net CAP04-2 renamed CAP04
- net CAP05-2 renamed CAP05
- net RESET0-2 renamed RESET1
- net RESET0-3 renamed RESET2
- net RESET0-4 renamed RESET3
- net RST00-2 renamed RST01
- net RST00-3 renamed RST02
- net RST00-4 renamed RST03
- net RST10-2 renamed RST11
- net RST10-3 renamed RST12
- net RST10-4 renamed RST13
- net RST20-2 renamed RST21
- net RST20-3 renamed RST22
- net RST20-4 renamed RST23
- net RST30-2 renamed RST31
- net RST30-3 renamed RST32
- net RST30-4 renamed RST33
- net RST40-2 renamed RST41
- net RST40-3 renamed RST42
- net RST40-4 renamed RST43
- removed net ADDR00-5: UC4.PB0
- removed net ADDR00-6: UC5.PB0
- removed net ADDR00-7: UC6.PB0
- removed net ADDR00-8: UC7.PB0
- removed net CAP01-3: C12.P$1, S08.CAP
- removed net CAP01-4: C17.P$1, S14.CAP
- removed net CAP01-5: C22.P$1, S19.CAP
- removed net CAP01-6: C27.P$1, S25.CAP
- removed net CAP01-7: C32.P$1, S31.CAP
- removed net CAP01-8: C37.P$1, S36.CAP
- removed net CAP02-3: C13.P$1, S09.CAP
- removed net CAP02-4: C18.P$1, S15.CAP
- removed net CAP02-5: C23.P$1, S21.CAP
- removed net CAP02-6: C28.P$1, S26.CAP
- removed net CAP02-7: C33.P$1, S32.CAP
- removed net CAP02-8: C38.P$1, S37.CAP
- removed net CAP03-3: C14.P$1, S11.CAP
- removed net CAP03-4: C19.P$1, S16.CAP
- removed net CAP03-5: C24.P$1, S22.CAP
- removed net CAP03-6: C29.P$1, S27.CAP
- removed net CAP03-7: C34.P$1, S33.CAP
- removed net CAP03-8: C39.P$1, S38.CAP
- removed net CAP04-3: C10.P$1, S06.CAP
- removed net CAP04-4: C15.P$1, S12.CAP
- removed net CAP04-5: C20.P$1, S17.CAP
- removed net CAP04-6: C25.P$1, S23.CAP
- removed net CAP04-7: C30.P$1, S28.CAP
- removed net CAP04-8: C35.P$1, S34.CAP
- removed net CAP05-3: C11.P$1, S07.CAP
- removed net CAP05-4: C16.P$1, S13.CAP
- removed net CAP05-5: C21.P$1, S18.CAP
- removed net CAP05-6: C26.P$1, S24.CAP
- removed net CAP05-7: C31.P$1, S29.CAP
- removed net CAP05-8: C36.P$1, S35.CAP
- removed net RESET0-5: PROG4.5, UC4.PB3/RESET
- removed net RESET0-6: PROG5.5, UC5.PB3/RESET
- removed net RESET0-7: PROG6.5, UC6.PB3/RESET
- removed net RESET0-8: PROG7.5, UC7.PB3/RESET
- removed net RST00-5: S17.RST, UC4.PA0/ADC0
- removed net RST00-6: S23.RST, UC5.PA0/ADC0
- removed net RST00-7: S28.RST, UC6.PA0/ADC0
- removed net RST00-8: S34.RST, UC7.PA0/ADC0
- removed net RST10-5: S18.RST, UC4.PA1/ADC1
- removed net RST10-6: S24.RST, UC5.PA1/ADC1
- removed net RST10-7: S29.RST, UC6.PA1/ADC1
- removed net RST10-8: S35.RST, UC7.PA1/ADC1
- removed net RST20-5: S19.RST, UC4.PA2/ADC2
- removed net RST20-6: S25.RST, UC5.PA2/ADC2
- removed net RST20-7: S31.RST, UC6.PA2/ADC2
- removed net RST20-8: S36.RST, UC7.PA2/ADC2
- removed net RST30-5: S21.RST, UC4.PA3/ADC3
- removed net RST30-6: S26.RST, UC5.PA3/ADC3
- removed net RST30-7: S32.RST, UC6.PA3/ADC3
- removed net RST30-8: S37.RST, UC7.PA3/ADC3
- removed net RST40-5: PROG4.1, S22.RST, UC4.PA5/MISO
- removed net RST40-6: PROG5.1, S27.RST, UC5.PA5/MISO
- removed net RST40-7: PROG6.1, S33.RST, UC6.PA5/MISO
- removed net RST40-8: PROG7.1, S38.RST, UC7.PA5/MISO
- new net 5V: 3.3V.VIN, CN1.VBUS, DAISY.6
- new net BOOTLOAD: IC1.PR0/XTAL2, PROG.4
- new net CAP06: C15.P$1, S08.CAP
- new net CAP07: C16.P$1, S09.CAP
- new net CAP08: C17.P$1, S11.CAP
- new net CAP09: C13.P$1, S06.CAP
- new net CAP11: C14.P$1, S07.CAP
- new net CAP12: C20.P$1, S14.CAP
- new net CAP13: C21.P$1, S15.CAP
- new net CAP14: C22.P$1, S16.CAP
- new net CAP15: C18.P$1, S12.CAP
- new net CAP16: C19.P$1, S13.CAP
- new net PDI-CLK: IC1.RESET/PDI-CLK, PROG.5
- new net PDI-DATA: IC1.PDI-DATA, PROG.1
- new net PE0: DAISY.5, IC1.OC0A/SDA/PE0, R4.1
- new net PE1: DAISY.4, IC1.XCK0/OC0B/SCL/PE1
- new net PE2: DAISY.3, IC1.RXD0/OC0C/PE2
- new net PE3: DAISY.2, IC1.TXD0/OC0D/PE3
- new net PR1: IC1.PR1/XTAL1, PROG.3, R1.1
- new net PR1-P: LED1.A, R1.2
- new net USB+: CN1.D+, IC1.TXD1/USB+/PD7
- new net USB-: CN1.D-, IC1.RXD1/MISO/USB-/PD6
- net 3.3V: now also 3.3V.VO, C10.P$2, C11.P$2, C12.P$2, IC1.AVCC, IC1.VCC@1, IC1.VCC@2, IC1.VCC@3, JP2.1, PROG0.2, R2.2, R3.2, R4.2; no longer PROG4.2, PROG5.2, PROG6.2, PROG7.2, S17.SHDN, S17.VDD, S18.SHDN, S18.VDD, S19.SHDN, S19.VDD, S21.SHDN, S21.VDD, S22.SHDN, S22.VDD, S23.SHDN, S23.VDD, S24.SHDN, S24.VDD, S25.SHDN, S25.VDD, S26.SHDN, S26.VDD, S27.SHDN, S27.VDD, S28.SHDN, S28.VDD, S29.SHDN, S29.VDD, S31.SHDN, S31.VDD, S32.SHDN, S32.VDD, S33.SHDN, S33.VDD, S34.SHDN, S34.VDD, S35.SHDN, S35.VDD, S36.SHDN, S36.VDD, S37.SHDN, S37.VDD, S38.SHDN, S38.VDD, UC4.VCC, UC5.VCC, UC6.VCC, UC7.VCC
- net GND: now also 3.3V.GND, C10.P$1, C11.P$1, C12.P$1, CN1.GND, DAISY.1, IC1.GND@1, IC1.GND@2, IC1.GND@3, IC1.GND@4, JP1.1, LED1.C, PROG0.6; no longer C10.P$2, C11.P$2, C12.P$2, C23.P$2, C24.P$2, C25.P$2, C26.P$2, C27.P$2, C28.P$2, C29.P$2, C30.P$2, C31.P$2, C32.P$2, C33.P$2, C34.P$2, C35.P$2, C36.P$2, C37.P$2, C38.P$2, C39.P$2, PROG4.6, PROG5.6, PROG6.6, PROG7.6, S17.GND, S18.GND, S19.GND, S21.GND, S22.GND, S23.GND, S24.GND, S25.GND, S26.GND, S27.GND, S28.GND, S29.GND, S31.GND, S32.GND, S33.GND, S34.GND, S35.GND, S36.GND, S37.GND, S38.GND, UC4.GND, UC4.GND@0, UC4.PA7/ADC7, UC4.PB1, UC4.PB2, UC5.GND, UC5.GND@0, UC5.PA7/ADC7, UC5.PB1, UC5.PB2, UC6.GND, UC6.GND@0, UC6.PA7/ADC7, UC6.PB1, UC6.PB2, UC7.GND, UC7.GND@0, UC7.PA7/ADC7, UC7.PB1, UC7.PB2
- net RESET0: now also PROG0.5; no longer PROG.5
- net RST40: now also PROG0.1; no longer PROG.1
- net SCL: now also IC1.PC1/OC0B/XCK0/SCL, PROG0.3, R2.1, SCL.1; no longer PROG.3, PROG4.3, PROG5.3, PROG6.3, PROG7.3, S17.SCL, S18.SCL, S19.SCL, S21.SCL, S22.SCL, S23.SCL, S24.SCL, S25.SCL, S26.SCL, S27.SCL, S28.SCL, S29.SCL, S31.SCL, S32.SCL, S33.SCL, S34.SCL, S35.SCL, S36.SCL, S37.SCL, S38.SCL, UC4.PA4/SCL, UC5.PA4/SCL, UC6.PA4/SCL, UC7.PA4/SCL
- net SDA: now also IC1.PC0/OC0A/SDA, PROG0.4, R3.1, SDA.1; no longer PROG.4, PROG4.4, PROG5.4, PROG6.4, PROG7.4, S17.SDA, S18.SDA, S19.SDA, S21.SDA, S22.SDA, S23.SDA, S24.SDA, S25.SDA, S26.SDA, S27.SDA, S28.SDA, S29.SDA, S31.SDA, S32.SDA, S33.SDA, S34.SDA, S35.SDA, S36.SDA, S37.SDA, S38.SDA, UC4.PA6/MOSI, UC5.PA6/MOSI, UC6.PA6/MOSI, UC7.PA6/MOSI

Commit message: full 8 rows with standardized naming
Parts:
- removed PROG0: (no value), nonolith:HEADER-2X3
- added (5,1), (5,2), (5,3), (5,4), (5,5), (6,1), (6,2), (6,3), (6,4), (6,5), (7,1), (7,2), (7,3), (7,4), (7,5), (8,1), (8,2), (8,3), (8,4), (8,5): MPL115A, nonolith:MPL115A
- added AT5, AT6, AT7, AT8: ATTINY24QFN, nonolith:ATTINY24QFN
- added C23, C24, C25, C26, C27, C28, C29, C30, C31, C32, C33, C34, C35, C36, C37, C38, C39, C40, C41, C42: (no value), nonolith:CAP_CERAMIC0603
- added PROG4, PROG5, PROG6, PROG7, PROG8: (no value), nonolith:HEADER-2X3
- renumbered S00 to (1,1), S01 to (2,1), S02 to (2,2), S03 to (2,3), S04 to (2,4), S05 to (2,5), S06 to (3,1), S07 to (3,2), S08 to (3,3), S09 to (3,4), S10 to (1,2), S11 to (3,5), S12 to (4,1), S13 to (4,2), S14 to (4,3), S15 to (4,4), S16 to (4,5), S20 to (1,3), S30 to (1,4), S40 to (1,5), UC0 to AT1, UC1 to AT2, UC2 to AT3, UC3 to AT4
Connections:
- net RST03 renamed RST14
- removed net RST00: (1,1).RST, AT1.PA0/ADC0
- removed net RST01: (2,1).RST, AT2.PA0/ADC0
- removed net RST02: (3,1).RST, AT3.PA0/ADC0
- removed net RST10: (1,2).RST, AT1.PA1/ADC1
- removed net RST20: (1,3).RST, AT1.PA2/ADC2
- removed net RST30: (1,4).RST, AT1.PA3/ADC3
- removed net RST40: (1,5).RST, AT1.PA5/MISO, PROG0.1
- new net ADDR04: AT5.PB0
- new net ADDR05: AT6.PB0
- new net ADDR06: AT7.PB0
- new net ADDR07: AT8.PB0
- new net CAP17: (5,3).CAP, C25.P$1
- new net CAP18: (5,4).CAP, C26.P$1
- new net CAP19: (5,5).CAP, C27.P$1
- new net CAP21: (5,1).CAP, C23.P$1
- new net CAP22: (5,2).CAP, C24.P$1
- new net CAP23: (6,3).CAP, C30.P$1
- new net CAP24: (6,4).CAP, C31.P$1
- new net CAP25: (6,5).CAP, C32.P$1
- new net CAP26: (6,1).CAP, C28.P$1
- new net CAP27: (6,2).CAP, C29.P$1
- new net CAP28: (7,3).CAP, C35.P$1
- new net CAP29: (7,4).CAP, C36.P$1
- new net CAP31: (7,5).CAP, C37.P$1
- new net CAP32: (7,1).CAP, C33.P$1
- new net CAP33: (7,2).CAP, C34.P$1
- new net CAP34: (8,3).CAP, C40.P$1
- new net CAP35: (8,4).CAP, C41.P$1
- new net CAP36: (8,5).CAP, C42.P$1
- new net CAP37: (8,1).CAP, C38.P$1
- new net CAP38: (8,2).CAP, C39.P$1
- new net RESET4: AT4.PB3/RESET, PROG4.5
- new net RESET5: AT5.PB3/RESET, PROG5.5
- new net RESET6: AT6.PB3/RESET, PROG6.5
- new net RESET7: AT7.PB3/RESET, PROG7.5
- new net RESET8: AT8.PB3/RESET, PROG8.5
- new net RST15: (5,1).RST, AT5.PA0/ADC0
- new net RST16: (6,1).RST, AT6.PA0/ADC0
- new net RST17: (7,1).RST, AT7.PA0/ADC0
- new net RST18: (8,1).RST, AT8.PA0/ADC0
- new net RST24: (4,2).RST, AT4.PA1/ADC1
- new net RST25: (5,2).RST, AT5.PA1/ADC1
- new net RST26: (6,2).RST, AT6.PA1/ADC1
- new net RST27: (7,2).RST, AT7.PA1/ADC1
- new net RST28: (8,2).RST, AT8.PA1/ADC1
- new net RST34: (4,3).RST, AT4.PA2/ADC2
- new net RST35: (5,3).RST, AT5.PA2/ADC2
- new net RST36: (6,3).RST, AT6.PA2/ADC2
- new net RST37: (7,3).RST, AT7.PA2/ADC2
- new net RST38: (8,3).RST, AT8.PA2/ADC2
- new net RST44: (4,4).RST, AT4.PA3/ADC3
- new net RST45: (5,4).RST, AT5.PA3/ADC3
- new net RST46: (6,4).RST, AT6.PA3/ADC3
- new net RST47: (7,4).RST, AT7.PA3/ADC3
- new net RST48: (8,4).RST, AT8.PA3/ADC3
- new net RST51: (1,5).RST, AT1.PA5/MISO, PROG1.1
- new net RST52: (2,5).RST, AT2.PA5/MISO, PROG2.1
- new net RST53: (3,5).RST, AT3.PA5/MISO, PROG3.1
- new net RST54: (4,5).RST, AT4.PA5/MISO, PROG4.1
- new net RST55: (5,5).RST, AT5.PA5/MISO, PROG5.1
- new net RST56: (6,5).RST, AT6.PA5/MISO, PROG6.1
- new net RST57: (7,5).RST, AT7.PA5/MISO, PROG7.1
- new net RST58: (8,5).RST, AT8.PA5/MISO, PROG8.1
- net 3.3V: now also (5,1).SHDN, (5,1).VDD, (5,2).SHDN, (5,2).VDD, (5,3).SHDN, (5,3).VDD, (5,4).SHDN, (5,4).VDD, (5,5).SHDN, (5,5).VDD, (6,1).SHDN, (6,1).VDD, (6,2).SHDN, (6,2).VDD, (6,3).SHDN, (6,3).VDD, (6,4).SHDN, (6,4).VDD, (6,5).SHDN, (6,5).VDD, (7,1).SHDN, (7,1).VDD, (7,2).SHDN, (7,2).VDD, (7,3).SHDN, (7,3).VDD, (7,4).SHDN, (7,4).VDD, (7,5).SHDN, (7,5).VDD, (8,1).SHDN, (8,1).VDD, (8,2).SHDN, (8,2).VDD, (8,3).SHDN, (8,3).VDD, (8,4).SHDN, (8,4).VDD, (8,5).SHDN, (8,5).VDD, AT5.VCC, AT6.VCC, AT7.VCC, AT8.VCC, PROG4.2, PROG5.2, PROG6.2, PROG7.2, PROG8.2; no longer PROG0.2
- net GND: now also (5,1).GND, (5,2).GND, (5,3).GND, (5,4).GND, (5,5).GND, (6,1).GND, (6,2).GND, (6,3).GND, (6,4).GND, (6,5).GND, (7,1).GND, (7,2).GND, (7,3).GND, (7,4).GND, (7,5).GND, (8,1).GND, (8,2).GND, (8,3).GND, (8,4).GND, (8,5).GND, AT5.GND, AT5.GND@0, AT5.PA7/ADC7, AT5.PB1, AT5.PB2, AT6.GND, AT6.GND@0, AT6.PA7/ADC7, AT6.PB1, AT6.PB2, AT7.GND, AT7.GND@0, AT7.PA7/ADC7, AT7.PB1, AT7.PB2, AT8.GND, AT8.GND@0, AT8.PA7/ADC7, AT8.PB1, AT8.PB2, C23.P$2, C24.P$2, C25.P$2, C26.P$2, C27.P$2, C28.P$2, C29.P$2, C30.P$2, C31.P$2, C32.P$2, C33.P$2, C34.P$2, C35.P$2, C36.P$2, C37.P$2, C38.P$2, C39.P$2, C40.P$2, C41.P$2, C42.P$2, PROG4.6, PROG5.6, PROG6.6, PROG7.6, PROG8.6; no longer PROG0.6
- net RESET0: no longer PROG0.5
- net RESET1: no longer AT2.PB3/RESET
- net RESET2: now also AT2.PB3/RESET; no longer AT3.PB3/RESET
- net RESET3: now also AT3.PB3/RESET; no longer AT4.PB3/RESET
- net RST11: now also (1,1).RST, AT1.PA0/ADC0; no longer (2,2).RST, AT2.PA1/ADC1
- net RST12: now also (2,1).RST, AT2.PA0/ADC0; no longer (3,2).RST, AT3.PA1/ADC1
- net RST13: now also (3,1).RST, AT3.PA0/ADC0; no longer (4,2).RST, AT4.PA1/ADC1
- net RST21: now also (1,2).RST, AT1.PA1/ADC1; no longer (2,3).RST, AT2.PA2/ADC2
- net RST22: now also (2,2).RST, AT2.PA1/ADC1; no longer (3,3).RST, AT3.PA2/ADC2
- net RST23: now also (3,2).RST, AT3.PA1/ADC1; no longer (4,3).RST, AT4.PA2/ADC2
- net RST31: now also (1,3).RST, AT1.PA2/ADC2; no longer (2,4).RST, AT2.PA3/ADC3
- net RST32: now also (2,3).RST, AT2.PA2/ADC2; no longer (3,4).RST, AT3.PA3/ADC3
- net RST33: now also (3,3).RST, AT3.PA2/ADC2; no longer (4,4).RST, AT4.PA3/ADC3
- net RST41: now also (1,4).RST, AT1.PA3/ADC3; no longer (2,5).RST, AT2.PA5/MISO, PROG1.1
- net RST42: now also (2,4).RST, AT2.PA3/ADC3; no longer (3,5).RST, AT3.PA5/MISO, PROG2.1
- net RST43: now also (3,4).RST, AT3.PA3/ADC3; no longer (4,5).RST, AT4.PA5/MISO, PROG3.1
- net SCL: now also (5,1).SCL, (5,2).SCL, (5,3).SCL, (5,4).SCL, (5,5).SCL, (6,1).SCL, (6,2).SCL, (6,3).SCL, (6,4).SCL, (6,5).SCL, (7,1).SCL, (7,2).SCL, (7,3).SCL, (7,4).SCL, (7,5).SCL, (8,1).SCL, (8,2).SCL, (8,3).SCL, (8,4).SCL, (8,5).SCL, AT5.PA4/SCL, AT6.PA4/SCL, AT7.PA4/SCL, AT8.PA4/SCL, PROG4.3, PROG5.3, PROG6.3, PROG7.3, PROG8.3; no longer PROG0.3
- net SDA: now also (5,1).SDA, (5,2).SDA, (5,3).SDA, (5,4).SDA, (5,5).SDA, (6,1).SDA, (6,2).SDA, (6,3).SDA, (6,4).SDA, (6,5).SDA, (7,1).SDA, (7,2).SDA, (7,3).SDA, (7,4).SDA, (7,5).SDA, (8,1).SDA, (8,2).SDA, (8,3).SDA, (8,4).SDA, (8,5).SDA, AT5.PA6/MOSI, AT6.PA6/MOSI, AT7.PA6/MOSI, AT8.PA6/MOSI, PROG4.4, PROG5.4, PROG6.4, PROG7.4, PROG8.4; no longer PROG0.4
