File: eagle/fullArray.sch (EAGLE design)
At the start: 113 parts

Commit message: now with proper address pin configurations
Connections:
- net ADDR00 renamed ADDR1
- removed net ADDR01: AT2.PB0
- removed net ADDR02: AT3.PB0
- removed net ADDR03: AT4.PB0
- removed net ADDR04: AT5.PB0
- removed net ADDR05: AT6.PB0
- removed net ADDR06: AT7.PB0
- removed net ADDR07: AT8.PB0
- new net ADDR2: AT2.PB1
- new net ADDR3: AT3.PB0, AT3.PB1
- new net ADDR4: AT4.PB2
- new net ADDR5: AT5.PB0, AT5.PB2
- new net ADDR6: AT6.PB1, AT6.PB2
- new net ADDR7: AT7.PB0, AT7.PB1, AT7.PB2
- new net ADDR8: AT8.PA7/ADC7
- net GND: now also AT2.PB0, AT4.PB0, AT6.PB0, AT8.PB0; no longer AT2.PB1, AT3.PB1, AT4.PB2, AT5.PB2, AT6.PB1, AT6.PB2, AT7.PB1, AT7.PB2, AT8.PA7/ADC7
Changed lines of the file:
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@@
 </segment>
 </net>
-<net name="ADDR00" class="0">
+<net name="ADDR1" class="0">
 <segment>
 <pinref part="AT1" gate="G$1" pin="PB0"/>
@@
 </segment>
 <segment>
-<pinref part="AT2" gate="G$1" pin="PB1"/>
-<wire x1="50.8" y1="7.62" x2="53.34" y2="7.62" width="0" layer="91"/>
-<label x="53.34" y="7.62" size="1.778" layer="95"/>
-</segment>
-<segment>
 <pinref part="AT2" gate="G$1" pin="PB2"/>
 <wire x1="50.8" y1="5.08" x2="53.34" y2="5.08" width="0" layer="91"/>
@@
 <wire x1="127" y1="5.08" x2="132.08" y2="5.08" width="0" layer="91"/>
 <label x="132.08" y="5.08" size="1.778" layer="95"/>
+</segment>
+<segment>
+<pinref part="AT2" gate="G$1" pin="PB0"/>
+<wire x1="50.8" y1="10.16" x2="53.34" y2="10.16" width="0" layer="91"/>
+<label x="53.34" y="10.16" size="1.778" layer="95"/>
 </segment>
 </net>
@@
 </segment>
 </net>
-<net name="ADDR01" class="0">
-<segment>
-<pinref part="AT2" gate="G$1" pin="PB0"/>
-<wire x1="50.8" y1="10.16" x2="53.34" y2="10.16" width="0" layer="91"/>
-<label x="53.34" y="10.16" size="1.778" layer="95"/>
-</segment>
-</net>
 <net name="RST52" class="0">
 <segment>
@@
 <pinref part="AT2" gate="G$1" pin="PA5/MISO"/>
 <pinref part="(2,5)" gate="G$1" pin="RST"/>
+</segment>
+</net>
+<net name="ADDR2" class="0">
+<segment>
+<pinref part="AT2" gate="G$1" pin="PB1"/>
+<wire x1="50.8" y1="7.62" x2="53.34" y2="7.62" width="0" layer="91"/>
+<label x="53.34" y="7.62" size="1.778" layer="95"/>
 </segment>
 </net>
@@
 <wire x1="50.8" y1="15.24" x2="53.34" y2="15.24" width="0" layer="91"/>
 <label x="53.34" y="15.24" size="1.778" layer="95"/>
-</segment>
-<segment>
-<pinref part="AT3" gate="G$1" pin="PB1"/>
-<wire x1="50.8" y1="7.62" x2="53.34" y2="7.62" width="0" layer="91"/>
-<label x="53.34" y="7.62" size="1.778" layer="95"/>
 </segment>
 <segment>
@@
 </segment>
 </net>
-<net name="ADDR02" class="0">
+<net name="ADDR3" class="0">
 <segment>
 <pinref part="AT3" gate="G$1" pin="PB0"/>
 <wire x1="50.8" y1="10.16" x2="53.34" y2="10.16" width="0" layer="91"/>
 <label x="53.34" y="10.16" size="1.778" layer="95"/>
+</segment>
+<segment>
+<pinref part="AT3" gate="G$1" pin="PB1"/>
+<wire x1="50.8" y1="7.62" x2="53.34" y2="7.62" width="0" layer="91"/>
+<label x="53.34" y="7.62" size="1.778" layer="95"/>
 </segment>
 </net>
@@
 </segment>
 <segment>
-<pinref part="AT4" gate="G$1" pin="PB2"/>
-<wire x1="50.8" y1="5.08" x2="53.34" y2="5.08" width="0" layer="91"/>
-<label x="53.34" y="5.08" size="1.778" layer="95"/>
-</segment>
-<segment>
 <pinref part="PROG4" gate="A" pin="6"/>
 <wire x1="127" y1="5.08" x2="132.08" y2="5.08" width="0" layer="91"/>
 <label x="132.08" y="5.08" size="1.778" layer="95"/>
+</segment>
+<segment>
+<pinref part="AT4" gate="G$1" pin="PB0"/>
+<wire x1="50.8" y1="10.16" x2="53.34" y2="10.16" width="0" layer="91"/>
+<label x="53.34" y="10.16" size="1.778" layer="95"/>
 </segment>
 </net>
@@
 </segment>
 </net>
-<net name="ADDR03" class="0">
-<segment>
-<pinref part="AT4" gate="G$1" pin="PB0"/>
-<wire x1="50.8" y1="10.16" x2="53.34" y2="10.16" width="0" layer="91"/>
-<label x="53.34" y="10.16" size="1.778" layer="95"/>
-</segment>
-</net>
 <net name="RESET4" class="0">
 <segment>
@@
 <wire x1="119.38" y1="10.16" x2="114.3" y2="10.16" width="0" layer="91"/>
 <label x="114.3" y="10.16" size="1.778" layer="95" rot="R180"/>
+</segment>
+</net>
+<net name="ADDR4" class="0">
+<segment>
+<pinref part="AT4" gate="G$1" pin="PB2"/>
+<wire x1="50.8" y1="5.08" x2="53.34" y2="5.08" width="0" layer="91"/>
+<label x="53.34" y="5.08" size="1.778" layer="95"/>
 </segment>
 </net>
@@
 <wire x1="50.8" y1="7.62" x2="53.34" y2="7.62" width="0" layer="91"/>
 <label x="53.34" y="7.62" size="1.778" layer="95"/>
-</segment>
-<segment>
-<pinref part="AT5" gate="G$1" pin="PB2"/>
-<wire x1="50.8" y1="5.08" x2="53.34" y2="5.08" width="0" layer="91"/>
-<label x="53.34" y="5.08" size="1.778" layer="95"/>
 </segment>
 <segment>
@@
 </segment>
 </net>
-<net name="ADDR04" class="0">
+<net name="ADDR5" class="0">
 <segment>
 <pinref part="AT5" gate="G$1" pin="PB0"/>
 <wire x1="50.8" y1="10.16" x2="53.34" y2="10.16" width="0" layer="91"/>
 <label x="53.34" y="10.16" size="1.778" layer="95"/>
+</segment>
+<segment>
+<pinref part="AT5" gate="G$1" pin="PB2"/>
+<wire x1="50.8" y1="5.08" x2="53.34" y2="5.08" width="0" layer="91"/>
+<label x="53.34" y="5.08" size="1.778" layer="95"/>
 </segment>
 </net>
@@
 </segment>
 <segment>
-<pinref part="AT6" gate="G$1" pin="PB1"/>
-<wire x1="50.8" y1="7.62" x2="53.34" y2="7.62" width="0" layer="91"/>
-<label x="53.34" y="7.62" size="1.778" layer="95"/>
-</segment>
-<segment>
-<pinref part="AT6" gate="G$1" pin="PB2"/>
-<wire x1="50.8" y1="5.08" x2="53.34" y2="5.08" width="0" layer="91"/>
-<label x="53.34" y="5.08" size="1.778" layer="95"/>
-</segment>
-<segment>
 <pinref part="PROG6" gate="A" pin="6"/>
 <wire x1="127" y1="5.08" x2="132.08" y2="5.08" width="0" layer="91"/>
 <label x="132.08" y="5.08" size="1.778" layer="95"/>
+</segment>
+<segment>
+<pinref part="AT6" gate="G$1" pin="PB0"/>
+<wire x1="50.8" y1="10.16" x2="53.34" y2="10.16" width="0" layer="91"/>
+<label x="53.34" y="10.16" size="1.778" layer="95"/>
 </segment>
 </net>
@@
 </segment>
 </net>
-<net name="ADDR05" class="0">
-<segment>
-<pinref part="AT6" gate="G$1" pin="PB0"/>
-<wire x1="50.8" y1="10.16" x2="53.34" y2="10.16" width="0" layer="91"/>
-<label x="53.34" y="10.16" size="1.778" layer="95"/>
-</segment>
-</net>
 <net name="RST56" class="0">
 <segment>
@@
 <pinref part="AT6" gate="G$1" pin="PA5/MISO"/>
 <pinref part="(6,5)" gate="G$1" pin="RST"/>
+</segment>
+</net>
+<net name="ADDR6" class="0">
+<segment>
+<pinref part="AT6" gate="G$1" pin="PB1"/>
+<wire x1="50.8" y1="7.62" x2="53.34" y2="7.62" width="0" layer="91"/>
+<label x="53.34" y="7.62" size="1.778" layer="95"/>
+</segment>
+<segment>
+<pinref part="AT6" gate="G$1" pin="PB2"/>
+<wire x1="50.8" y1="5.08" x2="53.34" y2="5.08" width="0" layer="91"/>
+<label x="53.34" y="5.08" size="1.778" layer="95"/>
 </segment>
 </net>
@@
 <wire x1="50.8" y1="15.24" x2="53.34" y2="15.24" width="0" layer="91"/>
 <label x="53.34" y="15.24" size="1.778" layer="95"/>
-</segment>
-<segment>
-<pinref part="AT7" gate="G$1" pin="PB1"/>
-<wire x1="50.8" y1="7.62" x2="53.34" y2="7.62" width="0" layer="91"/>
-<label x="53.34" y="7.62" size="1.778" layer="95"/>
-</segment>
-<segment>
-<pinref part="AT7" gate="G$1" pin="PB2"/>
-<wire x1="50.8" y1="5.08" x2="53.34" y2="5.08" width="0" layer="91"/>
-<label x="53.34" y="5.08" size="1.778" layer="95"/>
 </segment>
 <segment>
@@
 </segment>
 </net>
-<net name="ADDR06" class="0">
+<net name="ADDR7" class="0">
 <segment>
 <pinref part="AT7" gate="G$1" pin="PB0"/>
 <wire x1="50.8" y1="10.16" x2="53.34" y2="10.16" width="0" layer="91"/>
 <label x="53.34" y="10.16" size="1.778" layer="95"/>
+</segment>
+<segment>
+<pinref part="AT7" gate="G$1" pin="PB1"/>
+<wire x1="50.8" y1="7.62" x2="53.34" y2="7.62" width="0" layer="91"/>
+<label x="53.34" y="7.62" size="1.778" layer="95"/>
+</segment>
+<segment>
+<pinref part="AT7" gate="G$1" pin="PB2"/>
+<wire x1="50.8" y1="5.08" x2="53.34" y2="5.08" width="0" layer="91"/>
+<label x="53.34" y="5.08" size="1.778" layer="95"/>
 </segment>
 </net>
@@
 </segment>
 <segment>
-<pinref part="AT8" gate="G$1" pin="PA7/ADC7"/>
-<wire x1="50.8" y1="15.24" x2="53.34" y2="15.24" width="0" layer="91"/>
-<label x="53.34" y="15.24" size="1.778" layer="95"/>
-</segment>
-<segment>
 <pinref part="AT8" gate="G$1" pin="PB1"/>
 <wire x1="50.8" y1="7.62" x2="53.34" y2="7.62" width="0" layer="91"/>
@@
 </segment>
 <segment>
+<pinref part="PROG8" gate="A" pin="6"/>
+<wire x1="127" y1="5.08" x2="132.08" y2="5.08" width="0" layer="91"/>
+<label x="132.08" y="5.08" size="1.778" layer="95"/>
+</segment>
+<segment>
+<pinref part="AT8" gate="G$1" pin="PB0"/>
+<wire x1="50.8" y1="10.16" x2="53.34" y2="10.16" width="0" layer="91"/>
+<label x="53.34" y="10.16" size="1.778" layer="95"/>
+</segment>
+<segment>
 <pinref part="AT8" gate="G$1" pin="PB2"/>
 <wire x1="50.8" y1="5.08" x2="53.34" y2="5.08" width="0" layer="91"/>
 <label x="53.34" y="5.08" size="1.778" layer="95"/>
-</segment>
-<segment>
-<pinref part="PROG8" gate="A" pin="6"/>
-<wire x1="127" y1="5.08" x2="132.08" y2="5.08" width="0" layer="91"/>
-<label x="132.08" y="5.08" size="1.778" layer="95"/>
 </segment>
 </net>
@@
 </segment>
 </net>
-<net name="ADDR07" class="0">
-<segment>
-<pinref part="AT8" gate="G$1" pin="PB0"/>
-<wire x1="50.8" y1="10.16" x2="53.34" y2="10.16" width="0" layer="91"/>
-<label x="53.34" y="10.16" size="1.778" layer="95"/>
-</segment>
-</net>
+<net name="ADDR8" class="0">
+<segment>
+<pinref part="AT8" gate="G$1" pin="PA7/ADC7"/>
+<wire x1="50.8" y1="15.24" x2="53.34" y2="15.24" width="0" layer="91"/>
+<label x="53.34" y="15.24" size="1.778" layer="95"/>
+</segment>
+</net>

Commit message: fixed few ERC glitches and ADDR routing
Parts:
- R1: value (none) -> 120o
- R2, R3: value (none) -> 4.7K
- R4: value (none) -> 4.7k
Connections:
- removed net RESET0: AT1.PB3/RESET
- net RESET1: now also AT1.PB3/RESET
Changed lines of the file:
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@@
 <part name="C12" library="nonolith" deviceset="CAP_CERAMIC" device="0603" value=".01uF"/>
 <part name="PROG" library="nonolith" deviceset="HEADER-2X3" device=""/>
-<part name="R1" library="nonolith" deviceset="RESISTOR" device="0603"/>
+<part name="R1" library="nonolith" deviceset="RESISTOR" device="0603" value="120o"/>
 <part name="LED1" library="microbuilder" deviceset="LED" device="0603"/>
-<part name="R2" library="nonolith" deviceset="RESISTOR" device="0603"/>
-<part name="R3" library="nonolith" deviceset="RESISTOR" device="0603"/>
+<part name="R2" library="nonolith" deviceset="RESISTOR" device="0603" value="4.7K"/>
+<part name="R3" library="nonolith" deviceset="RESISTOR" device="0603" value="4.7K"/>
 <part name="DAISY" library="nonolith" deviceset="HEADER-1X6" device="2MM"/>
-<part name="R4" library="nonolith" deviceset="RESISTOR" device="0603"/>
+<part name="R4" library="nonolith" deviceset="RESISTOR" device="0603" value="4.7k"/>
 <part name="SCL" library="nonolith" deviceset="HEADER-1X1" device="2MM"/>
 <part name="SDA" library="nonolith" deviceset="HEADER-1X1" device="2MM"/>
@@
 <wire x1="114.3" y1="48.26" x2="127" y2="48.26" width="0" layer="91"/>
 <pinref part="SCL" gate="G$1" pin="1"/>
+<junction x="114.3" y="48.26"/>
 </segment>
 </net>
@@
 <wire x1="119.38" y1="45.72" x2="127" y2="45.72" width="0" layer="91"/>
 <pinref part="SDA" gate="G$1" pin="1"/>
+<junction x="119.38" y="45.72"/>
 </segment>
 </net>
@@
 </segment>
 </net>
-<net name="RESET0" class="0">
-<segment>
-<wire x1="50.8" y1="2.54" x2="55.88" y2="2.54" width="0" layer="91"/>
-<label x="55.88" y="2.54" size="1.778" layer="95"/>
-<pinref part="AT1" gate="G$1" pin="PB3/RESET"/>
-</segment>
-</net>
 <net name="ADDR1" class="0">
 <segment>
@@
 <label x="114.3" y="5.08" size="1.778" layer="95" rot="R180"/>
 </segment>
-</net>
+<segment>
+<wire x1="50.8" y1="2.54" x2="55.88" y2="2.54" width="0" layer="91"/>
+<label x="55.88" y="2.54" size="1.778" layer="95"/>
+<pinref part="AT1" gate="G$1" pin="PB3/RESET"/>
+</segment>
+</net>

Commit message: added values for all the things
Parts:
- C0, C1, C13, C14, C16, C17, C18, C19, C2, C20, C21, C22, C23, C24, C25, C26, C27, C28, C29, C3, C30, C31, C32, C33, C34, C35, C36, C37, C38, C39, C4, C40, C41, C42, C5, C6, C7, C8, C9: value (none) -> 1uF
- PROG: value (none) -> PROGX
- renumbered IC1 to XM1

Commit message: small tweaks to naming - filled in C15 and fixed PROGX
Parts:
- C15: value (none) -> 1uF
- PROGX: value PROGX -> (none)
- renumbered PROG to PROGX
Changed lines of the file:
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@@
 <part name="C11" library="nonolith" deviceset="CAP_CERAMIC" device="0603" value=".1uF"/>
 <part name="C12" library="nonolith" deviceset="CAP_CERAMIC" device="0603" value=".01uF"/>
-<part name="PROG" library="nonolith" deviceset="HEADER-2X3" device="" value="PROGX"/>
+<part name="PROGX" library="nonolith" deviceset="HEADER-2X3" device=""/>
 <part name="R1" library="nonolith" deviceset="RESISTOR" device="0603" value="120o"/>
 <part name="LED1" library="microbuilder" deviceset="LED" device="0603"/>
@@
 <part name="C13" library="nonolith" deviceset="CAP_CERAMIC" device="0603" value="1uF"/>
 <part name="C14" library="nonolith" deviceset="CAP_CERAMIC" device="0603" value="1uF"/>
-<part name="C15" library="nonolith" deviceset="CAP_CERAMIC" device="0603"/>
+<part name="C15" library="nonolith" deviceset="CAP_CERAMIC" device="0603" value="1uF"/>
 <part name="(3,4)" library="nonolith" deviceset="MPL115A" device=""/>
 <part name="(3,5)" library="nonolith" deviceset="MPL115A" device=""/>
@@
 <instance part="C11" gate="G$1" x="22.86" y="60.96"/>
 <instance part="C12" gate="G$1" x="33.02" y="60.96"/>
-<instance part="PROG" gate="A" x="149.86" y="63.5" rot="R90"/>
+<instance part="PROGX" gate="A" x="149.86" y="63.5" rot="R90"/>
 <instance part="R1" gate="G$1" x="116.84" y="81.28"/>
 <instance part="LED1" gate="G$1" x="129.54" y="81.28"/>
@@
 </segment>
 <segment>
-<pinref part="PROG" gate="A" pin="6"/>
+<pinref part="PROGX" gate="A" pin="6"/>
 <wire x1="152.4" y1="68.58" x2="152.4" y2="73.66" width="0" layer="91"/>
 <label x="152.4" y="73.66" size="1.778" layer="95" rot="R90"/>
@@
 </segment>
 <segment>
-<pinref part="PROG" gate="A" pin="2"/>
+<pinref part="PROGX" gate="A" pin="2"/>
 <wire x1="147.32" y1="68.58" x2="147.32" y2="73.66" width="0" layer="91"/>
 <label x="147.32" y="73.66" size="1.778" layer="95" rot="R90"/>
@@
 </segment>
 <segment>
-<pinref part="PROG" gate="A" pin="3"/>
+<pinref part="PROGX" gate="A" pin="3"/>
 <wire x1="149.86" y1="60.96" x2="149.86" y2="55.88" width="0" layer="91"/>
 <label x="149.86" y="55.88" size="1.778" layer="95" rot="R270"/>
@@
 </segment>
 <segment>
-<pinref part="PROG" gate="A" pin="4"/>
+<pinref part="PROGX" gate="A" pin="4"/>
 <wire x1="149.86" y1="68.58" x2="149.86" y2="73.66" width="0" layer="91"/>
 <label x="149.86" y="73.66" size="1.778" layer="95" rot="R90"/>
@@
 </segment>
 <segment>
-<pinref part="PROG" gate="A" pin="1"/>
+<pinref part="PROGX" gate="A" pin="1"/>
 <wire x1="147.32" y1="60.96" x2="147.32" y2="55.88" width="0" layer="91"/>
 <label x="147.32" y="55.88" size="1.778" layer="95" rot="R270"/>
@@
 </segment>
 <segment>
-<pinref part="PROG" gate="A" pin="5"/>
+<pinref part="PROGX" gate="A" pin="5"/>
 <wire x1="152.4" y1="60.96" x2="152.4" y2="55.88" width="0" layer="91"/>
 <label x="152.4" y="55.88" size="1.778" layer="95" rot="R270"/>
