File: eagle/fullArray.sch (EAGLE design)
At the start: 113 parts

Commit message: updated to match nonolith.lbr
Parts:
- (1,1), (1,2), (1,3), (1,4), (1,5), (2,1), (2,2), (2,3), (2,4), (2,5), (3,1), (3,2), (3,3), (3,4), (3,5), (4,1), (4,2), (4,3), (4,4), (4,5), (5,1), (5,2), (5,3), (5,4), (5,5), (6,1), (6,2), (6,3), (6,4), (6,5), (7,1), (7,2), (7,3), (7,4), (7,5), (8,1), (8,2), (8,3), (8,4), (8,5): value MPL115A -> MPL115A2; device nonolith:MPL115A -> nonolith:MPL115A2
- AT1, AT2, AT3, AT4, AT5, AT6, AT7, AT8: value ATTINY24QFN -> ATTINYX4AMMH; device nonolith:ATTINY24QFN -> nonolith:ATTINYX4AMMH

Commit message: part not MMH, part MH
Parts:
- AT1, AT2, AT3, AT4, AT5, AT6, AT7, AT8: value ATTINYX4AMMH -> ATTINYX4AMH; device nonolith:ATTINYX4AMMH -> nonolith:ATTINYX4AMH
Changed lines of the file:
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@@
 <part name="JP1" library="nonolith" deviceset="HEADER-1X1" device="2MM"/>
 <part name="JP2" library="nonolith" deviceset="HEADER-1X1" device="2MM"/>
-<part name="AT1" library="nonolith" deviceset="ATTINYX4A" device="MMH"/>
+<part name="AT1" library="nonolith" deviceset="ATTINYX4A" device="MH"/>
 <part name="(1,1)" library="nonolith" deviceset="MPL115A2" device=""/>
 <part name="(1,2)" library="nonolith" deviceset="MPL115A2" device=""/>
@@
 <part name="C4" library="nonolith" deviceset="CAP_CERAMIC" device="0603" value="1uF"/>
 <part name="PROG1" library="nonolith" deviceset="HEADER-2X3" device=""/>
-<part name="AT2" library="nonolith" deviceset="ATTINYX4A" device="MMH"/>
+<part name="AT2" library="nonolith" deviceset="ATTINYX4A" device="MH"/>
 <part name="(2,1)" library="nonolith" deviceset="MPL115A2" device=""/>
 <part name="(2,2)" library="nonolith" deviceset="MPL115A2" device=""/>
@@
 <part name="C9" library="nonolith" deviceset="CAP_CERAMIC" device="0603" value="1uF"/>
 <part name="PROG2" library="nonolith" deviceset="HEADER-2X3" device=""/>
-<part name="AT3" library="nonolith" deviceset="ATTINYX4A" device="MMH"/>
+<part name="AT3" library="nonolith" deviceset="ATTINYX4A" device="MH"/>
 <part name="(3,1)" library="nonolith" deviceset="MPL115A2" device=""/>
 <part name="(3,2)" library="nonolith" deviceset="MPL115A2" device=""/>
@@
 <part name="C17" library="nonolith" deviceset="CAP_CERAMIC" device="0603" value="1uF"/>
 <part name="PROG3" library="nonolith" deviceset="HEADER-2X3" device=""/>
-<part name="AT4" library="nonolith" deviceset="ATTINYX4A" device="MMH"/>
+<part name="AT4" library="nonolith" deviceset="ATTINYX4A" device="MH"/>
 <part name="(4,1)" library="nonolith" deviceset="MPL115A2" device=""/>
 <part name="(4,2)" library="nonolith" deviceset="MPL115A2" device=""/>
@@
 <part name="C22" library="nonolith" deviceset="CAP_CERAMIC" device="0603" value="1uF"/>
 <part name="PROG4" library="nonolith" deviceset="HEADER-2X3" device=""/>
-<part name="AT5" library="nonolith" deviceset="ATTINYX4A" device="MMH"/>
+<part name="AT5" library="nonolith" deviceset="ATTINYX4A" device="MH"/>
 <part name="(5,1)" library="nonolith" deviceset="MPL115A2" device=""/>
 <part name="(5,2)" library="nonolith" deviceset="MPL115A2" device=""/>
@@
 <part name="C27" library="nonolith" deviceset="CAP_CERAMIC" device="0603" value="1uF"/>
 <part name="PROG5" library="nonolith" deviceset="HEADER-2X3" device=""/>
-<part name="AT6" library="nonolith" deviceset="ATTINYX4A" device="MMH"/>
+<part name="AT6" library="nonolith" deviceset="ATTINYX4A" device="MH"/>
 <part name="(6,1)" library="nonolith" deviceset="MPL115A2" device=""/>
 <part name="(6,2)" library="nonolith" deviceset="MPL115A2" device=""/>
@@
 <part name="C32" library="nonolith" deviceset="CAP_CERAMIC" device="0603" value="1uF"/>
 <part name="PROG6" library="nonolith" deviceset="HEADER-2X3" device=""/>
-<part name="AT7" library="nonolith" deviceset="ATTINYX4A" device="MMH"/>
+<part name="AT7" library="nonolith" deviceset="ATTINYX4A" device="MH"/>
 <part name="(7,1)" library="nonolith" deviceset="MPL115A2" device=""/>
 <part name="(7,2)" library="nonolith" deviceset="MPL115A2" device=""/>
@@
 <part name="C37" library="nonolith" deviceset="CAP_CERAMIC" device="0603" value="1uF"/>
 <part name="PROG7" library="nonolith" deviceset="HEADER-2X3" device=""/>
-<part name="AT8" library="nonolith" deviceset="ATTINYX4A" device="MMH"/>
+<part name="AT8" library="nonolith" deviceset="ATTINYX4A" device="MH"/>
 <part name="(8,1)" library="nonolith" deviceset="MPL115A2" device=""/>
 <part name="(8,2)" library="nonolith" deviceset="MPL115A2" device=""/>

Commit message: change cell indexing from 2d to 1d
Parts:
- renumbered (1,1) to 0, (1,2) to 1, (1,3) to 2, (1,4) to 3, (1,5) to 4, (2,1) to 5, (2,2) to 6, (2,3) to 7, (2,4) to 8, (2,5) to 9, (3,1) to 10, (3,2) to 11, (3,3) to 12, (3,4) to 13, (3,5) to 14, (4,1) to 15, (4,2) to 16, (4,3) to 17, (4,4) to 18, (4,5) to 19, (5,1) to 20, (5,2) to 21, (5,3) to 22, (5,4) to 23, (5,5) to 24, (6,1) to 25, (6,2) to 26, (6,3) to 27, (6,4) to 28, (6,5) to 29, (7,1) to 30, (7,2) to 31, (7,3) to 32, (7,4) to 33, (7,5) to 34, (8,1) to 35, (8,2) to 36, (8,3) to 37, (8,4) to 38, (8,5) to 39

Commit message: redo power section and host interface part of board
Parts:
- added C43: (no value), microbuilder:CAP_TANTALUMD/7343_REFLOW
- 3.3V: value VREG -> VREGAP1117; device nonolith:VREG -> nonolith:VREGAP1117
Connections:
- net 3.3V: now also C43.+
- net GND: now also C43.-; no longer AT1.GND@0, AT2.GND@0, AT3.GND@0, AT4.GND@0, AT5.GND@0, AT6.GND@0, AT7.GND@0, AT8.GND@0
Changed lines of the file:
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@@
 <?xml version="1.0" encoding="utf-8"?>
 <!DOCTYPE eagle SYSTEM "eagle.dtd">
-<eagle version="6.1">
+<eagle version="6.3">
 <drawing>
 <settings>
@@
 <part name="XM1" library="nonolith" deviceset="ATXMEGAXXA4U" device="-MH"/>
 <part name="CN1" library="nonolith" deviceset="USB" device="MICROB"/>
-<part name="3.3V" library="nonolith" deviceset="VREG" device=""/>
+<part name="3.3V" library="nonolith" deviceset="VREG" device="AP1117"/>
 <part name="C10" library="nonolith" deviceset="CAP_CERAMIC" device="0603" value="1uF"/>
 <part name="C11" library="nonolith" deviceset="CAP_CERAMIC" device="0603" value=".1uF"/>
@@
 <part name="C42" library="nonolith" deviceset="CAP_CERAMIC" device="0603" value="1uF"/>
 <part name="PROG8" library="nonolith" deviceset="HEADER-2X3" device=""/>
+<part name="C43" library="microbuilder" deviceset="CAP_TANTALUM" device="D/7343_REFLOW"/>
 </parts>
 <sheets>
@@
 <instance part="JP1" gate="G$1" x="124.46" y="43.18" rot="R180"/>
 <instance part="JP2" gate="G$1" x="124.46" y="40.64" rot="R180"/>
+<instance part="C43" gate="G$1" x="-5.08" y="38.1" rot="R180"/>
 </instances>
 <busses>
@@
 <wire x1="22.86" y1="73.66" x2="12.7" y2="73.66" width="0" layer="91"/>
 <wire x1="12.7" y1="73.66" x2="5.08" y2="73.66" width="0" layer="91"/>
-<wire x1="5.08" y1="73.66" x2="5.08" y2="40.64" width="0" layer="91"/>
+<wire x1="5.08" y1="73.66" x2="5.08" y2="43.18" width="0" layer="91"/>
 <junction x="43.18" y="78.74"/>
 <junction x="43.18" y="76.2"/>
 <junction x="43.18" y="73.66"/>
 <pinref part="C10" gate="G$1" pin="P$1"/>
+<wire x1="5.08" y1="43.18" x2="5.08" y2="40.64" width="0" layer="91"/>
 <wire x1="12.7" y1="73.66" x2="12.7" y2="66.04" width="0" layer="91"/>
 <pinref part="C11" gate="G$1" pin="P$1"/>
@@
 <junction x="12.7" y="73.66"/>
 <label x="5.08" y="73.66" size="1.778" layer="95" rot="R180"/>
+<pinref part="C43" gate="G$1" pin="-"/>
+<wire x1="-5.08" y1="40.64" x2="-5.08" y2="43.18" width="0" layer="91"/>
+<wire x1="-5.08" y1="43.18" x2="5.08" y2="43.18" width="0" layer="91"/>
+<junction x="5.08" y="43.18"/>
 </segment>
 <segment>
@@
 <junction x="33.02" y="50.8"/>
 <label x="2.54" y="50.8" size="1.778" layer="95" rot="R180"/>
+<pinref part="C43" gate="G$1" pin="+"/>
+<wire x1="-5.08" y1="33.02" x2="2.54" y2="33.02" width="0" layer="91"/>
+<wire x1="2.54" y1="33.02" x2="2.54" y2="35.56" width="0" layer="91"/>
 </segment>
 <segment>
@@
 <segment>
 <wire x1="10.16" y1="5.08" x2="7.62" y2="5.08" width="0" layer="91"/>
-<wire x1="10.16" y1="2.54" x2="7.62" y2="2.54" width="0" layer="91"/>
 <wire x1="7.62" y1="5.08" x2="7.62" y2="2.54" width="0" layer="91"/>
 <label x="7.62" y="2.54" size="1.778" layer="95" rot="R180"/>
 <pinref part="AT1" gate="G$1" pin="GND"/>
-<pinref part="AT1" gate="G$1" pin="GND@0"/>
 </segment>
 <segment>
@@
 <segment>
 <wire x1="10.16" y1="5.08" x2="7.62" y2="5.08" width="0" layer="91"/>
-<wire x1="10.16" y1="2.54" x2="7.62" y2="2.54" width="0" layer="91"/>
 <wire x1="7.62" y1="5.08" x2="7.62" y2="2.54" width="0" layer="91"/>
 <label x="7.62" y="2.54" size="1.778" layer="95" rot="R180"/>
 <pinref part="AT2" gate="G$1" pin="GND"/>
-<pinref part="AT2" gate="G$1" pin="GND@0"/>
 </segment>
 <segment>
@@
 <segment>
 <wire x1="10.16" y1="5.08" x2="7.62" y2="5.08" width="0" layer="91"/>
-<wire x1="10.16" y1="2.54" x2="7.62" y2="2.54" width="0" layer="91"/>
 <wire x1="7.62" y1="5.08" x2="7.62" y2="2.54" width="0" layer="91"/>
 <label x="7.62" y="2.54" size="1.778" layer="95" rot="R180"/>
 <pinref part="AT3" gate="G$1" pin="GND"/>
-<pinref part="AT3" gate="G$1" pin="GND@0"/>
 </segment>
 <segment>
@@
 <segment>
 <wire x1="10.16" y1="5.08" x2="7.62" y2="5.08" width="0" layer="91"/>
-<wire x1="10.16" y1="2.54" x2="7.62" y2="2.54" width="0" layer="91"/>
 <wire x1="7.62" y1="5.08" x2="7.62" y2="2.54" width="0" layer="91"/>
 <label x="7.62" y="2.54" size="1.778" layer="95" rot="R180"/>
 <pinref part="AT4" gate="G$1" pin="GND"/>
-<pinref part="AT4" gate="G$1" pin="GND@0"/>
 </segment>
 <segment>
@@
 <segment>
 <wire x1="10.16" y1="5.08" x2="7.62" y2="5.08" width="0" layer="91"/>
-<wire x1="10.16" y1="2.54" x2="7.62" y2="2.54" width="0" layer="91"/>
 <wire x1="7.62" y1="5.08" x2="7.62" y2="2.54" width="0" layer="91"/>
 <label x="7.62" y="2.54" size="1.778" layer="95" rot="R180"/>
 <pinref part="AT5" gate="G$1" pin="GND"/>
-<pinref part="AT5" gate="G$1" pin="GND@0"/>
 </segment>
 <segment>
@@
 <segment>
 <wire x1="10.16" y1="5.08" x2="7.62" y2="5.08" width="0" layer="91"/>
-<wire x1="10.16" y1="2.54" x2="7.62" y2="2.54" width="0" layer="91"/>
 <wire x1="7.62" y1="5.08" x2="7.62" y2="2.54" width="0" layer="91"/>
 <label x="7.62" y="2.54" size="1.778" layer="95" rot="R180"/>
 <pinref part="AT6" gate="G$1" pin="GND"/>
-<pinref part="AT6" gate="G$1" pin="GND@0"/>
 </segment>
 <segment>
@@
 <segment>
 <wire x1="10.16" y1="5.08" x2="7.62" y2="5.08" width="0" layer="91"/>
-<wire x1="10.16" y1="2.54" x2="7.62" y2="2.54" width="0" layer="91"/>
 <wire x1="7.62" y1="5.08" x2="7.62" y2="2.54" width="0" layer="91"/>
 <label x="7.62" y="2.54" size="1.778" layer="95" rot="R180"/>
 <pinref part="AT7" gate="G$1" pin="GND"/>
-<pinref part="AT7" gate="G$1" pin="GND@0"/>
 </segment>
 <segment>
@@
 <segment>
 <wire x1="10.16" y1="5.08" x2="7.62" y2="5.08" width="0" layer="91"/>
-<wire x1="10.16" y1="2.54" x2="7.62" y2="2.54" width="0" layer="91"/>
 <wire x1="7.62" y1="5.08" x2="7.62" y2="2.54" width="0" layer="91"/>
 <label x="7.62" y="2.54" size="1.778" layer="95" rot="R180"/>
 <pinref part="AT8" gate="G$1" pin="GND"/>
-<pinref part="AT8" gate="G$1" pin="GND@0"/>
-</segment>
-<segment>
+</segment>
+<segment>

Commit message: add 1206 decoupling capacitor to 5v0 supply
Parts:
- added C44: 10uF, nonolith:CAP_CERAMIC1206
- C43: value (none) -> 470uF
Connections:
- net 5V: now also C44.P$2
- net GND: now also C44.P$1
Changed lines of the file:
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@@
 <part name="C42" library="nonolith" deviceset="CAP_CERAMIC" device="0603" value="1uF"/>
 <part name="PROG8" library="nonolith" deviceset="HEADER-2X3" device=""/>
-<part name="C43" library="microbuilder" deviceset="CAP_TANTALUM" device="D/7343_REFLOW"/>
+<part name="C43" library="microbuilder" deviceset="CAP_TANTALUM" device="D/7343_REFLOW" value="470uF"/>
+<part name="C44" library="nonolith" deviceset="CAP_CERAMIC" device="1206" value="10uF"/>
 </parts>
 <sheets>
@@
 <instance part="JP2" gate="G$1" x="124.46" y="40.64" rot="R180"/>
 <instance part="C43" gate="G$1" x="-5.08" y="38.1" rot="R180"/>
+<instance part="C44" gate="G$1" x="22.86" y="27.94" rot="R180"/>
 </instances>
 <busses>
@@
 <label x="132.08" y="43.18" size="1.778" layer="95"/>
 </segment>
+<segment>
+<pinref part="C44" gate="G$1" pin="P$1"/>
+<wire x1="22.86" y1="22.86" x2="20.32" y2="22.86" width="0" layer="91"/>
+<label x="20.32" y="22.86" size="1.778" layer="95" rot="R180"/>
+</segment>
 </net>
 <net name="3.3V" class="0">
@@
 <pinref part="3.3V" gate="G$1" pin="VIN"/>
 <wire x1="25.4" y1="38.1" x2="27.94" y2="38.1" width="0" layer="91"/>
-<wire x1="27.94" y1="38.1" x2="27.94" y2="12.7" width="0" layer="91"/>
+<wire x1="27.94" y1="38.1" x2="27.94" y2="30.48" width="0" layer="91"/>
 <pinref part="CN1" gate="G$1" pin="VBUS"/>
+<wire x1="27.94" y1="30.48" x2="27.94" y2="12.7" width="0" layer="91"/>
 <wire x1="27.94" y1="12.7" x2="20.32" y2="12.7" width="0" layer="91"/>
 <label x="27.94" y="38.1" size="1.778" layer="95"/>
-</segment>
-<segment>
+<pinref part="C44" gate="G$1" pin="P$2"/>
+<wire x1="22.86" y1="30.48" x2="27.94" y2="30.48" width="0" layer="91"/>
+<junction x="27.94" y="30.48"/>
+</segment>
+<segment>

Commit message: need to tweak address pins, but should be manufacturable
Parts:
- removed 0, 1, 2, 3, 4, 5, 6, 7, 8, 9: MPL115A2, nonolith:MPL115A2
- removed AT1, AT2, AT3, AT4, AT5, AT6, AT7, AT8: ATTINYX4AMH, nonolith:ATTINYX4AMH
- removed C0, C1, C2, C3, C4, C5, C7, C8, C9: 1uF, nonolith:CAP_CERAMIC0603
- removed PROG1, PROG2, PROG3, PROG4, PROG5, PROG6, PROG7, PROG8: (no value), nonolith:HEADER-2X3
- added 01, 02, 03, 04, 05, 06, 07, 08, 09, 40: MPL115A, nonolith:MPL115A
- added C01, C02, C03, C04, C05, C07, C08, C09, C45, C46, C47, C48, C49, C50, C51: (no value), nonolith:CAP_CERAMIC0402
- added C52: 470uF, microbuilder:CAP_TANTALUMD/7343_REFLOW
- added C53: 10uF, nonolith:CAP_CERAMIC1206
- added UC01, UC02, UC03, UC04, UC05, UC06, UC07, UC08: ATTINY24QFN, nonolith:ATTINY24QFN
- 10, 11, 12, 13, 14, 15, 16, 17, 18, 19, 20, 21, 22, 23, 24, 25, 26, 27, 28, 29, 30, 31, 32, 33, 34, 35, 36, 37, 38, 39: value MPL115A2 -> MPL115A; device nonolith:MPL115A2 -> nonolith:MPL115A
- C13, C14, C15, C16, C17, C18, C19, C20, C21, C22, C23, C24, C25, C26, C27, C28, C29, C30, C31, C32, C33, C34, C35, C36, C37, C38, C39, C40, C41, C42, C6: value 1uF -> (none); device nonolith:CAP_CERAMIC0603 -> nonolith:CAP_CERAMIC0402
- C43: value 470uF -> (none); device microbuilder:CAP_TANTALUMD/7343_REFLOW -> nonolith:CAP_CERAMIC0402
- C44: value 10uF -> (none); device nonolith:CAP_CERAMIC1206 -> nonolith:CAP_CERAMIC0402
Connections:
- removed net ADDR1: AT1.PB0
- removed net ADDR2: AT2.PB1
- removed net ADDR3: AT3.PB0, AT3.PB1
- removed net ADDR4: AT4.PB2
- removed net ADDR5: AT5.PB0, AT5.PB2
- removed net ADDR6: AT6.PB1, AT6.PB2
- removed net ADDR7: AT7.PB0, AT7.PB1, AT7.PB2
- removed net ADDR8: AT8.PA7/ADC7
- removed net CAP00: 0.CAP, C0.P$1
- removed net RESET1: AT1.PB3/RESET, PROG1.5
- removed net RESET2: AT2.PB3/RESET, PROG2.5
- removed net RESET3: AT3.PB3/RESET, PROG3.5
- removed net RESET4: AT4.PB3/RESET, PROG4.5
- removed net RESET5: AT5.PB3/RESET, PROG5.5
- removed net RESET6: AT6.PB3/RESET, PROG6.5
- removed net RESET7: AT7.PB3/RESET, PROG7.5
- removed net RESET8: AT8.PB3/RESET, PROG8.5
- removed net RST18: 35.RST, AT8.PA0/ADC0
- removed net RST41: 3.RST, AT1.PA3/ADC3
- removed net RST42: 8.RST, AT2.PA3/ADC3
- removed net RST43: 13.RST, AT3.PA3/ADC3
- removed net RST44: 18.RST, AT4.PA3/ADC3
- removed net RST45: 23.RST, AT5.PA3/ADC3
- removed net RST46: 28.RST, AT6.PA3/ADC3
- removed net RST47: 33.RST, AT7.PA3/ADC3
- removed net RST48: 38.RST, AT8.PA3/ADC3
- removed net RST51: 4.RST, AT1.PA5/MISO, PROG1.1
- removed net RST52: 9.RST, AT2.PA5/MISO, PROG2.1
- removed net RST53: 14.RST, AT3.PA5/MISO, PROG3.1
- removed net RST54: 19.RST, AT4.PA5/MISO, PROG4.1
- removed net RST55: 24.RST, AT5.PA5/MISO, PROG5.1
- removed net RST56: 29.RST, AT6.PA5/MISO, PROG6.1
- removed net RST57: 34.RST, AT7.PA5/MISO, PROG7.1
- removed net RST58: 39.RST, AT8.PA5/MISO, PROG8.1
- new net ADDR00: UC01.PB0, UC02.PB0, UC03.PB0, UC04.PB0, UC05.PB0, UC06.PB0, UC07.PB0, UC08.PB0
- new net CAP39: 36.CAP, C46.P$1
- new net RESET01: UC01.PB3/RESET
- new net RESET02: UC02.PB3/RESET
- new net RESET03: UC03.PB3/RESET
- new net RESET04: UC04.PB3/RESET
- new net RESET05: UC05.PB3/RESET
- new net RESET06: UC06.PB3/RESET, UC07.PB3/RESET
- new net RESET08: UC08.PB3/RESET
- new net RST01: 01.RST, UC01.PA0/ADC0
- new net RST018: 18.RST, UC04.PA2/ADC2
- new net RST02: 02.RST, UC01.PA1/ADC1
- new net RST03: 03.RST, UC01.PA2/ADC2
- new net RST04: 04.RST, UC01.PA3/ADC3
- new net RST05: 05.RST, UC01.PA5/MISO
- new net RST06: 06.RST, UC02.PA0/ADC0
- new net RST07: 07.RST, UC02.PA1/ADC1
- new net RST08: 08.RST, UC02.PA2/ADC2
- new net RST09: 09.RST, UC02.PA3/ADC3
- new net RST10: 10.RST, UC02.PA5/MISO
- new net RST19: 19.RST, UC04.PA3/ADC3
- new net RST20: 20.RST, UC04.PA5/MISO
- new net RST29: 29.RST, UC06.PA3/ADC3
- new net RST30: 30.RST, UC06.PA5/MISO
- new net RST39: 39.RST, UC08.PA3/ADC3
- new net RST40: 40.RST, UC08.PA5/MISO
- net 3.3V: now also 01.SHDN, 01.VDD, 02.SHDN, 02.VDD, 03.SHDN, 03.VDD, 04.SHDN, 04.VDD, 05.SHDN, 05.VDD, 06.SHDN, 06.VDD, 07.SHDN, 07.VDD, 08.SHDN, 08.VDD, 09.SHDN, 09.VDD, 40.SHDN, 40.VDD, C15.P$1, C21.P$1, C27.P$1, C33.P$1, C39.P$1, C45.P$1, C51.P$1, C52.+, C6.P$1, UC01.VCC, UC02.VCC, UC03.VCC, UC04.VCC, UC05.VCC, UC06.VCC, UC07.VCC, UC08.VCC; no longer 0.SHDN, 0.VDD, 1.SHDN, 1.VDD, 2.SHDN, 2.VDD, 3.SHDN, 3.VDD, 4.SHDN, 4.VDD, 5.SHDN, 5.VDD, 6.SHDN, 6.VDD, 7.SHDN, 7.VDD, 8.SHDN, 8.VDD, 9.SHDN, 9.VDD, AT1.VCC, AT2.VCC, AT3.VCC, AT4.VCC, AT5.VCC, AT6.VCC, AT7.VCC, AT8.VCC, C43.+, PROG1.2, PROG2.2, PROG3.2, PROG4.2, PROG5.2, PROG6.2, PROG7.2, PROG8.2
- net 5V: now also C53.P$2; no longer C44.P$2
- net CAP01: now also 01.CAP, C01.P$1; no longer 7.CAP, C7.P$1
- net CAP02: now also 02.CAP, C02.P$1; no longer 8.CAP, C8.P$1
- net CAP03: now also 03.CAP, C03.P$1; no longer 9.CAP, C9.P$1
- net CAP04: now also 04.CAP, C04.P$1; no longer 5.CAP, C5.P$1
- net CAP05: now also 05.CAP, C05.P$1; no longer 6.CAP, C6.P$1
- net CAP06: now also 08.CAP, C09.P$1; no longer 12.CAP, C15.P$1
- net CAP07: now also 09.CAP, C13.P$1; no longer 13.CAP, C16.P$1
- net CAP08: now also 10.CAP, C14.P$1; no longer 14.CAP, C17.P$1
- net CAP09: now also 06.CAP, C07.P$1; no longer 10.CAP, C13.P$1
- net CAP10: now also 07.CAP, C08.P$1; no longer 1.CAP, C1.P$1
- net CAP11: now also 13.CAP, C18.P$1; no longer 11.CAP, C14.P$1
- net CAP12: now also 14.CAP, C19.P$1; no longer 17.CAP, C20.P$1
- net CAP13: now also 15.CAP, C20.P$1; no longer 18.CAP, C21.P$1
- net CAP14: now also 11.CAP, C16.P$1; no longer 19.CAP, C22.P$1
- net CAP15: now also 12.CAP, C17.P$1; no longer 15.CAP, C18.P$1
- net CAP16: now also 18.CAP, C24.P$1; no longer 16.CAP, C19.P$1
- net CAP17: now also 19.CAP; no longer 22.CAP
- net CAP18: now also 20.CAP; no longer 23.CAP
- net CAP19: now also 16.CAP, C22.P$1; no longer 24.CAP, C27.P$1
- net CAP20: now also 17.CAP, C23.P$1; no longer 2.CAP, C2.P$1
- net CAP21: now also 23.CAP, C30.P$1; no longer 20.CAP, C23.P$1
- net CAP22: now also 24.CAP, C31.P$1; no longer 21.CAP, C24.P$1
- net CAP23: now also 25.CAP, C32.P$1; no longer 27.CAP, C30.P$1
- net CAP24: now also 21.CAP, C28.P$1; no longer 28.CAP, C31.P$1
- net CAP25: now also 22.CAP, C29.P$1; no longer 29.CAP, C32.P$1
- net CAP26: now also 28.CAP, C36.P$1; no longer 25.CAP, C28.P$1
- net CAP27: now also 29.CAP, C37.P$1; no longer 26.CAP, C29.P$1
- net CAP28: now also 30.CAP, C38.P$1; no longer 32.CAP, C35.P$1
- net CAP29: now also 26.CAP, C34.P$1; no longer 33.CAP, C36.P$1
- net CAP30: now also 27.CAP, C35.P$1; no longer 3.CAP, C3.P$1
- net CAP31: now also 33.CAP, C42.P$1; no longer 34.CAP, C37.P$1
- net CAP32: now also 34.CAP, C43.P$1; no longer 30.CAP, C33.P$1
- net CAP33: now also 35.CAP, C44.P$1; no longer 31.CAP, C34.P$1
- net CAP34: now also 31.CAP; no longer 37.CAP
- net CAP35: now also 32.CAP; no longer 38.CAP
- net CAP36: now also 38.CAP, C48.P$1; no longer 39.CAP, C42.P$1
- net CAP37: now also 39.CAP, C49.P$1; no longer 35.CAP, C38.P$1
- net CAP38: now also 40.CAP, C50.P$1; no longer 36.CAP, C39.P$1
- net CAP40: now also 37.CAP, C47.P$1; no longer 4.CAP, C4.P$1
- net GND: now also 01.GND, 02.GND, 03.GND, 04.GND, 05.GND, 06.GND, 07.GND, 08.GND, 09.GND, 40.GND, C01.P$2, C02.P$2, C03.P$2, C04.P$2, C05.P$2, C07.P$2, C08.P$2, C09.P$2, C43.P$2, C44.P$2, C45.P$2, C46.P$2, C47.P$2, C48.P$2, C49.P$2, C50.P$2, C51.P$2, C52.-, C53.P$1, UC01.GND, UC01.GND@0, UC01.PA7/ADC7, UC01.PB1, UC01.PB2, UC02.GND, UC02.GND@0, UC02.PA7/ADC7, UC02.PB1, UC02.PB2, UC03.GND, UC03.GND@0, UC03.PA7/ADC7, UC03.PB1, UC03.PB2, UC04.GND, UC04.GND@0, UC04.PA7/ADC7, UC04.PB1, UC04.PB2, UC05.GND, UC05.GND@0, UC05.PA7/ADC7, UC05.PB1, UC05.PB2, UC06.GND, UC06.GND@0, UC06.PA7/ADC7, UC06.PB1, UC06.PB2, UC07.GND, UC07.GND@0, UC07.PA7/ADC7, UC07.PB1, UC07.PB2, UC08.GND, UC08.GND@0, UC08.PA7/ADC7, UC08.PB1, UC08.PB2; no longer 0.GND, 1.GND, 2.GND, 3.GND, 4.GND, 5.GND, 6.GND, 7.GND, 8.GND, 9.GND, AT1.GND, AT1.PA7/ADC7, AT1.PB1, AT1.PB2, AT2.GND, AT2.PA7/ADC7, AT2.PB0, AT2.PB2, AT3.GND, AT3.PA7/ADC7, AT3.PB2, AT4.GND, AT4.PA7/ADC7, AT4.PB0, AT4.PB1, AT5.GND, AT5.PA7/ADC7, AT5.PB1, AT6.GND, AT6.PA7/ADC7, AT6.PB0, AT7.GND, AT7.PA7/ADC7, AT8.GND, AT8.PB0, AT8.PB1, AT8.PB2, C0.P$2, C1.P$2, C2.P$2, C3.P$2, C4.P$2, C43.-, C44.P$1, C5.P$2, C7.P$2, C8.P$2, C9.P$2, PROG1.6, PROG2.6, PROG3.6, PROG4.6, PROG5.6, PROG6.6, PROG7.6, PROG8.6
- net RST11: now also 11.RST, UC03.PA0/ADC0; no longer 0.RST, AT1.PA0/ADC0
- net RST12: now also 12.RST, UC03.PA1/ADC1; no longer 5.RST, AT2.PA0/ADC0
- net RST13: now also 13.RST, UC03.PA2/ADC2; no longer 10.RST, AT3.PA0/ADC0
- net RST14: now also 14.RST, UC03.PA3/ADC3; no longer 15.RST, AT4.PA0/ADC0
- net RST15: now also 15.RST, UC03.PA5/MISO; no longer 20.RST, AT5.PA0/ADC0
- net RST16: now also 16.RST, UC04.PA0/ADC0; no longer 25.RST, AT6.PA0/ADC0
- net RST17: now also 17.RST, UC04.PA1/ADC1; no longer 30.RST, AT7.PA0/ADC0
- net RST21: now also 21.RST, UC05.PA0/ADC0; no longer 1.RST, AT1.PA1/ADC1
- net RST22: now also 22.RST, UC05.PA1/ADC1; no longer 6.RST, AT2.PA1/ADC1
- net RST23: now also 23.RST, UC05.PA2/ADC2; no longer 11.RST, AT3.PA1/ADC1
- net RST24: now also 24.RST, UC05.PA3/ADC3; no longer 16.RST, AT4.PA1/ADC1
- net RST25: now also 25.RST, UC05.PA5/MISO; no longer 21.RST, AT5.PA1/ADC1
- net RST26: now also UC06.PA0/ADC0; no longer AT6.PA1/ADC1
- net RST27: now also 27.RST, UC06.PA1/ADC1; no longer 31.RST, AT7.PA1/ADC1
- net RST28: now also 28.RST, UC06.PA2/ADC2; no longer 36.RST, AT8.PA1/ADC1
- net RST31: now also 31.RST, UC07.PA0/ADC0; no longer 2.RST, AT1.PA2/ADC2
- net RST32: now also 32.RST, UC07.PA1/ADC1; no longer 7.RST, AT2.PA2/ADC2
- net RST33: now also 33.RST, UC07.PA2/ADC2; no longer 12.RST, AT3.PA2/ADC2
- net RST34: now also 34.RST, UC07.PA3/ADC3; no longer 17.RST, AT4.PA2/ADC2
- net RST35: now also 35.RST, UC07.PA5/MISO; no longer 22.RST, AT5.PA2/ADC2
- net RST36: now also 36.RST, UC08.PA0/ADC0; no longer 27.RST, AT6.PA2/ADC2
- net RST37: now also 37.RST, UC08.PA1/ADC1; no longer 32.RST, AT7.PA2/ADC2
- net RST38: now also 38.RST, UC08.PA2/ADC2; no longer 37.RST, AT8.PA2/ADC2
- net SCL: now also 01.SCL, 02.SCL, 03.SCL, 04.SCL, 05.SCL, 06.SCL, 07.SCL, 08.SCL, 09.SCL, 40.SCL, UC01.PA4/SCL, UC02.PA4/SCL, UC03.PA4/SCL, UC04.PA4/SCL, UC05.PA4/SCL, UC06.PA4/SCL, UC07.PA4/SCL, UC08.PA4/SCL; no longer 0.SCL, 1.SCL, 2.SCL, 3.SCL, 4.SCL, 5.SCL, 6.SCL, 7.SCL, 8.SCL, 9.SCL, AT1.PA4/SCL, AT2.PA4/SCL, AT3.PA4/SCL, AT4.PA4/SCL, AT5.PA4/SCL, AT6.PA4/SCL, AT7.PA4/SCL, AT8.PA4/SCL, PROG1.3, PROG2.3, PROG3.3, PROG4.3, PROG5.3, PROG6.3, PROG7.3, PROG8.3
- net SDA: now also 01.SDA, 02.SDA, 03.SDA, 04.SDA, 05.SDA, 06.SDA, 07.SDA, 08.SDA, 09.SDA, 40.SDA, UC01.PA6/MOSI, UC02.PA6/MOSI, UC03.PA6/MOSI, UC04.PA6/MOSI, UC05.PA6/MOSI, UC06.PA6/MOSI, UC07.PA6/MOSI, UC08.PA6/MOSI; no longer 0.SDA, 1.SDA, 2.SDA, 3.SDA, 4.SDA, 5.SDA, 6.SDA, 7.SDA, 8.SDA, 9.SDA, AT1.PA6/MOSI, AT2.PA6/MOSI, AT3.PA6/MOSI, AT4.PA6/MOSI, AT5.PA6/MOSI, AT6.PA6/MOSI, AT7.PA6/MOSI, AT8.PA6/MOSI, PROG1.4, PROG2.4, PROG3.4, PROG4.4, PROG5.4, PROG6.4, PROG7.4, PROG8.4

Commit message: no airwires save address pins
Connections:
- new net RESET07: UC07.PB3/RESET
- net RESET06: no longer UC07.PB3/RESET
Changed lines of the file:
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@@
-</segment>
-</net>
-<net name="RESET06" class="0">
-<segment>
-<wire x1="50.8" y1="2.54" x2="55.88" y2="2.54" width="0" layer="91"/>
-<label x="55.88" y="2.54" size="1.778" layer="95"/>
-<pinref part="UC07" gate="G$1" pin="PB3/RESET"/>
 </segment>
 </net>
@@
 </segment>
 </net>
+<net name="RESET07" class="0">
+<segment>
+<wire x1="50.8" y1="2.54" x2="55.88" y2="2.54" width="0" layer="91"/>
+<label x="55.88" y="2.54" size="1.778" layer="95"/>
+<pinref part="UC07" gate="G$1" pin="PB3/RESET"/>
+</segment>
+</net>
