File: eagle/fullArray.sch (EAGLE design)
At the start: 115 parts

Commit message: fixed addressing logic pin assignment, zero airwires, zero todos
Connections:
- removed net ADDR00: UC01.PB0, UC02.PB0, UC03.PB0, UC04.PB0, UC05.PB0, UC06.PB0, UC07.PB0, UC08.PB0
- new net ADDR1A: UC01.PB0
- new net ADDR2A: UC02.PB1
- new net ADDR3A: UC03.PB0
- new net ADDR3B: UC03.PB1
- new net ADDR4A: UC04.PB2
- new net ADDR5A: UC05.PB0
- new net ADDR5B: UC05.PB2
- new net ADDR6A: UC06.PB1
- new net ADDR6B: UC06.PB2
- new net ADDR7A: UC07.PB0
- new net ADDR7B: UC07.PB1
- new net ADDR7C: UC07.PB2
- new net ADDR8A: UC08.PA7/ADC7
- net GND: now also UC02.PB0, UC04.PB0, UC06.PB0, UC08.PB0; no longer UC02.PB1, UC03.PB1, UC04.PB2, UC05.PB2, UC06.PB1, UC06.PB2, UC07.PB1, UC07.PB2, UC08.PA7/ADC7
Changed lines of the file:
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@@
 </segment>
 </net>
-<net name="ADDR00" class="0">
+<net name="ADDR1A" class="0">
 <segment>
 <pinref part="UC01" gate="G$1" pin="PB0"/>
@@
 </segment>
 <segment>
-<pinref part="UC02" gate="G$1" pin="PB1"/>
-<wire x1="50.8" y1="7.62" x2="53.34" y2="7.62" width="0" layer="91"/>
-<label x="53.34" y="7.62" size="1.778" layer="95"/>
-</segment>
-<segment>
 <pinref part="UC02" gate="G$1" pin="PB2"/>
 <wire x1="50.8" y1="5.08" x2="53.34" y2="5.08" width="0" layer="91"/>
@@
 <pinref part="C15" gate="G$1" pin="P$2"/>
 <wire x1="139.7" y1="5.08" x2="144.78" y2="5.08" width="0" layer="91"/>
+</segment>
+<segment>
+<pinref part="UC02" gate="G$1" pin="PB0"/>
+<wire x1="50.8" y1="10.16" x2="53.34" y2="10.16" width="0" layer="91"/>
+<label x="53.34" y="10.16" size="1.778" layer="95"/>
 </segment>
 </net>
@@
 </segment>
 </net>
-<net name="ADDR00" class="0">
-<segment>
-<pinref part="UC02" gate="G$1" pin="PB0"/>
-<wire x1="50.8" y1="10.16" x2="53.34" y2="10.16" width="0" layer="91"/>
-<label x="53.34" y="10.16" size="1.778" layer="95"/>
+<net name="ADDR2A" class="0">
+<segment>
+<pinref part="UC02" gate="G$1" pin="PB1"/>
+<wire x1="50.8" y1="7.62" x2="53.34" y2="7.62" width="0" layer="91"/>
+<label x="53.34" y="7.62" size="1.778" layer="95"/>
 </segment>
 </net>
@@
 <wire x1="50.8" y1="15.24" x2="53.34" y2="15.24" width="0" layer="91"/>
 <label x="53.34" y="15.24" size="1.778" layer="95"/>
-</segment>
-<segment>
-<pinref part="UC03" gate="G$1" pin="PB1"/>
-<wire x1="50.8" y1="7.62" x2="53.34" y2="7.62" width="0" layer="91"/>
-<label x="53.34" y="7.62" size="1.778" layer="95"/>
 </segment>
 <segment>
@@
 </segment>
 </net>
-<net name="ADDR00" class="0">
+<net name="ADDR3B" class="0">
+<segment>
+<pinref part="UC03" gate="G$1" pin="PB1"/>
+<wire x1="50.8" y1="7.62" x2="53.34" y2="7.62" width="0" layer="91"/>
+<label x="53.34" y="7.62" size="1.778" layer="95"/>
+</segment>
+</net>
+<net name="ADDR3A" class="0">
 <segment>
 <pinref part="UC03" gate="G$1" pin="PB0"/>
@@
 </segment>
 <segment>
-<pinref part="UC04" gate="G$1" pin="PB2"/>
-<wire x1="50.8" y1="5.08" x2="53.34" y2="5.08" width="0" layer="91"/>
-<label x="53.34" y="5.08" size="1.778" layer="95"/>
-</segment>
-<segment>
 <label x="139.7" y="5.08" size="1.778" layer="95" rot="R180"/>
 <pinref part="C27" gate="G$1" pin="P$2"/>
 <wire x1="139.7" y1="5.08" x2="144.78" y2="5.08" width="0" layer="91"/>
+</segment>
+<segment>
+<pinref part="UC04" gate="G$1" pin="PB0"/>
+<wire x1="50.8" y1="10.16" x2="53.34" y2="10.16" width="0" layer="91"/>
+<label x="53.34" y="10.16" size="1.778" layer="95"/>
 </segment>
 </net>
@@
 </segment>
 </net>
-<net name="ADDR00" class="0">
-<segment>
-<pinref part="UC04" gate="G$1" pin="PB0"/>
-<wire x1="50.8" y1="10.16" x2="53.34" y2="10.16" width="0" layer="91"/>
-<label x="53.34" y="10.16" size="1.778" layer="95"/>
+<net name="ADDR4A" class="0">
+<segment>
+<pinref part="UC04" gate="G$1" pin="PB2"/>
+<wire x1="50.8" y1="5.08" x2="53.34" y2="5.08" width="0" layer="91"/>
+<label x="53.34" y="5.08" size="1.778" layer="95"/>
 </segment>
 </net>
@@
 <wire x1="50.8" y1="7.62" x2="53.34" y2="7.62" width="0" layer="91"/>
 <label x="53.34" y="7.62" size="1.778" layer="95"/>
-</segment>
-<segment>
-<pinref part="UC05" gate="G$1" pin="PB2"/>
-<wire x1="50.8" y1="5.08" x2="53.34" y2="5.08" width="0" layer="91"/>
-<label x="53.34" y="5.08" size="1.778" layer="95"/>
 </segment>
 <segment>
@@
 </segment>
 </net>
-<net name="ADDR00" class="0">
+<net name="ADDR5B" class="0">
+<segment>
+<pinref part="UC05" gate="G$1" pin="PB2"/>
+<wire x1="50.8" y1="5.08" x2="53.34" y2="5.08" width="0" layer="91"/>
+<label x="53.34" y="5.08" size="1.778" layer="95"/>
+</segment>
+</net>
+<net name="ADDR5A" class="0">
 <segment>
 <pinref part="UC05" gate="G$1" pin="PB0"/>
@@
 </segment>
 <segment>
-<pinref part="UC06" gate="G$1" pin="PB1"/>
-<wire x1="50.8" y1="7.62" x2="53.34" y2="7.62" width="0" layer="91"/>
-<label x="53.34" y="7.62" size="1.778" layer="95"/>
-</segment>
-<segment>
-<pinref part="UC06" gate="G$1" pin="PB2"/>
-<wire x1="50.8" y1="5.08" x2="53.34" y2="5.08" width="0" layer="91"/>
-<label x="53.34" y="5.08" size="1.778" layer="95"/>
-</segment>
-<segment>
 <label x="139.7" y="5.08" size="1.778" layer="95" rot="R180"/>
 <pinref part="C39" gate="G$1" pin="P$2"/>
 <wire x1="139.7" y1="5.08" x2="144.78" y2="5.08" width="0" layer="91"/>
+</segment>
+<segment>
+<pinref part="UC06" gate="G$1" pin="PB0"/>
+<wire x1="50.8" y1="10.16" x2="53.34" y2="10.16" width="0" layer="91"/>
+<label x="53.34" y="10.16" size="1.778" layer="95"/>
 </segment>
 </net>
@@
 </segment>
 </net>
-<net name="ADDR00" class="0">
-<segment>
-<pinref part="UC06" gate="G$1" pin="PB0"/>
-<wire x1="50.8" y1="10.16" x2="53.34" y2="10.16" width="0" layer="91"/>
-<label x="53.34" y="10.16" size="1.778" layer="95"/>
+<net name="ADDR6B" class="0">
+<segment>
+<pinref part="UC06" gate="G$1" pin="PB2"/>
+<wire x1="50.8" y1="5.08" x2="53.34" y2="5.08" width="0" layer="91"/>
+<label x="53.34" y="5.08" size="1.778" layer="95"/>
+</segment>
+</net>
+<net name="ADDR6A" class="0">
+<segment>
+<pinref part="UC06" gate="G$1" pin="PB1"/>
+<wire x1="50.8" y1="7.62" x2="53.34" y2="7.62" width="0" layer="91"/>
+<label x="53.34" y="7.62" size="1.778" layer="95"/>
 </segment>
 </net>
@@
 </segment>
 <segment>
+<label x="139.7" y="5.08" size="1.778" layer="95" rot="R180"/>
+<pinref part="C45" gate="G$1" pin="P$2"/>
+<wire x1="139.7" y1="5.08" x2="144.78" y2="5.08" width="0" layer="91"/>
+</segment>
+<segment>
 <pinref part="UC07" gate="G$1" pin="PA7/ADC7"/>
 <wire x1="50.8" y1="15.24" x2="53.34" y2="15.24" width="0" layer="91"/>
 <label x="53.34" y="15.24" size="1.778" layer="95"/>
-</segment>
-<segment>
-<pinref part="UC07" gate="G$1" pin="PB1"/>
-<wire x1="50.8" y1="7.62" x2="53.34" y2="7.62" width="0" layer="91"/>
-<label x="53.34" y="7.62" size="1.778" layer="95"/>
-</segment>
-<segment>
-<pinref part="UC07" gate="G$1" pin="PB2"/>
-<wire x1="50.8" y1="5.08" x2="53.34" y2="5.08" width="0" layer="91"/>
-<label x="53.34" y="5.08" size="1.778" layer="95"/>
-</segment>
-<segment>
-<label x="139.7" y="5.08" size="1.778" layer="95" rot="R180"/>
-<pinref part="C45" gate="G$1" pin="P$2"/>
-<wire x1="139.7" y1="5.08" x2="144.78" y2="5.08" width="0" layer="91"/>
 </segment>
 </net>
@@
 </segment>
 </net>
-<net name="ADDR00" class="0">
+<net name="RESET07" class="0">
+<segment>
+<wire x1="50.8" y1="2.54" x2="55.88" y2="2.54" width="0" layer="91"/>
+<label x="55.88" y="2.54" size="1.778" layer="95"/>
+<pinref part="UC07" gate="G$1" pin="PB3/RESET"/>
+</segment>
+</net>
+<net name="ADDR7A" class="0">
 <segment>
 <pinref part="UC07" gate="G$1" pin="PB0"/>
@@
 </segment>
 </net>
-<net name="RESET07" class="0">
-<segment>
-<wire x1="50.8" y1="2.54" x2="55.88" y2="2.54" width="0" layer="91"/>
-<label x="55.88" y="2.54" size="1.778" layer="95"/>
-<pinref part="UC07" gate="G$1" pin="PB3/RESET"/>
+<net name="ADDR7B" class="0">
+<segment>
+<pinref part="UC07" gate="G$1" pin="PB1"/>
+<wire x1="50.8" y1="7.62" x2="53.34" y2="7.62" width="0" layer="91"/>
+<label x="53.34" y="7.62" size="1.778" layer="95"/>
+</segment>
+</net>
+<net name="ADDR7C" class="0">
+<segment>
+<pinref part="UC07" gate="G$1" pin="PB2"/>
+<wire x1="50.8" y1="5.08" x2="53.34" y2="5.08" width="0" layer="91"/>
+<label x="53.34" y="5.08" size="1.778" layer="95"/>
 </segment>
 </net>
@@
 </segment>
 <segment>
-<pinref part="UC08" gate="G$1" pin="PA7/ADC7"/>
-<wire x1="50.8" y1="15.24" x2="53.34" y2="15.24" width="0" layer="91"/>
-<label x="53.34" y="15.24" size="1.778" layer="95"/>
-</segment>
-<segment>
 <pinref part="UC08" gate="G$1" pin="PB1"/>
 <wire x1="50.8" y1="7.62" x2="53.34" y2="7.62" width="0" layer="91"/>
@@
 <pinref part="C51" gate="G$1" pin="P$2"/>
 <wire x1="139.7" y1="5.08" x2="144.78" y2="5.08" width="0" layer="91"/>
+</segment>
+<segment>
+<pinref part="UC08" gate="G$1" pin="PB0"/>
+<wire x1="50.8" y1="10.16" x2="53.34" y2="10.16" width="0" layer="91"/>
+<label x="53.34" y="10.16" size="1.778" layer="95"/>
 </segment>
 </net>
@@
 </segment>
 </net>
-<net name="ADDR00" class="0">
-<segment>
-<pinref part="UC08" gate="G$1" pin="PB0"/>
-<wire x1="50.8" y1="10.16" x2="53.34" y2="10.16" width="0" layer="91"/>
-<label x="53.34" y="10.16" size="1.778" layer="95"/>
-</segment>
-</net>
+<net name="ADDR8A" class="0">
+<segment>
+<pinref part="UC08" gate="G$1" pin="PA7/ADC7"/>
+<wire x1="50.8" y1="15.24" x2="53.34" y2="15.24" width="0" layer="91"/>
+<label x="53.34" y="15.24" size="1.778" layer="95"/>
+</segment>
+</net>
