File: eagle/fullArray.sch (EAGLE design)
At the start: 115 parts

Commit message: cosmetic rearrangements, drop programming header on xmega, center board
Parts:
- removed PROGX: (no value), nonolith:HEADER-2X3
Connections:
- net 3.3V: no longer PROGX.2
- net BOOTLOAD: no longer PROGX.4
- net GND: no longer PROGX.6
- net PDI-CLK: no longer PROGX.5
- net PDI-DATA: no longer PROGX.1
- net PR1: no longer PROGX.3
Changed lines of the file:
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@@
 <part name="C11" library="nonolith" deviceset="CAP_CERAMIC" device="0603" value=".1uF"/>
 <part name="C12" library="nonolith" deviceset="CAP_CERAMIC" device="0603" value=".01uF"/>
-<part name="PROGX" library="nonolith" deviceset="HEADER-2X3" device=""/>
 <part name="R1" library="nonolith" deviceset="RESISTOR" device="0603" value="120o"/>
 <part name="LED1" library="microbuilder" deviceset="LED" device="0603"/>
@@
 <instance part="C11" gate="G$1" x="22.86" y="60.96"/>
 <instance part="C12" gate="G$1" x="33.02" y="60.96"/>
-<instance part="PROGX" gate="A" x="149.86" y="63.5" rot="R90"/>
 <instance part="R1" gate="G$1" x="116.84" y="81.28"/>
 <instance part="LED1" gate="G$1" x="129.54" y="81.28"/>
@@
 </segment>
 <segment>
-<pinref part="PROGX" gate="A" pin="6"/>
-<wire x1="152.4" y1="68.58" x2="152.4" y2="73.66" width="0" layer="91"/>
-<label x="152.4" y="73.66" size="1.778" layer="95" rot="R90"/>
-</segment>
-<segment>
 <pinref part="DAISY" gate="A" pin="1"/>
 <wire x1="129.54" y1="12.7" x2="134.62" y2="12.7" width="0" layer="91"/>
@@
 </segment>
 <segment>
-<pinref part="PROGX" gate="A" pin="2"/>
-<wire x1="147.32" y1="68.58" x2="147.32" y2="73.66" width="0" layer="91"/>
-<label x="147.32" y="73.66" size="1.778" layer="95" rot="R90"/>
-</segment>
-<segment>
 <pinref part="R2" gate="G$1" pin="2"/>
 <wire x1="114.3" y1="58.42" x2="114.3" y2="60.96" width="0" layer="91"/>
@@
 <wire x1="106.68" y1="81.28" x2="111.76" y2="81.28" width="0" layer="91"/>
 </segment>
-<segment>
-<pinref part="PROGX" gate="A" pin="3"/>
-<wire x1="149.86" y1="60.96" x2="149.86" y2="55.88" width="0" layer="91"/>
-<label x="149.86" y="55.88" size="1.778" layer="95" rot="R270"/>
-</segment>
 </net>
 <net name="PR1-P" class="0">
@@
 <label x="111.76" y="76.2" size="1.778" layer="95"/>
 </segment>
-<segment>
-<pinref part="PROGX" gate="A" pin="4"/>
-<wire x1="149.86" y1="68.58" x2="149.86" y2="73.66" width="0" layer="91"/>
-<label x="149.86" y="73.66" size="1.778" layer="95" rot="R90"/>
-</segment>
 </net>
 <net name="PDI-DATA" class="0">
@@
 <label x="111.76" y="68.58" size="1.778" layer="95"/>
 </segment>
-<segment>
-<pinref part="PROGX" gate="A" pin="1"/>
-<wire x1="147.32" y1="60.96" x2="147.32" y2="55.88" width="0" layer="91"/>
-<label x="147.32" y="55.88" size="1.778" layer="95" rot="R270"/>
-</segment>
 </net>
 <net name="PDI-CLK" class="0">
@@
 <label x="111.76" y="2.54" size="1.778" layer="95"/>
 </segment>
-<segment>
-<pinref part="PROGX" gate="A" pin="5"/>
-<wire x1="152.4" y1="60.96" x2="152.4" y2="55.88" width="0" layer="91"/>
-<label x="152.4" y="55.88" size="1.778" layer="95" rot="R270"/>
-</segment>
-</net>
+</net>

Commit message: s/0603 resistor/solder jumper/, clean power traces, add 0.5mm vias for PDI-DATA and PDI-CLK
Parts:
- removed R4: 4.7k, nonolith:RESISTOR0603
- added SJ1: (no value), jumper:SJ
Connections:
- net 3.3V: now also SJ1.2; no longer R4.2
- net PE0: now also SJ1.1; no longer R4.1
Changed lines of the file:
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@@
 <part name="R3" library="nonolith" deviceset="RESISTOR" device="0603" value="4.7K"/>
 <part name="DAISY" library="nonolith" deviceset="HEADER-1X6" device="2MM"/>
-<part name="R4" library="nonolith" deviceset="RESISTOR" device="0603" value="4.7k"/>
 <part name="SCL" library="nonolith" deviceset="HEADER-1X1" device="2MM"/>
 <part name="SDA" library="nonolith" deviceset="HEADER-1X1" device="2MM"/>
@@
 <part name="C52" library="microbuilder" deviceset="CAP_TANTALUM" device="D/7343_REFLOW" value="470uF"/>
 <part name="C53" library="nonolith" deviceset="CAP_CERAMIC" device="1206" value="10uF"/>
+<part name="SJ1" library="jumper" deviceset="SJ" device=""/>
 </parts>
 <sheets>
@@
 <instance part="R3" gate="G$1" x="119.38" y="50.8" rot="R90"/>
 <instance part="DAISY" gate="A" x="127" y="20.32" rot="R180"/>
-<instance part="R4" gate="G$1" x="147.32" y="22.86"/>
 <instance part="SCL" gate="G$1" x="129.54" y="48.26"/>
 <instance part="SDA" gate="G$1" x="129.54" y="45.72"/>
@@
 <instance part="C52" gate="G$1" x="-5.08" y="38.1" rot="R180"/>
 <instance part="C53" gate="G$1" x="22.86" y="27.94" rot="R180"/>
+<instance part="SJ1" gate="1" x="147.32" y="22.86"/>
 </instances>
 <busses>
@@
 <wire x1="167.64" y1="22.86" x2="167.64" y2="25.4" width="0" layer="91"/>
 <label x="167.64" y="25.4" size="1.778" layer="95"/>
-<pinref part="R4" gate="G$1" pin="2"/>
 <wire x1="167.64" y1="22.86" x2="152.4" y2="22.86" width="0" layer="91"/>
+<pinref part="SJ1" gate="1" pin="2"/>
 </segment>
 <segment>
@@
 <pinref part="DAISY" gate="A" pin="5"/>
 <label x="134.62" y="22.86" size="1.778" layer="95"/>
-<pinref part="R4" gate="G$1" pin="1"/>
 <wire x1="129.54" y1="22.86" x2="142.24" y2="22.86" width="0" layer="91"/>
-</segment>
-</net>
+<pinref part="SJ1" gate="1" pin="1"/>
+</segment>
+</net>
