File: eagle/usbInterface.sch (EAGLE design)
At the start: 17 parts

Commit message: added up to date usb interface board
Parts:
- added C43: 470uF, microbuilder:CAP_TANTALUMD/7343_REFLOW
- added C44: 10uF, nonolith:CAP_CERAMIC1206
- 3.3V: value VREG -> VREGAP1117; device nonolith:VREG -> nonolith:VREGAP1117
Connections:
- net 3.3V: now also C43.+
- net 5V: now also C44.P$2
- net GND: now also C43.-, C44.P$1
Changed lines of the file:
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@@
 <?xml version="1.0" encoding="utf-8"?>
 <!DOCTYPE eagle SYSTEM "eagle.dtd">
-<eagle version="6.1">
+<eagle version="6.3">
 <drawing>
 <settings>
@@
 <part name="XM1" library="nonolith" deviceset="ATXMEGAXXA4U" device="-MH"/>
 <part name="CN1" library="nonolith" deviceset="USB" device="MICROB"/>
-<part name="3.3V" library="nonolith" deviceset="VREG" device=""/>
+<part name="3.3V" library="nonolith" deviceset="VREG" device="AP1117"/>
 <part name="C10" library="nonolith" deviceset="CAP_CERAMIC" device="0603" value="1uF"/>
 <part name="C11" library="nonolith" deviceset="CAP_CERAMIC" device="0603" value=".1uF"/>
@@
 <part name="JP1" library="nonolith" deviceset="HEADER-1X1" device="2MM"/>
 <part name="JP2" library="nonolith" deviceset="HEADER-1X1" device="2MM"/>
+<part name="C43" library="microbuilder" deviceset="CAP_TANTALUM" device="D/7343_REFLOW" value="470uF"/>
+<part name="C44" library="nonolith" deviceset="CAP_CERAMIC" device="1206" value="10uF"/>
 </parts>
 <sheets>
@@
 <instance part="JP1" gate="G$1" x="124.46" y="43.18" rot="R180"/>
 <instance part="JP2" gate="G$1" x="124.46" y="40.64" rot="R180"/>
+<instance part="C43" gate="G$1" x="-5.08" y="38.1" rot="R180"/>
+<instance part="C44" gate="G$1" x="22.86" y="27.94" rot="R180"/>
 </instances>
 <busses>
@@
 <wire x1="22.86" y1="73.66" x2="12.7" y2="73.66" width="0" layer="91"/>
 <wire x1="12.7" y1="73.66" x2="5.08" y2="73.66" width="0" layer="91"/>
-<wire x1="5.08" y1="73.66" x2="5.08" y2="40.64" width="0" layer="91"/>
+<wire x1="5.08" y1="73.66" x2="5.08" y2="43.18" width="0" layer="91"/>
 <junction x="43.18" y="78.74"/>
 <junction x="43.18" y="76.2"/>
 <junction x="43.18" y="73.66"/>
 <pinref part="C10" gate="G$1" pin="P$1"/>
+<wire x1="5.08" y1="43.18" x2="5.08" y2="40.64" width="0" layer="91"/>
 <wire x1="12.7" y1="73.66" x2="12.7" y2="66.04" width="0" layer="91"/>
 <pinref part="C11" gate="G$1" pin="P$1"/>
@@
 <junction x="12.7" y="73.66"/>
 <label x="5.08" y="73.66" size="1.778" layer="95" rot="R180"/>
+<pinref part="C43" gate="G$1" pin="-"/>
+<wire x1="-5.08" y1="40.64" x2="-5.08" y2="43.18" width="0" layer="91"/>
+<wire x1="-5.08" y1="43.18" x2="5.08" y2="43.18" width="0" layer="91"/>
+<junction x="5.08" y="43.18"/>
 </segment>
 <segment>
@@
 <wire x1="127" y1="43.18" x2="132.08" y2="43.18" width="0" layer="91"/>
 <label x="132.08" y="43.18" size="1.778" layer="95"/>
+</segment>
+<segment>
+<pinref part="C44" gate="G$1" pin="P$1"/>
+<wire x1="22.86" y1="22.86" x2="20.32" y2="22.86" width="0" layer="91"/>
+<label x="20.32" y="22.86" size="1.778" layer="95" rot="R180"/>
 </segment>
 </net>
@@
 <junction x="33.02" y="50.8"/>
 <label x="2.54" y="50.8" size="1.778" layer="95" rot="R180"/>
+<pinref part="C43" gate="G$1" pin="+"/>
+<wire x1="-5.08" y1="33.02" x2="2.54" y2="33.02" width="0" layer="91"/>
+<wire x1="2.54" y1="33.02" x2="2.54" y2="35.56" width="0" layer="91"/>
 </segment>
 <segment>
@@
 <pinref part="3.3V" gate="G$1" pin="VIN"/>
 <wire x1="25.4" y1="38.1" x2="27.94" y2="38.1" width="0" layer="91"/>
-<wire x1="27.94" y1="38.1" x2="27.94" y2="12.7" width="0" layer="91"/>
+<wire x1="27.94" y1="38.1" x2="27.94" y2="30.48" width="0" layer="91"/>
 <pinref part="CN1" gate="G$1" pin="VBUS"/>
+<wire x1="27.94" y1="30.48" x2="27.94" y2="12.7" width="0" layer="91"/>
 <wire x1="27.94" y1="12.7" x2="20.32" y2="12.7" width="0" layer="91"/>
 <label x="27.94" y="38.1" size="1.778" layer="95"/>
-</segment>
-<segment>
+<pinref part="C44" gate="G$1" pin="P$2"/>
+<wire x1="22.86" y1="30.48" x2="27.94" y2="30.48" width="0" layer="91"/>
+<junction x="27.94" y="30.48"/>
+</segment>
+<segment>
