File: eagle/tessellate.sch (EAGLE design)
At the start: 12 parts

Commit message: reworked silkscreen and snap on tesselate.brd
Parts:
- renumbered PROG to PROG0
Changed lines of the file:
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@@
 <part name="C3" library="nonolith" deviceset="CAP_CERAMIC" device="0603"/>
 <part name="C4" library="nonolith" deviceset="CAP_CERAMIC" device="0603"/>
-<part name="PROG" library="nonolith" deviceset="HEADER-2X3" device=""/>
+<part name="PROG0" library="nonolith" deviceset="HEADER-2X3" device=""/>
 </parts>
 <sheets>
@@
 <instance part="C3" gate="G$1" x="134.62" y="58.42"/>
 <instance part="C4" gate="G$1" x="172.72" y="58.42"/>
-<instance part="PROG" gate="A" x="121.92" y="7.62"/>
+<instance part="PROG0" gate="A" x="121.92" y="7.62"/>
 </instances>
 <busses>
@@
 </segment>
 <segment>
-<pinref part="PROG" gate="A" pin="6"/>
+<pinref part="PROG0" gate="A" pin="6"/>
 <wire x1="127" y1="5.08" x2="132.08" y2="5.08" width="0" layer="91"/>
 <label x="132.08" y="5.08" size="1.778" layer="95"/>
@@
 </segment>
 <segment>
-<pinref part="PROG" gate="A" pin="2"/>
+<pinref part="PROG0" gate="A" pin="2"/>
 <wire x1="127" y1="10.16" x2="132.08" y2="10.16" width="0" layer="91"/>
 <label x="132.08" y="10.16" size="1.778" layer="95"/>
@@
 </segment>
 <segment>
-<pinref part="PROG" gate="A" pin="4"/>
+<pinref part="PROG0" gate="A" pin="4"/>
 <wire x1="127" y1="7.62" x2="132.08" y2="7.62" width="0" layer="91"/>
 <label x="132.08" y="7.62" size="1.778" layer="95"/>
@@
 </segment>
 <segment>
-<pinref part="PROG" gate="A" pin="3"/>
+<pinref part="PROG0" gate="A" pin="3"/>
 <wire x1="119.38" y1="7.62" x2="114.3" y2="7.62" width="0" layer="91"/>
 <label x="114.3" y="7.62" size="1.778" layer="95" rot="R180"/>
@@
 </segment>
 <segment>
-<pinref part="PROG" gate="A" pin="5"/>
+<pinref part="PROG0" gate="A" pin="5"/>
 <wire x1="119.38" y1="5.08" x2="114.3" y2="5.08" width="0" layer="91"/>
 <label x="114.3" y="5.08" size="1.778" layer="95" rot="R180"/>
@@
 </segment>
 <segment>
-<pinref part="PROG" gate="A" pin="1"/>
+<pinref part="PROG0" gate="A" pin="1"/>
 <wire x1="119.38" y1="10.16" x2="114.3" y2="10.16" width="0" layer="91"/>
 <label x="114.3" y="10.16" size="1.778" layer="95" rot="R180"/>

Commit message: start of repeatable / chainable rows w/ 7mm spacing and no vias under qfn tiny
Parts:
- added C5: (no value), nonolith:CAP_CERAMIC0402
- C0, C1, C2, C3, C4: device nonolith:CAP_CERAMIC0603 -> nonolith:CAP_CERAMIC0402
Connections:
- net 3.3V: now also C5.P$1
- net GND: now also C5.P$2
Changed lines of the file:
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@@
 <?xml version="1.0" encoding="utf-8"?>
 <!DOCTYPE eagle SYSTEM "eagle.dtd">
-<eagle version="6.1">
+<eagle version="6.3">
 <drawing>
 <settings>
@@
 <grid distance="0.1" unitdist="inch" unit="inch" style="lines" multiple="1" display="no" altdistance="0.01" altunitdist="inch" altunit="inch"/>
 <layers>
-<layer number="1" name="Top" color="4" fill="1" visible="no" active="no"/>
-<layer number="2" name="Route2" color="1" fill="3" visible="no" active="no"/>
-<layer number="3" name="Route3" color="4" fill="3" visible="no" active="no"/>
-<layer number="4" name="Route4" color="1" fill="4" visible="no" active="no"/>
-<layer number="5" name="Route5" color="4" fill="4" visible="no" active="no"/>
-<layer number="6" name="Route6" color="1" fill="8" visible="no" active="no"/>
-<layer number="7" name="Route7" color="4" fill="8" visible="no" active="no"/>
-<layer number="8" name="Route8" color="1" fill="2" visible="no" active="no"/>
-<layer number="9" name="Route9" color="4" fill="2" visible="no" active="no"/>
-<layer number="10" name="Route10" color="1" fill="7" visible="no" active="no"/>
-<layer number="11" name="Route11" color="4" fill="7" visible="no" active="no"/>
-<layer number="12" name="Route12" color="1" fill="5" visible="no" active="no"/>
-<layer number="13" name="Route13" color="4" fill="5" visible="no" active="no"/>
-<layer number="14" name="Route14" color="1" fill="6" visible="no" active="no"/>
-<layer number="15" name="Route15" color="4" fill="6" visible="no" active="no"/>
-<layer number="16" name="Bottom" color="1" fill="1" visible="no" active="no"/>
-<layer number="17" name="Pads" color="2" fill="1" visible="no" active="no"/>
-<layer number="18" name="Vias" color="2" fill="1" visible="no" active="no"/>
-<layer number="19" name="Unrouted" color="6" fill="1" visible="no" active="no"/>
-<layer number="20" name="Dimension" color="15" fill="1" visible="no" active="no"/>
-<layer number="21" name="tPlace" color="7" fill="1" visible="no" active="no"/>
-<layer number="22" name="bPlace" color="7" fill="1" visible="no" active="no"/>
-<layer number="23" name="tOrigins" color="15" fill="1" visible="no" active="no"/>
-<layer number="24" name="bOrigins" color="15" fill="1" visible="no" active="no"/>
-<layer number="25" name="tNames" color="7" fill="1" visible="no" active="no"/>
-<layer number="26" name="bNames" color="7" fill="1" visible="no" active="no"/>
-<layer number="27" name="tValues" color="7" fill="1" visible="no" active="no"/>
-<layer number="28" name="bValues" color="7" fill="1" visible="no" active="no"/>
+<layer number="1" name="Top" color="4" fill="1" visible="yes" active="no"/>
+<layer number="2" name="Route2" color="1" fill="3" visible="yes" active="no"/>
+<layer number="3" name="Route3" color="4" fill="3" visible="yes" active="no"/>
+<layer number="4" name="Route4" color="1" fill="4" visible="yes" active="no"/>
+<layer number="5" name="Route5" color="4" fill="4" visible="yes" active="no"/>
+<layer number="6" name="Route6" color="1" fill="8" visible="yes" active="no"/>
+<layer number="7" name="Route7" color="4" fill="8" visible="yes" active="no"/>
+<layer number="8" name="Route8" color="1" fill="2" visible="yes" active="no"/>
+<layer number="9" name="Route9" color="4" fill="2" visible="yes" active="no"/>
+<layer number="10" name="Route10" color="1" fill="7" visible="yes" active="no"/>
+<layer number="11" name="Route11" color="4" fill="7" visible="yes" active="no"/>
+<layer number="12" name="Route12" color="1" fill="5" visible="yes" active="no"/>
+<layer number="13" name="Route13" color="4" fill="5" visible="yes" active="no"/>
+<layer number="14" name="Route14" color="1" fill="6" visible="yes" active="no"/>
+<layer number="15" name="Route15" color="4" fill="6" visible="yes" active="no"/>
+<layer number="16" name="Bottom" color="1" fill="1" visible="yes" active="no"/>
+<layer number="17" name="Pads" color="2" fill="1" visible="yes" active="no"/>
+<layer number="18" name="Vias" color="2" fill="1" visible="yes" active="no"/>
+<layer number="19" name="Unrouted" color="6" fill="1" visible="yes" active="no"/>
+<layer number="20" name="Dimension" color="15" fill="1" visible="yes" active="no"/>
+<layer number="21" name="tPlace" color="7" fill="1" visible="yes" active="no"/>
+<layer number="22" name="bPlace" color="7" fill="1" visible="yes" active="no"/>
+<layer number="23" name="tOrigins" color="15" fill="1" visible="yes" active="no"/>
+<layer number="24" name="bOrigins" color="15" fill="1" visible="yes" active="no"/>
+<layer number="25" name="tNames" color="7" fill="1" visible="yes" active="no"/>
+<layer number="26" name="bNames" color="7" fill="1" visible="yes" active="no"/>
+<layer number="27" name="tValues" color="7" fill="1" visible="yes" active="no"/>
+<layer number="28" name="bValues" color="7" fill="1" visible="yes" active="no"/>
 <layer number="29" name="tStop" color="7" fill="3" visible="no" active="no"/>
 <layer number="30" name="bStop" color="7" fill="6" visible="no" active="no"/>
@@
 <layer number="35" name="tGlue" color="7" fill="4" visible="no" active="no"/>
 <layer number="36" name="bGlue" color="7" fill="5" visible="no" active="no"/>
-<layer number="37" name="tTest" color="7" fill="1" visible="no" active="no"/>
-<layer number="38" name="bTest" color="7" fill="1" visible="no" active="no"/>
+<layer number="37" name="tTest" color="7" fill="1" visible="yes" active="no"/>
+<layer number="38" name="bTest" color="7" fill="1" visible="yes" active="no"/>
 <layer number="39" name="tKeepout" color="4" fill="11" visible="no" active="no"/>
 <layer number="40" name="bKeepout" color="1" fill="11" visible="no" active="no"/>
@@
 <layer number="44" name="Drills" color="7" fill="1" visible="no" active="no"/>
 <layer number="45" name="Holes" color="7" fill="1" visible="no" active="no"/>
-<layer number="46" name="Milling" color="3" fill="1" visible="no" active="no"/>
-<layer number="47" name="Measures" color="7" fill="1" visible="no" active="no"/>
-<layer number="48" name="Document" color="7" fill="1" visible="no" active="no"/>
-<layer number="49" name="Reference" color="7" fill="1" visible="no" active="no"/>
-<layer number="50" name="dxf" color="7" fill="1" visible="no" active="no"/>
-<layer number="51" name="tDocu" color="7" fill="1" visible="no" active="no"/>
-<layer number="52" name="bDocu" color="7" fill="1" visible="no" active="no"/>
-<layer number="53" name="tGND_GNDA" color="7" fill="9" visible="no" active="no"/>
-<layer number="54" name="bGND_GNDA" color="1" fill="9" visible="no" active="no"/>
-<layer number="56" name="wert" color="7" fill="1" visible="no" active="no"/>
+<layer number="46" name="Milling" color="3" fill="1" visible="yes" active="no"/>
+<layer number="47" name="Measures" color="7" fill="1" visible="yes" active="no"/>
+<layer number="48" name="Document" color="7" fill="1" visible="yes" active="no"/>
+<layer number="49" name="Reference" color="7" fill="1" visible="yes" active="no"/>
+<layer number="50" name="dxf" color="7" fill="1" visible="yes" active="no"/>
+<layer number="51" name="tDocu" color="7" fill="1" visible="yes" active="no"/>
+<layer number="52" name="bDocu" color="7" fill="1" visible="yes" active="no"/>
+<layer number="53" name="tGND_GNDA" color="7" fill="9" visible="yes" active="no"/>
+<layer number="54" name="bGND_GNDA" color="1" fill="9" visible="yes" active="no"/>
+<layer number="56" name="wert" color="7" fill="1" visible="yes" active="no"/>
 <layer number="91" name="Nets" color="2" fill="1" visible="yes" active="yes"/>
 <layer number="92" name="Busses" color="1" fill="1" visible="yes" active="yes"/>
@@
 <part name="S10" library="nonolith" deviceset="MPL115A" device=""/>
 <part name="S20" library="nonolith" deviceset="MPL115A" device=""/>
-<part name="C0" library="nonolith" deviceset="CAP_CERAMIC" device="0603"/>
-<part name="C1" library="nonolith" deviceset="CAP_CERAMIC" device="0603"/>
-<part name="C2" library="nonolith" deviceset="CAP_CERAMIC" device="0603"/>
+<part name="C0" library="nonolith" deviceset="CAP_CERAMIC" device="0402"/>
+<part name="C1" library="nonolith" deviceset="CAP_CERAMIC" device="0402"/>
+<part name="C2" library="nonolith" deviceset="CAP_CERAMIC" device="0402"/>
 <part name="S30" library="nonolith" deviceset="MPL115A" device=""/>
 <part name="S40" library="nonolith" deviceset="MPL115A" device=""/>
-<part name="C3" library="nonolith" deviceset="CAP_CERAMIC" device="0603"/>
-<part name="C4" library="nonolith" deviceset="CAP_CERAMIC" device="0603"/>
+<part name="C3" library="nonolith" deviceset="CAP_CERAMIC" device="0402"/>
+<part name="C4" library="nonolith" deviceset="CAP_CERAMIC" device="0402"/>
 <part name="PROG0" library="nonolith" deviceset="HEADER-2X3" device=""/>
+<part name="C5" library="nonolith" deviceset="CAP_CERAMIC" device="0402"/>
 </parts>
 <sheets>
@@
 <instance part="C4" gate="G$1" x="172.72" y="58.42"/>
 <instance part="PROG0" gate="A" x="121.92" y="7.62"/>
+<instance part="C5" gate="G$1" x="144.78" y="7.62"/>
 </instances>
 <busses>
@@
 <segment>
 <pinref part="PROG0" gate="A" pin="6"/>
-<wire x1="127" y1="5.08" x2="132.08" y2="5.08" width="0" layer="91"/>
 <label x="132.08" y="5.08" size="1.778" layer="95"/>
+<pinref part="C5" gate="G$1" pin="P$2"/>
+<wire x1="127" y1="5.08" x2="144.78" y2="5.08" width="0" layer="91"/>
 </segment>
 </net>
@@
 <segment>
 <pinref part="PROG0" gate="A" pin="2"/>
-<wire x1="127" y1="10.16" x2="132.08" y2="10.16" width="0" layer="91"/>
 <label x="132.08" y="10.16" size="1.778" layer="95"/>
-</segment>
-</net>
+<wire x1="127" y1="10.16" x2="142.24" y2="10.16" width="0" layer="91"/>
+<wire x1="142.24" y1="10.16" x2="142.24" y2="12.7" width="0" layer="91"/>
+<pinref part="C5" gate="G$1" pin="P$1"/>
+<wire x1="142.24" y1="12.7" x2="144.78" y2="12.7" width="0" layer="91"/>
+</segment>
+</net>

Commit message: major rework of tesselate file - needs a tiny bit of tweaking for full tesselation
Parts:
- removed PROG0: (no value), nonolith:HEADER-2X3
- renumbered S00 to 0, S10 to 1, S20 to 2, S30 to 3, S40 to 4
Connections:
- net 3.3V: no longer PROG0.2
- net GND: no longer PROG0.6
- net RESET0: no longer PROG0.5
- net RST40: no longer PROG0.1
- net SCL: no longer PROG0.3
- net SDA: no longer PROG0.4

Commit message: one index sensors
Parts:
- removed 0: MPL115A, nonolith:MPL115A
- added 5: MPL115A, nonolith:MPL115A
Connections:
- net 3.3V: now also 5.SHDN, 5.VDD; no longer 0.SHDN, 0.VDD
- net CAP00: now also 1.CAP; no longer 0.CAP
- net CAP10: now also 2.CAP; no longer 1.CAP
- net CAP20: now also 3.CAP; no longer 2.CAP
- net CAP30: now also 4.CAP; no longer 3.CAP
- net CAP40: now also 5.CAP; no longer 4.CAP
- net GND: now also 5.GND; no longer 0.GND
- net RST00: now also 1.RST; no longer 0.RST
- net RST10: now also 2.RST; no longer 1.RST
- net RST20: now also 3.RST; no longer 2.RST
- net RST30: now also 4.RST; no longer 3.RST
- net RST40: now also 5.RST; no longer 4.RST
- net SCL: now also 5.SCL; no longer 0.SCL
- net SDA: now also 5.SDA; no longer 0.SDA
Other:
- moved on the sheet: 1, 2, 3, 4
Changed lines of the file:
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@@
 <parts>
 <part name="UC0" library="nonolith" deviceset="ATTINY24" device="QFN"/>
-<part name="0" library="nonolith" deviceset="MPL115A" device=""/>
 <part name="1" library="nonolith" deviceset="MPL115A" device=""/>
 <part name="2" library="nonolith" deviceset="MPL115A" device=""/>
+<part name="3" library="nonolith" deviceset="MPL115A" device=""/>
 <part name="C0" library="nonolith" deviceset="CAP_CERAMIC" device="0402"/>
 <part name="C1" library="nonolith" deviceset="CAP_CERAMIC" device="0402"/>
 <part name="C2" library="nonolith" deviceset="CAP_CERAMIC" device="0402"/>
-<part name="3" library="nonolith" deviceset="MPL115A" device=""/>
 <part name="4" library="nonolith" deviceset="MPL115A" device=""/>
+<part name="5" library="nonolith" deviceset="MPL115A" device=""/>
 <part name="C3" library="nonolith" deviceset="CAP_CERAMIC" device="0402"/>
 <part name="C4" library="nonolith" deviceset="CAP_CERAMIC" device="0402"/>
@@
 <instances>
 <instance part="UC0" gate="G$1" x="30.48" y="17.78"/>
-<instance part="0" gate="G$1" x="33.02" y="60.96"/>
-<instance part="1" gate="G$1" x="76.2" y="60.96"/>
-<instance part="2" gate="G$1" x="114.3" y="60.96"/>
+<instance part="1" gate="G$1" x="33.02" y="60.96"/>
+<instance part="2" gate="G$1" x="76.2" y="60.96"/>
+<instance part="3" gate="G$1" x="114.3" y="60.96"/>
 <instance part="C0" gate="G$1" x="15.24" y="58.42"/>
 <instance part="C1" gate="G$1" x="58.42" y="58.42"/>
 <instance part="C2" gate="G$1" x="96.52" y="58.42"/>
-<instance part="3" gate="G$1" x="152.4" y="60.96"/>
-<instance part="4" gate="G$1" x="190.5" y="60.96"/>
+<instance part="4" gate="G$1" x="152.4" y="60.96"/>
+<instance part="5" gate="G$1" x="190.5" y="60.96"/>
 <instance part="C3" gate="G$1" x="134.62" y="58.42"/>
 <instance part="C4" gate="G$1" x="172.72" y="58.42"/>
@@
 <wire x1="96.52" y1="63.5" x2="101.6" y2="63.5" width="0" layer="91"/>
 <pinref part="C2" gate="G$1" pin="P$1"/>
-<pinref part="2" gate="G$1" pin="CAP"/>
+<pinref part="3" gate="G$1" pin="CAP"/>
 </segment>
 </net>
@@
 <segment>
 <wire x1="139.7" y1="63.5" x2="134.62" y2="63.5" width="0" layer="91"/>
-<pinref part="3" gate="G$1" pin="CAP"/>
+<pinref part="4" gate="G$1" pin="CAP"/>
 <pinref part="C3" gate="G$1" pin="P$1"/>
 </segment>
@@
 <wire x1="172.72" y1="63.5" x2="177.8" y2="63.5" width="0" layer="91"/>
 <pinref part="C4" gate="G$1" pin="P$1"/>
-<pinref part="4" gate="G$1" pin="CAP"/>
+<pinref part="5" gate="G$1" pin="CAP"/>
 </segment>
 </net>
@@
 <wire x1="60.96" y1="55.88" x2="60.96" y2="58.42" width="0" layer="91"/>
 <wire x1="58.42" y1="55.88" x2="60.96" y2="55.88" width="0" layer="91"/>
-<pinref part="1" gate="G$1" pin="GND"/>
+<pinref part="2" gate="G$1" pin="GND"/>
 <pinref part="C1" gate="G$1" pin="P$2"/>
 </segment>
@@
 <wire x1="99.06" y1="55.88" x2="99.06" y2="58.42" width="0" layer="91"/>
 <wire x1="96.52" y1="55.88" x2="99.06" y2="55.88" width="0" layer="91"/>
-<pinref part="2" gate="G$1" pin="GND"/>
+<pinref part="3" gate="G$1" pin="GND"/>
 <pinref part="C2" gate="G$1" pin="P$2"/>
 </segment>
@@
 <wire x1="137.16" y1="55.88" x2="137.16" y2="58.42" width="0" layer="91"/>
 <wire x1="134.62" y1="55.88" x2="137.16" y2="55.88" width="0" layer="91"/>
-<pinref part="3" gate="G$1" pin="GND"/>
+<pinref part="4" gate="G$1" pin="GND"/>
 <pinref part="C3" gate="G$1" pin="P$2"/>
 </segment>
@@
 <wire x1="175.26" y1="55.88" x2="175.26" y2="58.42" width="0" layer="91"/>
 <wire x1="172.72" y1="55.88" x2="175.26" y2="55.88" width="0" layer="91"/>
-<pinref part="4" gate="G$1" pin="GND"/>
+<pinref part="5" gate="G$1" pin="GND"/>
 <pinref part="C4" gate="G$1" pin="P$2"/>
 </segment>
@@
 <wire x1="17.78" y1="55.88" x2="17.78" y2="58.42" width="0" layer="91"/>
 <wire x1="15.24" y1="55.88" x2="17.78" y2="55.88" width="0" layer="91"/>
-<pinref part="0" gate="G$1" pin="GND"/>
+<pinref part="1" gate="G$1" pin="GND"/>
 <pinref part="C0" gate="G$1" pin="P$2"/>
 </segment>
@@
 <wire x1="63.5" y1="68.58" x2="60.96" y2="68.58" width="0" layer="91"/>
 <label x="60.96" y="68.58" size="1.778" layer="95" rot="R180"/>
-<pinref part="1" gate="G$1" pin="VDD"/>
+<pinref part="2" gate="G$1" pin="VDD"/>
 </segment>
 <segment>
 <wire x1="20.32" y1="68.58" x2="17.78" y2="68.58" width="0" layer="91"/>
 <label x="17.78" y="68.58" size="1.778" layer="95" rot="R180"/>
-<pinref part="0" gate="G$1" pin="VDD"/>
+<pinref part="1" gate="G$1" pin="VDD"/>
 </segment>
 <segment>
 <wire x1="101.6" y1="68.58" x2="99.06" y2="68.58" width="0" layer="91"/>
 <label x="99.06" y="68.58" size="1.778" layer="95" rot="R180"/>
-<pinref part="2" gate="G$1" pin="VDD"/>
+<pinref part="3" gate="G$1" pin="VDD"/>
 </segment>
 <segment>
 <wire x1="139.7" y1="68.58" x2="137.16" y2="68.58" width="0" layer="91"/>
 <label x="137.16" y="68.58" size="1.778" layer="95" rot="R180"/>
-<pinref part="3" gate="G$1" pin="VDD"/>
+<pinref part="4" gate="G$1" pin="VDD"/>
 </segment>
 <segment>
 <wire x1="177.8" y1="68.58" x2="175.26" y2="68.58" width="0" layer="91"/>
 <label x="175.26" y="68.58" size="1.778" layer="95" rot="R180"/>
-<pinref part="4" gate="G$1" pin="VDD"/>
+<pinref part="5" gate="G$1" pin="VDD"/>
 </segment>
 <segment>
@@
 <wire x1="63.5" y1="53.34" x2="60.96" y2="53.34" width="0" layer="91"/>
 <label x="60.96" y="53.34" size="1.778" layer="95" rot="R180"/>
-<pinref part="1" gate="G$1" pin="SHDN"/>
+<pinref part="2" gate="G$1" pin="SHDN"/>
 </segment>
 <segment>
 <wire x1="101.6" y1="53.34" x2="99.06" y2="53.34" width="0" layer="91"/>
 <label x="99.06" y="53.34" size="1.778" layer="95" rot="R180"/>
-<pinref part="2" gate="G$1" pin="SHDN"/>
+<pinref part="3" gate="G$1" pin="SHDN"/>
 </segment>
 <segment>
 <wire x1="139.7" y1="53.34" x2="137.16" y2="53.34" width="0" layer="91"/>
 <label x="137.16" y="53.34" size="1.778" layer="95" rot="R180"/>
-<pinref part="3" gate="G$1" pin="SHDN"/>
+<pinref part="4" gate="G$1" pin="SHDN"/>
 </segment>
 <segment>
 <wire x1="177.8" y1="53.34" x2="175.26" y2="53.34" width="0" layer="91"/>
 <label x="175.26" y="53.34" size="1.778" layer="95" rot="R180"/>
-<pinref part="4" gate="G$1" pin="SHDN"/>
+<pinref part="5" gate="G$1" pin="SHDN"/>
 </segment>
 <segment>
 <wire x1="20.32" y1="53.34" x2="17.78" y2="53.34" width="0" layer="91"/>
 <label x="17.78" y="53.34" size="1.778" layer="95" rot="R180"/>
-<pinref part="0" gate="G$1" pin="SHDN"/>
+<pinref part="1" gate="G$1" pin="SHDN"/>
 </segment>
 <segment>
@@
 <wire x1="15.24" y1="63.5" x2="20.32" y2="63.5" width="0" layer="91"/>
 <pinref part="C0" gate="G$1" pin="P$1"/>
-<pinref part="0" gate="G$1" pin="CAP"/>
+<pinref part="1" gate="G$1" pin="CAP"/>
 </segment>
 </net>
@@
 <junction x="55.88" y="73.66"/>
 <label x="58.42" y="17.78" size="1.778" layer="95"/>
-<pinref part="0" gate="G$1" pin="SDA"/>
+<pinref part="1" gate="G$1" pin="SDA"/>
+<pinref part="5" gate="G$1" pin="SDA"/>
 <pinref part="4" gate="G$1" pin="SDA"/>
 <pinref part="3" gate="G$1" pin="SDA"/>
 <pinref part="2" gate="G$1" pin="SDA"/>
-<pinref part="1" gate="G$1" pin="SDA"/>
 <pinref part="UC0" gate="G$1" pin="PA6/MOSI"/>
 </segment>
@@
 <label x="58.42" y="22.86" size="1.778" layer="95"/>
 <pinref part="UC0" gate="G$1" pin="PA4/SCL"/>
-<pinref part="0" gate="G$1" pin="SCL"/>
+<pinref part="1" gate="G$1" pin="SCL"/>
+<pinref part="5" gate="G$1" pin="SCL"/>
 <pinref part="4" gate="G$1" pin="SCL"/>
 <pinref part="3" gate="G$1" pin="SCL"/>
 <pinref part="2" gate="G$1" pin="SCL"/>
-<pinref part="1" gate="G$1" pin="SCL"/>
 </segment>
 </net>
@@
 <label x="58.42" y="33.02" size="1.778" layer="95"/>
 <pinref part="UC0" gate="G$1" pin="PA0/ADC0"/>
-<pinref part="0" gate="G$1" pin="RST"/>
+<pinref part="1" gate="G$1" pin="RST"/>
 </segment>
 </net>
@@
 <label x="58.42" y="30.48" size="1.778" layer="95"/>
 <pinref part="UC0" gate="G$1" pin="PA1/ADC1"/>
-<pinref part="1" gate="G$1" pin="RST"/>
+<pinref part="2" gate="G$1" pin="RST"/>
 </segment>
 </net>
@@
 <label x="58.42" y="27.94" size="1.778" layer="95"/>
 <pinref part="UC0" gate="G$1" pin="PA2/ADC2"/>
-<pinref part="2" gate="G$1" pin="RST"/>
+<pinref part="3" gate="G$1" pin="RST"/>
 </segment>
 </net>
@@
 <label x="58.42" y="25.4" size="1.778" layer="95"/>
 <pinref part="UC0" gate="G$1" pin="PA3/ADC3"/>
-<pinref part="3" gate="G$1" pin="RST"/>
+<pinref part="4" gate="G$1" pin="RST"/>
 </segment>
 </net>
@@
 <wire x1="58.42" y1="63.5" x2="63.5" y2="63.5" width="0" layer="91"/>
 <pinref part="C1" gate="G$1" pin="P$1"/>
-<pinref part="1" gate="G$1" pin="CAP"/>
+<pinref part="2" gate="G$1" pin="CAP"/>
 </segment>
 </net>
@@
 <label x="58.42" y="20.32" size="1.778" layer="95"/>
 <pinref part="UC0" gate="G$1" pin="PA5/MISO"/>
-<pinref part="4" gate="G$1" pin="RST"/>
-</segment>
-</net>
+<pinref part="5" gate="G$1" pin="RST"/>
+</segment>
+</net>
