File: eagle/tessellate.sch (EAGLE design)
At the start: 12 parts

Commit message: rename some signals and stuff
Parts:
- removed C0: (no value), nonolith:CAP_CERAMIC0402
- added C6: (no value), nonolith:CAP_CERAMIC0402
- renumbered UC0 to UC1
Connections:
- net RESET0 renamed RESET1
- net RST00 renamed RST1
- net RST10 renamed RST2
- net RST20 renamed RST3
- net RST30 renamed RST4
- net RST40 renamed RST5
- net 3.3V: now also C6.P$1; no longer C5.P$1
- net CAP00: now also C1.P$1; no longer C0.P$1
- net CAP10: now also C2.P$1; no longer C1.P$1
- net CAP20: now also C3.P$1; no longer C2.P$1
- net CAP30: now also C4.P$1; no longer C3.P$1
- net CAP40: now also C5.P$1; no longer C4.P$1
- net GND: now also C6.P$2; no longer C0.P$2
Other:
- moved on the sheet: C1, C2, C3, C4, C5
Changed lines of the file:
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@@
 </classes>
 <parts>
-<part name="UC0" library="nonolith" deviceset="ATTINY24" device="QFN"/>
+<part name="UC1" library="nonolith" deviceset="ATTINY24" device="QFN"/>
 <part name="1" library="nonolith" deviceset="MPL115A" device=""/>
 <part name="2" library="nonolith" deviceset="MPL115A" device=""/>
 <part name="3" library="nonolith" deviceset="MPL115A" device=""/>
-<part name="C0" library="nonolith" deviceset="CAP_CERAMIC" device="0402"/>
 <part name="C1" library="nonolith" deviceset="CAP_CERAMIC" device="0402"/>
 <part name="C2" library="nonolith" deviceset="CAP_CERAMIC" device="0402"/>
+<part name="C3" library="nonolith" deviceset="CAP_CERAMIC" device="0402"/>
 <part name="4" library="nonolith" deviceset="MPL115A" device=""/>
 <part name="5" library="nonolith" deviceset="MPL115A" device=""/>
-<part name="C3" library="nonolith" deviceset="CAP_CERAMIC" device="0402"/>
 <part name="C4" library="nonolith" deviceset="CAP_CERAMIC" device="0402"/>
 <part name="C5" library="nonolith" deviceset="CAP_CERAMIC" device="0402"/>
+<part name="C6" library="nonolith" deviceset="CAP_CERAMIC" device="0402"/>
 </parts>
 <sheets>
@@
 </plain>
 <instances>
-<instance part="UC0" gate="G$1" x="30.48" y="17.78"/>
+<instance part="UC1" gate="G$1" x="30.48" y="17.78"/>
 <instance part="1" gate="G$1" x="33.02" y="60.96"/>
 <instance part="2" gate="G$1" x="76.2" y="60.96"/>
 <instance part="3" gate="G$1" x="114.3" y="60.96"/>
-<instance part="C0" gate="G$1" x="15.24" y="58.42"/>
-<instance part="C1" gate="G$1" x="58.42" y="58.42"/>
-<instance part="C2" gate="G$1" x="96.52" y="58.42"/>
+<instance part="C1" gate="G$1" x="15.24" y="58.42"/>
+<instance part="C2" gate="G$1" x="58.42" y="58.42"/>
+<instance part="C3" gate="G$1" x="96.52" y="58.42"/>
 <instance part="4" gate="G$1" x="152.4" y="60.96"/>
 <instance part="5" gate="G$1" x="190.5" y="60.96"/>
-<instance part="C3" gate="G$1" x="134.62" y="58.42"/>
-<instance part="C4" gate="G$1" x="172.72" y="58.42"/>
-<instance part="C5" gate="G$1" x="144.78" y="7.62"/>
+<instance part="C4" gate="G$1" x="134.62" y="58.42"/>
+<instance part="C5" gate="G$1" x="172.72" y="58.42"/>
+<instance part="C6" gate="G$1" x="144.78" y="7.62"/>
 </instances>
 <busses>
@@
 <segment>
 <wire x1="96.52" y1="63.5" x2="101.6" y2="63.5" width="0" layer="91"/>
-<pinref part="C2" gate="G$1" pin="P$1"/>
+<pinref part="C3" gate="G$1" pin="P$1"/>
 <pinref part="3" gate="G$1" pin="CAP"/>
 </segment>
@@
 <wire x1="139.7" y1="63.5" x2="134.62" y2="63.5" width="0" layer="91"/>
 <pinref part="4" gate="G$1" pin="CAP"/>
-<pinref part="C3" gate="G$1" pin="P$1"/>
+<pinref part="C4" gate="G$1" pin="P$1"/>
 </segment>
 </net>
@@
 <segment>
 <wire x1="172.72" y1="63.5" x2="177.8" y2="63.5" width="0" layer="91"/>
-<pinref part="C4" gate="G$1" pin="P$1"/>
+<pinref part="C5" gate="G$1" pin="P$1"/>
 <pinref part="5" gate="G$1" pin="CAP"/>
 </segment>
@@
 <wire x1="7.62" y1="5.08" x2="7.62" y2="2.54" width="0" layer="91"/>
 <label x="7.62" y="2.54" size="1.778" layer="95" rot="R180"/>
-<pinref part="UC0" gate="G$1" pin="GND"/>
-<pinref part="UC0" gate="G$1" pin="GND@0"/>
+<pinref part="UC1" gate="G$1" pin="GND"/>
+<pinref part="UC1" gate="G$1" pin="GND@0"/>
 </segment>
 <segment>
@@
 <wire x1="58.42" y1="55.88" x2="60.96" y2="55.88" width="0" layer="91"/>
 <pinref part="2" gate="G$1" pin="GND"/>
-<pinref part="C1" gate="G$1" pin="P$2"/>
+<pinref part="C2" gate="G$1" pin="P$2"/>
 </segment>
 <segment>
@@
 <wire x1="96.52" y1="55.88" x2="99.06" y2="55.88" width="0" layer="91"/>
 <pinref part="3" gate="G$1" pin="GND"/>
-<pinref part="C2" gate="G$1" pin="P$2"/>
+<pinref part="C3" gate="G$1" pin="P$2"/>
 </segment>
 <segment>
@@
 <wire x1="134.62" y1="55.88" x2="137.16" y2="55.88" width="0" layer="91"/>
 <pinref part="4" gate="G$1" pin="GND"/>
-<pinref part="C3" gate="G$1" pin="P$2"/>
+<pinref part="C4" gate="G$1" pin="P$2"/>
 </segment>
 <segment>
@@
 <wire x1="172.72" y1="55.88" x2="175.26" y2="55.88" width="0" layer="91"/>
 <pinref part="5" gate="G$1" pin="GND"/>
-<pinref part="C4" gate="G$1" pin="P$2"/>
+<pinref part="C5" gate="G$1" pin="P$2"/>
 </segment>
 <segment>
@@
 <wire x1="15.24" y1="55.88" x2="17.78" y2="55.88" width="0" layer="91"/>
 <pinref part="1" gate="G$1" pin="GND"/>
-<pinref part="C0" gate="G$1" pin="P$2"/>
-</segment>
-<segment>
-<pinref part="UC0" gate="G$1" pin="PA7/ADC7"/>
+<pinref part="C1" gate="G$1" pin="P$2"/>
+</segment>
+<segment>
+<pinref part="UC1" gate="G$1" pin="PA7/ADC7"/>
 <wire x1="50.8" y1="15.24" x2="53.34" y2="15.24" width="0" layer="91"/>
 <label x="53.34" y="15.24" size="1.778" layer="95"/>
 </segment>
 <segment>
-<pinref part="UC0" gate="G$1" pin="PB1"/>
+<pinref part="UC1" gate="G$1" pin="PB1"/>
 <wire x1="50.8" y1="7.62" x2="53.34" y2="7.62" width="0" layer="91"/>
 <label x="53.34" y="7.62" size="1.778" layer="95"/>
 </segment>
 <segment>
-<pinref part="UC0" gate="G$1" pin="PB2"/>
+<pinref part="UC1" gate="G$1" pin="PB2"/>
 <wire x1="50.8" y1="5.08" x2="53.34" y2="5.08" width="0" layer="91"/>
 <label x="53.34" y="5.08" size="1.778" layer="95"/>
@@
 <segment>
 <label x="139.7" y="5.08" size="1.778" layer="95" rot="R180"/>
-<pinref part="C5" gate="G$1" pin="P$2"/>
+<pinref part="C6" gate="G$1" pin="P$2"/>
 <wire x1="139.7" y1="5.08" x2="144.78" y2="5.08" width="0" layer="91"/>
 </segment>
@@
 <wire x1="10.16" y1="33.02" x2="7.62" y2="33.02" width="0" layer="91"/>
 <label x="7.62" y="33.02" size="1.778" layer="95" rot="R180"/>
-<pinref part="UC0" gate="G$1" pin="VCC"/>
+<pinref part="UC1" gate="G$1" pin="VCC"/>
 </segment>
 <segment>
@@
 <segment>
 <label x="139.7" y="12.7" size="1.778" layer="95" rot="R180"/>
-<pinref part="C5" gate="G$1" pin="P$1"/>
+<pinref part="C6" gate="G$1" pin="P$1"/>
 <wire x1="139.7" y1="12.7" x2="144.78" y2="12.7" width="0" layer="91"/>
 </segment>
@@
 <segment>
 <wire x1="15.24" y1="63.5" x2="20.32" y2="63.5" width="0" layer="91"/>
-<pinref part="C0" gate="G$1" pin="P$1"/>
+<pinref part="C1" gate="G$1" pin="P$1"/>
 <pinref part="1" gate="G$1" pin="CAP"/>
 </segment>
@@
 <pinref part="3" gate="G$1" pin="SDA"/>
 <pinref part="2" gate="G$1" pin="SDA"/>
-<pinref part="UC0" gate="G$1" pin="PA6/MOSI"/>
+<pinref part="UC1" gate="G$1" pin="PA6/MOSI"/>
 </segment>
 </net>
@@
 <junction x="53.34" y="78.74"/>
 <label x="58.42" y="22.86" size="1.778" layer="95"/>
-<pinref part="UC0" gate="G$1" pin="PA4/SCL"/>
+<pinref part="UC1" gate="G$1" pin="PA4/SCL"/>
 <pinref part="1" gate="G$1" pin="SCL"/>
 <pinref part="5" gate="G$1" pin="SCL"/>
@@
 </segment>
 </net>
-<net name="RST00" class="0">
+<net name="RST1" class="0">
 <segment>
 <wire x1="50.8" y1="33.02" x2="50.8" y2="53.34" width="0" layer="91"/>
 <wire x1="50.8" y1="53.34" x2="45.72" y2="53.34" width="0" layer="91"/>
 <label x="58.42" y="33.02" size="1.778" layer="95"/>
-<pinref part="UC0" gate="G$1" pin="PA0/ADC0"/>
+<pinref part="UC1" gate="G$1" pin="PA0/ADC0"/>
 <pinref part="1" gate="G$1" pin="RST"/>
 </segment>
 </net>
-<net name="RST10" class="0">
+<net name="RST2" class="0">
 <segment>
 <wire x1="50.8" y1="30.48" x2="88.9" y2="30.48" width="0" layer="91"/>
 <wire x1="88.9" y1="30.48" x2="88.9" y2="53.34" width="0" layer="91"/>
 <label x="58.42" y="30.48" size="1.778" layer="95"/>
-<pinref part="UC0" gate="G$1" pin="PA1/ADC1"/>
+<pinref part="UC1" gate="G$1" pin="PA1/ADC1"/>
 <pinref part="2" gate="G$1" pin="RST"/>
 </segment>
 </net>
-<net name="RST20" class="0">
+<net name="RST3" class="0">
 <segment>
 <wire x1="50.8" y1="27.94" x2="127" y2="27.94" width="0" layer="91"/>
 <wire x1="127" y1="27.94" x2="127" y2="53.34" width="0" layer="91"/>
 <label x="58.42" y="27.94" size="1.778" layer="95"/>
-<pinref part="UC0" gate="G$1" pin="PA2/ADC2"/>
+<pinref part="UC1" gate="G$1" pin="PA2/ADC2"/>
 <pinref part="3" gate="G$1" pin="RST"/>
 </segment>
 </net>
-<net name="RST30" class="0">
+<net name="RST4" class="0">
 <segment>
 <wire x1="50.8" y1="25.4" x2="165.1" y2="25.4" width="0" layer="91"/>
 <wire x1="165.1" y1="25.4" x2="165.1" y2="53.34" width="0" layer="91"/>
 <label x="58.42" y="25.4" size="1.778" layer="95"/>
-<pinref part="UC0" gate="G$1" pin="PA3/ADC3"/>
+<pinref part="UC1" gate="G$1" pin="PA3/ADC3"/>
 <pinref part="4" gate="G$1" pin="RST"/>
 </segment>
@@
 <segment>
 <wire x1="58.42" y1="63.5" x2="63.5" y2="63.5" width="0" layer="91"/>
-<pinref part="C1" gate="G$1" pin="P$1"/>
+<pinref part="C2" gate="G$1" pin="P$1"/>
 <pinref part="2" gate="G$1" pin="CAP"/>
 </segment>
 </net>
-<net name="RESET0" class="0">
+<net name="RESET1" class="0">
 <segment>
 <wire x1="50.8" y1="2.54" x2="55.88" y2="2.54" width="0" layer="91"/>
 <label x="55.88" y="2.54" size="1.778" layer="95"/>
-<pinref part="UC0" gate="G$1" pin="PB3/RESET"/>
-</segment>
-</net>
-<net name="RST40" class="0">
+<pinref part="UC1" gate="G$1" pin="PB3/RESET"/>
+</segment>
+</net>
+<net name="RST5" class="0">
 <segment>
 <wire x1="50.8" y1="20.32" x2="203.2" y2="20.32" width="0" layer="91"/>
 <wire x1="203.2" y1="20.32" x2="203.2" y2="53.34" width="0" layer="91"/>
 <label x="58.42" y="20.32" size="1.778" layer="95"/>
-<pinref part="UC0" gate="G$1" pin="PA5/MISO"/>
+<pinref part="UC1" gate="G$1" pin="PA5/MISO"/>
 <pinref part="5" gate="G$1" pin="RST"/>
 </segment>
@@
 <net name="ADDR00" class="0">
 <segment>
-<pinref part="UC0" gate="G$1" pin="PB0"/>
+<pinref part="UC1" gate="G$1" pin="PB0"/>
 <wire x1="50.8" y1="10.16" x2="53.34" y2="10.16" width="0" layer="91"/>
 <label x="53.34" y="10.16" size="1.778" layer="95"/>

Commit message: fix numbering scheme for tesselation
Parts:
- renumbered 1 to 01, 2 to 02, 3 to 03, 4 to 04, 5 to 05, C1 to C01, C2 to C02, C3 to C03, C4 to C04, C5 to C05, UC1 to UC01
Connections:
- net CAP00 renamed CAP01
- net CAP10 renamed CAP02
- net CAP20 renamed CAP03
- net CAP30 renamed CAP04
- net CAP40 renamed CAP05
- net RESET1 renamed RESET01
- net RST1 renamed RST01
- net RST2 renamed RST02
- net RST3 renamed RST03
- net RST4 renamed RST04
- net RST5 renamed RST05
